File: REVISION 1/211006_lmu_r0/Lower Active Balance Group.sch (KiCad schematic (older format))
At the start: 7 parts

Commit message: Finished schematic, ready for pcb layout
Parts:
- removed C?: 100n, symbol Device:C
- removed D?: D_Schottky, symbol Device:D_Schottky
- removed R?: 23.7k, symbol Device:R
- removed R?: R, symbol Device:R
- removed R?: 33.2k, symbol Device:R
- removed R?: 1M, symbol Device:R
- removed U?: LTC3300ILXE-2#PBF, QFP50P900X900X160-49N, symbol LTC3300ILXE-2_PBF:LTC3300ILXE-2#PBF
- added C?: 100n, symbol Device:C
- added D?: D_Schottky, symbol Device:D_Schottky
- added R?: 33.2k, symbol Device:R
- added R?: 1M, symbol Device:R
- added R?: 23.7k, symbol Device:R
- added R?: R, symbol Device:R
- added U?: LTC3300ILXE-2#PBF, QFP50P900X900X160-49N, symbol LTC3300ILXE-2_PBF:LTC3300ILXE-2#PBF
Connections:
- net A0: now also U?.43 (A0)
- net A1: now also U?.44 (A1)
- net A2: now also U?.45 (A2)
- net A3: now also U?.46 (A3)
- net A4: now also U?.47 (A4)
- net ACTIVE_TAP0: now also R?.2, R?.2, U?.15 (CTRL), U?.21 (V-), U?.49 (V-)
- net C1: now also U?.24 (C1)
- net C2: now also U?.27 (C2)
- net C3: now also U?.30 (C3)
- net C4: now also U?.33 (C4)
- net C5: now also U?.36 (C5)
- net C6: now also R?.2, U?.39 (C6)
- net PG1: now also U?.23 (G1P)
- net PG2: now also U?.26 (G2P)
- net PG3: now also U?.29 (G3P)
- net PG4: now also U?.32 (G4P)
- net PG5: now also U?.35 (G5P)
- net PG6: now also U?.38 (G6P)
- net PI1: now also U?.22 (I1P)
- net PI2: now also U?.25 (I2P)
- net PI3: now also U?.28 (I3P)
- net PI4: now also U?.31 (I4P)
- net PI5: now also U?.34 (I5P)
- net PI6: now also U?.37 (I6P)
- net SCKI: now also U?.17 (SCKI)
- net SDI: now also U?.18 (SDI)
- net SDO: now also U?.19 (SDO)
- net SG1: now also U?.11 (G1S)
- net SG2: now also U?.9 (G2S)
- net SG3: now also U?.7 (G3S)
- net SG4: now also U?.5 (G4S)
- net SG5: now also U?.3 (G5S)
- net SG6: now also U?.1 (G6S)
- net SI1: now also U?.12 (I1S)
- net SI2: now also U?.10 (I2S)
- net SI3: now also U?.8 (I3S)
- net SI4: now also U?.6 (I4S)
- net SI5: now also U?.4 (I5S)
- net SI6: now also U?.2 (I6S)
- net VREG: now also R?.1, U?.42 (BOOST), U?.48 (VREG)
- net WDT: now also R?.2, U?.20 (WDT)
- net nCSBI: now also U?.16 (~CSBI)
- new net: R?.1, U?.13 (RTONS)
- new net: R?.1, U?.14 (RTONP)
- new net: C?.1, U?.40 (BOOSTP)
- new net: C?.2, D?.1 (K), U?.41 (BOOSTN)
- new net: D?.2 (A), R?.1
Changed lines of the file:
@@
 $Sheet
 S 2700 600  1400 1000
-U 6234DCC2
+U 6196A6CE
 F0 "Active_Passive_Balance_Filter" 50
 F1 "active_passive_balance.sch" 50
@@
 $Sheet
 S 2700 1800 1400 1000
-U 6196DB56
+U 6234DCC3
 F0 "sheet6196DB49" 50
 F1 "active_passive_balance.sch" 50
@@
 $Sheet
 S 2700 3050 1400 1000
-U 6196F035
+U 6234DCC4
 F0 "sheet6196F027" 50
 F1 "active_passive_balance.sch" 50
@@
 $Sheet
 S 2700 4250 1400 1000
-U 6196F042
+U 6234DCC5
 F0 "sheet6196F028" 50
 F1 "active_passive_balance.sch" 50
@@
 $Sheet
 S 2700 5500 1400 1000
-U 6196F9B1
+U 6234DCC6
 F0 "sheet6196F9A3" 50
 F1 "active_passive_balance.sch" 50
@@
 $Sheet
 S 2700 6700 1400 1000
-U 6196F9BE
+U 6234DCC7
 F0 "sheet6196F9A4" 50
 F1 "active_passive_balance.sch" 50
@@
 $Comp
 L LTC3300ILXE-2_PBF:LTC3300ILXE-2#PBF U?
-U 1 1 6234DCC8
+U 1 1 619B505D
 P 8050 3400
-AR Path="/6196A5FC/6234DCC8" Ref="U?"  Part="1"
-AR Path="/61619F34/6161AC01/6234DCC8" Ref="U?"  Part="1"
-AR Path="/61619F34/6161D6CD/6234DCC8" Ref="U?"  Part="1"
-AR Path="/61619F34/61F7AB68/6234DCC8" Ref="U?"  Part="1"
-AR Path="/61619F34/62061D33/6234DCC8" Ref="U?"  Part="1"
-AR Path="/61619F34/6209AB17/6234DCC8" Ref="U?"  Part="1"
+AR Path="/6196A5FC/619B505D" Ref="U?"  Part="1"
+AR Path="/61619F34/6161AC01/619B505D" Ref="U?"  Part="1"
+AR Path="/61619F34/6161D6CD/619B505D" Ref="U?"  Part="1"
+AR Path="/61619F34/61F7AB68/619B505D" Ref="U?"  Part="1"
+AR Path="/61619F34/62061D33/619B505D" Ref="U?"  Part="1"
+AR Path="/61619F34/6209AB17/619B505D" Ref="U?"  Part="1"
 F 0 "U?" H 8050 4970 50  0000 C CNN
 F 1 "LTC3300ILXE-2#PBF" H 8050 4879 50  0000 C CNN
@@
 $Comp
 L Device:R R?
-U 1 1 61F30A1E
+U 1 1 6234DCC9
 P 10250 4500
-AR Path="/61619F34/6161AC01/61F30A1E" Ref="R?"  Part="1"
-AR Path="/61619F34/61F7AB68/61F30A1E" Ref="R?"  Part="1"
-AR Path="/61619F34/62061D33/61F30A1E" Ref="R?"  Part="1"
-AR Path="/61619F34/6209AB17/61F30A1E" Ref="R?"  Part="1"
+AR Path="/61619F34/6161AC01/6234DCC9" Ref="R?"  Part="1"
+AR Path="/61619F34/61F7AB68/6234DCC9" Ref="R?"  Part="1"
+AR Path="/61619F34/62061D33/6234DCC9" Ref="R?"  Part="1"
+AR Path="/61619F34/6209AB17/6234DCC9" Ref="R?"  Part="1"
 F 0 "R?" H 10320 4546 50  0000 L CNN
 F 1 "23.7k" H 10320 4455 50  0000 L CNN
@@
 $Comp
 L Device:R R?
-U 1 1 6234DCCA
+U 1 1 61F36DB3
 P 10600 4500
-AR Path="/61619F34/6161AC01/6234DCCA" Ref="R?"  Part="1"
-AR Path="/61619F34/61F7AB68/6234DCCA" Ref="R?"  Part="1"
-AR Path="/61619F34/62061D33/6234DCCA" Ref="R?"  Part="1"
-AR Path="/61619F34/6209AB17/6234DCCA" Ref="R?"  Part="1"
+AR Path="/61619F34/6161AC01/61F36DB3" Ref="R?"  Part="1"
+AR Path="/61619F34/61F7AB68/61F36DB3" Ref="R?"  Part="1"
+AR Path="/61619F34/62061D33/61F36DB3" Ref="R?"  Part="1"
+AR Path="/61619F34/6209AB17/61F36DB3" Ref="R?"  Part="1"
 F 0 "R?" H 10670 4546 50  0000 L CNN
 F 1 "33.2k" H 10670 4455 50  0000 L CNN
@@
 $Comp
 L Device:D_Schottky D?
-U 1 1 6222295F
+U 1 1 6234DCCB
 P 9450 4900
 F 0 "D?" V 9404 4980 50  0000 L CNN
@@
 $Comp
 L Device:R R?
-U 1 1 622462AA
+U 1 1 6234DCCC
 P 9450 5200
 F 0 "R?" H 9520 5246 50  0000 L CNN
@@
 $Comp
 L Device:C C?
-U 1 1 62253C9B
+U 1 1 6234DCCD
 P 9800 4550
 F 0 "C?" H 9915 4596 50  0000 L CNN
@@
 $Comp
 L Device:R R?
-U 1 1 6234DCCE
+U 1 1 6228C6A6
 P 10050 3300
-AR Path="/61619F34/6161AC01/6234DCCE" Ref="R?"  Part="1"
-AR Path="/61619F34/61F7AB68/6234DCCE" Ref="R?"  Part="1"
-AR Path="/61619F34/62061D33/6234DCCE" Ref="R?"  Part="1"
-AR Path="/61619F34/6209AB17/6234DCCE" Ref="R?"  Part="1"
+AR Path="/61619F34/6161AC01/6228C6A6" Ref="R?"  Part="1"
+AR Path="/61619F34/61F7AB68/6228C6A6" Ref="R?"  Part="1"
+AR Path="/61619F34/62061D33/6228C6A6" Ref="R?"  Part="1"
+AR Path="/61619F34/6209AB17/6228C6A6" Ref="R?"  Part="1"
 F 0 "R?" H 10120 3346 50  0000 L CNN
 F 1 "1M" H 10120 3255 50  0000 L CNN
