File: REVISION 1/211006_lmu_r0/Lwer Active Balance Group.sch (KiCad schematic (older format))
At the start: 7 parts

Commit message: Finished schematic, ready for pcb layout
Parts:
- removed C?: 100n, symbol Device:C
- removed D?: D_Schottky, symbol Device:D_Schottky
- removed R?: R, symbol Device:R
- removed R?: 33.2k, symbol Device:R
- removed R?: 1M, symbol Device:R
- removed U?: LTC3300ILXE-2#PBF, QFP50P900X900X160-49N, symbol LTC3300ILXE-2_PBF:LTC3300ILXE-2#PBF
- added R?: R, symbol Device:R
- added U?: LTC3300ILXE-2#PBF, QFP50P900X900X160-49N, symbol LTC3300ILXE-2_PBF:LTC3300ILXE-2#PBF
- R?: value 23.7k -> R
Connections:
- net A0: now also U?.43 (A0)
- net A1: now also U?.44 (A1)
- net A2: now also U?.45 (A2)
- net A3: now also U?.46 (A3)
- net A4: now also U?.47 (A4)
- net ACTIVE_TAP0: now also R?.2, U?.15 (CTRL), U?.21 (V-), U?.49 (V-)
- net PG1: now also U?.23 (G1P)
- net PG2: now also U?.26 (G2P)
- net PG3: now also U?.29 (G3P)
- net PG4: now also U?.32 (G4P)
- net PG5: now also U?.35 (G5P)
- net PG6: now also U?.38 (G6P)
- net PI1: now also U?.22 (I1P)
- net PI2: now also U?.25 (I2P)
- net PI3: now also U?.28 (I3P)
- net PI4: now also U?.31 (I4P)
- net PI5: now also U?.34 (I5P)
- net PI6: now also U?.37 (I6P)
- net SCKI: now also U?.17 (SCKI)
- net SDI: now also U?.18 (SDI)
- net SDO: now also U?.19 (SDO)
- net SG1: now also U?.11 (G1S)
- net SG2: now also U?.9 (G2S)
- net SG3: now also U?.7 (G3S)
- net SG4: now also U?.5 (G4S)
- net SG5: now also U?.3 (G5S)
- net SG6: now also U?.1 (G6S)
- net SI1: now also U?.12 (I1S)
- net SI2: now also U?.10 (I2S)
- net SI3: now also U?.8 (I3S)
- net SI4: now also U?.6 (I4S)
- net SI5: now also U?.4 (I5S)
- net SI6: now also U?.2 (I6S)
- net VREG: now also U?.42 (BOOST), U?.48 (VREG)
- net nCSBI: now also U?.16 (~CSBI)
- net at R?.1: now also U?.41 (BOOSTN)
- new net: R?.1, U?.40 (BOOSTP)
Other:
- moved on the sheet: R?
Changed lines of the file:
@@
 $Descr A4 11693 8268
 encoding utf-8
-Sheet 24 35
+Sheet 16 32
 Title ""
 Date ""
@@
 $Sheet
 S 2700 600  1400 1000
-U 6234DCC2
+U 6196A6CE
 F0 "Active_Passive_Balance_Filter" 50
 F1 "active_passive_balance.sch" 50
@@
 $Comp
 L LTC3300ILXE-2_PBF:LTC3300ILXE-2#PBF U?
-U 1 1 6234DCC8
+U 1 1 619B505D
 P 8050 3400
-AR Path="/6196A5FC/6234DCC8" Ref="U?"  Part="1"
-AR Path="/61619F34/6161AC01/6234DCC8" Ref="U?"  Part="1"
-AR Path="/61619F34/6161D6CD/6234DCC8" Ref="U?"  Part="1"
-AR Path="/61619F34/61F7AB68/6234DCC8" Ref="U?"  Part="1"
-AR Path="/61619F34/62061D33/6234DCC8" Ref="U?"  Part="1"
-AR Path="/61619F34/6209AB17/6234DCC8" Ref="U?"  Part="1"
+AR Path="/6196A5FC/619B505D" Ref="U?"  Part="1"
+AR Path="/61619F34/6161AC01/619B505D" Ref="U?"  Part="1"
+AR Path="/61619F34/6161D6CD/619B505D" Ref="U?"  Part="1"
+AR Path="/61619F34/61F7AB68/619B505D" Ref="U?"  Part="1"
 F 0 "U?" H 8050 4970 50  0000 C CNN
 F 1 "LTC3300ILXE-2#PBF" H 8050 4879 50  0000 C CNN
@@
 L Device:R R?
 U 1 1 61F30A1E
-P 10250 4500
+P 9750 4700
 AR Path="/61619F34/6161AC01/61F30A1E" Ref="R?"  Part="1"
 AR Path="/61619F34/61F7AB68/61F30A1E" Ref="R?"  Part="1"
-AR Path="/61619F34/62061D33/61F30A1E" Ref="R?"  Part="1"
-AR Path="/61619F34/6209AB17/61F30A1E" Ref="R?"  Part="1"
-F 0 "R?" H 10320 4546 50  0000 L CNN
-F 1 "23.7k" H 10320 4455 50  0000 L CNN
-F 2 "" V 10180 4500 50  0001 C CNN
-F 3 "~" H 10250 4500 50  0001 C CNN
-	1    10250 4500
+F 0 "R?" H 9820 4746 50  0000 L CNN
+F 1 "R" H 9820 4655 50  0000 L CNN
+F 2 "" V 9680 4700 50  0001 C CNN
+F 3 "~" H 9750 4700 50  0001 C CNN
+	1    9750 4700
 	1    0    0    -1
 $EndComp
 Wire Wire Line
-	8950 4300 10250 4300
-Wire Wire Line
-	10250 4300 10250 4350
+	8950 4500 9750 4500
+Wire Wire Line
+	9750 4500 9750 4550
 $Comp
 L Device:R R?
-U 1 1 6234DCCA
-P 10600 4500
-AR Path="/61619F34/6161AC01/6234DCCA" Ref="R?"  Part="1"
-AR Path="/61619F34/61F7AB68/6234DCCA" Ref="R?"  Part="1"
-AR Path="/61619F34/62061D33/6234DCCA" Ref="R?"  Part="1"
-AR Path="/61619F34/6209AB17/6234DCCA" Ref="R?"  Part="1"
-F 0 "R?" H 10670 4546 50  0000 L CNN
-F 1 "33.2k" H 10670 4455 50  0000 L CNN
-F 2 "" V 10530 4500 50  0001 C CNN
-F 3 "~" H 10600 4500 50  0001 C CNN
-	1    10600 4500
+U 1 1 61F36DB3
+P 10100 4700
+AR Path="/61619F34/6161AC01/61F36DB3" Ref="R?"  Part="1"
+AR Path="/61619F34/61F7AB68/61F36DB3" Ref="R?"  Part="1"
+F 0 "R?" H 10170 4746 50  0000 L CNN
+F 1 "R" H 10170 4655 50  0000 L CNN
+F 2 "" V 10030 4700 50  0001 C CNN
+F 3 "~" H 10100 4700 50  0001 C CNN
+	1    10100 4700
 	1    0    0    -1
 $EndComp
 Wire Wire Line
-	8950 4200 10600 4200
-Wire Wire Line
-	10600 4200 10600 4350
-Text Label 10250 4800 0    50   ~ 0
+	8950 4400 10100 4400
+Wire Wire Line
+	10100 4400 10100 4550
+Text Label 9750 5000 0    50   ~ 0
 V-
-Text Label 10600 4800 0    50   ~ 0
+Text Label 10100 5000 0    50   ~ 0
 V-
 Wire Wire Line
-	10250 4650 10250 4800
-Wire Wire Line
-	10600 4800 10600 4650
-Text HLabel 6700 4500 0    50   Input ~ 0
-VREG
-Text Label 9150 3600 0    50   ~ 0
-C1
-Text Label 9150 3700 0    50   ~ 0
-C2
-Text Label 9150 3800 0    50   ~ 0
-C3
-Text Label 9150 3900 0    50   ~ 0
-C4
-Text Label 9150 4000 0    50   ~ 0
-C5
-Text Label 9150 4100 0    50   ~ 0
-C6
-Wire Wire Line
-	8950 4100 9150 4100
-Wire Wire Line
-	8950 4000 9150 4000
-Wire Wire Line
-	9150 3900 8950 3900
-Wire Wire Line
-	8950 3800 9150 3800
-Wire Wire Line
-	9150 3700 8950 3700
-Wire Wire Line
-	8950 3600 9150 3600
-$Comp
-L Device:D_Schottky D?
-U 1 1 6222295F
-P 9450 4900
-F 0 "D?" V 9404 4980 50  0000 L CNN
-F 1 "D_Schottky" V 9495 4980 50  0000 L CNN
-F 2 "" H 9450 4900 50  0001 C CNN
-F 3 "~" H 9450 4900 50  0001 C CNN
-	1    9450 4900
-	0    1    1    0
-$EndComp
-Text Label 9650 5500 0    50   ~ 0
-C6
-$Comp
-L Device:R R?
-U 1 1 622462AA
-P 9450 5200
-F 0 "R?" H 9520 5246 50  0000 L CNN
-F 1 "R" H 9520 5155 50  0000 L CNN
-F 2 "" V 9380 5200 50  0001 C CNN
-F 3 "~" H 9450 5200 50  0001 C CNN
-	1    9450 5200
-	1    0    0    -1
-$EndComp
-$Comp
-L Device:C C?
-U 1 1 62253C9B
-P 9800 4550
-F 0 "C?" H 9915 4596 50  0000 L CNN
-F 1 "100n" H 9915 4505 50  0000 L CNN
-F 2 "" H 9838 4400 50  0001 C CNN
-F 3 "~" H 9800 4550 50  0001 C CNN
-	1    9800 4550
-	1    0    0    -1
-$EndComp
-Wire Wire Line
-	9800 4400 8950 4400
-Wire Wire Line
-	8950 4500 9450 4500
-Wire Wire Line
-	9450 4500 9450 4700
-Wire Wire Line
-	9800 4700 9450 4700
-Connection ~ 9450 4700
-Wire Wire Line
-	9450 4700 9450 4750
-Wire Wire Line
-	9450 5350 9450 5500
-Wire Wire Line
-	9450 5500 9650 5500
-$Comp
-L Device:R R?
-U 1 1 6234DCCE
-P 10050 3300
-AR Path="/61619F34/6161AC01/6234DCCE" Ref="R?"  Part="1"
-AR Path="/61619F34/61F7AB68/6234DCCE" Ref="R?"  Part="1"
-AR Path="/61619F34/62061D33/6234DCCE" Ref="R?"  Part="1"
-AR Path="/61619F34/6209AB17/6234DCCE" Ref="R?"  Part="1"
-F 0 "R?" H 10120 3346 50  0000 L CNN
-F 1 "1M" H 10120 3255 50  0000 L CNN
-F 2 "" V 9980 3300 50  0001 C CNN
-F 3 "~" H 10050 3300 50  0001 C CNN
-	1    10050 3300
-	1    0    0    -1
-$EndComp
-Text Label 10050 3000 0    50   ~ 0
-VREG
-Wire Wire Line
-	10050 3000 10050 3150
-Wire Wire Line
-	10050 3450 10050 3500
-Wire Wire Line
-	10050 3500 8950 3500
-Text HLabel 10300 3500 2    50   Input ~ 0
-WDT
-Wire Wire Line
-	10300 3500 10050 3500
-Connection ~ 10050 3500
+	9750 4850 9750 5000
+Wire Wire Line
+	10100 5000 10100 4850
 $EndSCHEMATC
