File: REVISION 1/211006_lmu_r0/active_passive_balance.sch (KiCad schematic (older format))
At the start: 30 parts

Commit message: LMU design init
Changed lines of the file:
@@
 $Descr A4 11693 8268
 encoding utf-8
-Sheet 10 30
+Sheet 17 30
 Title ""
 Date ""
@@
 Text Notes 7500 3950 0    50   ~ 0
 Secondary connected to the highest \nand lowest potential of the active \nbalancing interface.
-Text Notes 4450 4950 0    50   ~ 0
+Text Notes 4500 5000 0    50   ~ 0
 Uses a shunt resistor to measure the\n current through the coils\n
-Text Notes 4400 2600 0    50   ~ 0
+Text Notes 4450 2600 0    50   ~ 0
 The coil is configured to act as a 2:1 coil.\nCan move 10A if required.
 Text Notes 1250 4950 0    50   ~ 0

Commit message: Finished schematic, ready for pcb layout
Parts:
- removed C?: OPTIONAL, symbol Device:C
- removed C? (x2): 470, symbol Device:C
- removed C? (x4): 100u, symbol Device:C
- removed C?: 2.2n, symbol Device:C
- removed Q? (x2): SiR882DP, Package_SO:PowerPAK_SO-8_Single, symbol sir882dp:SiR882DP
- removed R?: 3.3k, symbol Device:R
- removed R?: 470, symbol Device:R
- removed R? (x4): 20, symbol Device:R
- removed R? (x2): 25m, symbol Device:R
- removed R?: 5.1, symbol Device:R
- removed T?: 750312504, EP13_SMT_H_8PIN_(750312504), symbol 750312504:750312504
- added C?: OPTIONAL, symbol Device:C
- added C? (x2): 470, symbol Device:C
- added C? (x4): 100u, symbol Device:C
- added C?: 2.2n, symbol Device:C
- added Q? (x2): SiR882DP, Package_SO:PowerPAK_SO-8_Single, symbol sir882dp:SiR882DP
- added R?: 3.3k, symbol Device:R
- added R?: 470, symbol Device:R
- added R? (x4): 20, symbol Device:R
- added R? (x2): 25m, symbol Device:R
- added R?: 5.1, symbol Device:R
- added T?: 750312504, EP13_SMT_H_8PIN_(750312504), symbol 750312504:750312504
Connections:
- net BOOST: now also C?.2, C?.2, R?.2, T?.5
- net C_FILTERED_N: now also C?.2
- net C_N: now also C?.2, C?.2, R?.2, T?.1, T?.2
- net C_N-1: now also C?.1, C?.1, C?.1, R?.2
- net GND: now also C?.1
- net PG_N: now also R?.2
- net PI_N: now also C?.2, R?.1
- net SI_N: now also R?.1
- net SN: now also R?.2
- net V-: now also C?.1, C?.1, R?.2
- net at Q?.1 (G): now also R?.1
- net at Q?.3 (D), R?.2: now also R?.2
- net at D?.2 (A): now also R?.1
- net at R?.1: now also Q?.4 (G)
- new net: C?.1, Q?.5 (D), T?.10, T?.9
- new net: T?.4, T?.6
- new net: C?.1, Q?.5 (D), T?.7
- new net: C?.2, R?.1 (x2)
- new net: Q?.1 (S), Q?.2 (S), Q?.3 (S), R?.1, R?.2 (x2)
- new net: Q?.4 (G), R?.1
