File: REVISION 1/211006_lmu_r0/file615D6D62.sch (KiCad schematic (older format))
At the start: 23 parts

Commit message: LMU design init
Connections:
- net 3.3V_ISO is gone; now on net +3V3: TP?.1
Changed lines of the file:
@@
 Wire Wire Line
 	4650 2350 4250 2350
-$Comp
-L power:GND #PWR?
-U 1 1 61655B4F
-P 9350 2850
-F 0 "#PWR?" H 9350 2600 50  0001 C CNN
-F 1 "GND" H 9355 2677 50  0000 C CNN
-F 2 "" H 9350 2850 50  0001 C CNN
-F 3 "" H 9350 2850 50  0001 C CNN
-	1    9350 2850
-	1    0    0    -1
-$EndComp
 Wire Wire Line
 	9000 2750 9350 2750
 Wire Wire Line
 	9350 2750 9350 2850
-$Comp
-L power:+3.3V #PWR?
-U 1 1 61656186
-P 9350 2350
-F 0 "#PWR?" H 9350 2200 50  0001 C CNN
-F 1 "+3.3V" H 9365 2523 50  0000 C CNN
-F 2 "" H 9350 2350 50  0001 C CNN
-F 3 "" H 9350 2350 50  0001 C CNN
-	1    9350 2350
-	1    0    0    -1
-$EndComp
 Wire Wire Line
 	9350 2350 9000 2350
@@
 Wire Wire Line
 	9350 2350 9350 2400
-Connection ~ 9350 2350
 Wire Wire Line
 	9350 2700 9350 2750
@@
 $EndComp
 $Comp
-L power:GND #PWR?
-U 1 1 61670B84
-P 9050 4100
-F 0 "#PWR?" H 9050 3850 50  0001 C CNN
-F 1 "GND" H 9055 3927 50  0000 C CNN
-F 2 "" H 9050 4100 50  0001 C CNN
-F 3 "" H 9050 4100 50  0001 C CNN
-	1    9050 4100
-	1    0    0    -1
-$EndComp
-$Comp
 L Device:R R?
 U 1 1 616744A4
@@
 Wire Wire Line
 	9700 2750 9350 2750
-Wire Wire Line
-	9400 2350 9700 2350
 $Comp
 L power:+5V #PWR?
@@
 	10100 2350 9700 2350
 Connection ~ 9700 2350
+$Comp
+L +3v3_iso:+3V3_ISO #PWR?
+U 1 1 616407F5
+P 9350 2350
+F 0 "#PWR?" H 9350 2200 50  0001 C CNN
+F 1 "+3V3_ISO" H 9365 2523 50  0000 C CNN
+F 2 "" H 9350 2350 50  0001 C CNN
+F 3 "" H 9350 2350 50  0001 C CNN
+	1    9350 2350
+	1    0    0    -1
+$EndComp
+Connection ~ 9350 2350
+Wire Wire Line
+	9350 2350 9700 2350
+$Comp
+L gnd_iso:GND_ISO #PWR?
+U 1 1 61642E17
+P 9350 2850
+F 0 "#PWR?" H 9350 2600 50  0001 C CNN
+F 1 "GND_ISO" H 9355 2677 50  0000 C CNN
+F 2 "" H 9350 2850 50  0001 C CNN
+F 3 "" H 9350 2850 50  0001 C CNN
+	1    9350 2850
+	1    0    0    -1
+$EndComp
+$Comp
+L gnd_iso:GND_ISO #PWR?
+U 1 1 616436D0
+P 9050 4100
+F 0 "#PWR?" H 9050 3850 50  0001 C CNN
+F 1 "GND_ISO" H 9055 3927 50  0000 C CNN
+F 2 "" H 9050 4100 50  0001 C CNN
+F 3 "" H 9050 4100 50  0001 C CNN
+	1    9050 4100
+	1    0    0    -1
+$EndComp
 $EndSCHEMATC
