File: REVISION 1/211006_lmu_r0/file61619F33.sch (KiCad schematic (older format))
At the start: 1 part

Commit message: LMU design init
Parts:
- added C? (x5): C, symbol Device:C
- added F? (x13): Fuse, symbol Device:Fuse
- added J? (x2): Conn_01x03, symbol Connector_Generic:Conn_01x03
- added J?: Conn_01x02, symbol Connector_Generic:Conn_01x02
- added Q?: CZT5551, Package_TO_SOT_SMD:SOT-223-3_TabPin2, symbol czt5551:CZT5551
- added R? (x13): R, symbol Device:R
Connections:
- net TAP0: now also F?.1
- net TAP1: now also F?.1
- net TAP10: now also F?.1
- net TAP11: now also F?.1
- net TAP12: now also F?.1
- net TAP2: now also F?.1
- net TAP3: now also F?.1
- net TAP4: now also F?.1
- net TAP5: now also F?.1
- net TAP6: now also F?.1
- net TAP7: now also F?.1
- net TAP8: now also F?.1
- net TAP9: now also F?.1
- net V+: now reaches U?.1 (V+)
- net V+: now also F?.2, R?.1, R?.2
- net GND: now reaches U?.30 (V-), U?.31 (V-)
- net GND: now also C?.1, C?.2, C?.2, C?.2, C?.2, F?.2, J?.1 (Pin_1), J?.1 (Pin_1), R?.1, R?.2, R?.2, R?.2, R?.2
- net V_TEMP_SENSOR_REF: now reaches U?.34 (VREF2)
- net V_TEMP_SENSOR_REF: now also C?.1
- net at U?.35 (VREF1): now also C?.1
- net DTEN: now reaches U?.36 (DTEN)
- net DTEN: now also J?.2 (Pin_2)
- net VREG: now reaches U?.37 (VREG)
- net VREG: now also C?.1, J?.3 (Pin_3), J?.3 (Pin_3), Q?.3 (E), R?.1, R?.1, R?.1, R?.1, R?.1
- net DRIVE: now reaches U?.38 (DRIVE)
- net DRIVE: now also Q?.1 (B)
- net at U?.39 (WDT): now also R?.2
- net ISOMD: now reaches U?.40 (ISOMD)
- net ISOMD: now also J?.2 (Pin_2)
- net CS: now reaches U?.41 (CSB/IMA)
- net CS: now also J?.1 (Pin_1)
- net SCK: now reaches U?.42 (SCK/IPA)
- net SCK: now also J?.2 (Pin_2)
- net SDI: now reaches U?.43 (SDI/ICMP)
- net SDI: now also R?.1, R?.2
- net SDO: now reaches U?.44 (SDO/IBIAS)
- net SDO: now also R?.2
- net A0: now reaches U?.45 (A0)
- net A0: now also R?.1, R?.2
- net A1: now reaches U?.46 (A1)
- net A1: now also R?.1, R?.2
- net A2: now reaches U?.47 (A2)
- net A2: now also R?.1, R?.2
- net A3: now reaches U?.48 (A3)
- net A3: now also R?.1, R?.2
- new net: C?.1, R?.1
- new net: C?.2, Q?.2 (C), R?.2
- new net Lower Active Balance Group/ACTIVE_TAP1: F?.2
- new net Lower Active Balance Group/ACTIVE_TAP2: F?.2
- new net Lower Active Balance Group/ACTIVE_TAP3: F?.2
- new net Lower Active Balance Group/ACTIVE_TAP4: F?.2
- new net Lower Active Balance Group/ACTIVE_TAP5: F?.2
- new net Lower Active Balance Group/ACTIVE_TAP6: F?.2
- new net Upper Active Balance Group/ACTIVE_TAP1: F?.2
- new net Upper Active Balance Group/ACTIVE_TAP2: F?.2
- new net Upper Active Balance Group/ACTIVE_TAP3: F?.2
- new net Upper Active Balance Group/ACTIVE_TAP4: F?.2
- new net Upper Active Balance Group/ACTIVE_TAP5: F?.2
Other:
- note added: "DEPOPULATE\nUsed for biasing 2-wire mode"
- note added: "DTEN (Active High) is used to enable the discharge timer on each switch. See D-Sheet for more information."
- note added: "ISOMD Enables the two wire serial communication mode - connected to a seperate isolating transformer."
- note added: "Tap for potential 2 wire \ncommunication mode."

Commit message: Finished schematic, ready for pcb layout
Parts:
- removed R? (x8): R, symbol Device:R
- R?: value R -> 1M
Connections:
- net WDT: now reaches R?.2, U?.39 (WDT)
- net A0 renamed sheet6215FBCF/A0
- net A1 renamed sheet6215FBCF/A1
- net A2 renamed sheet6215FBCF/A2
- net A3 renamed sheet6215FBCF/A3
- net Lower Active Balance Group/ACTIVE_TAP1 renamed sheet6209AAF7/ACTIVE_TAP1
- net Lower Active Balance Group/ACTIVE_TAP2 renamed sheet6209AAF7/ACTIVE_TAP2
- net Lower Active Balance Group/ACTIVE_TAP3 renamed sheet6209AAF7/ACTIVE_TAP3
- net Lower Active Balance Group/ACTIVE_TAP4 renamed sheet6209AAF7/ACTIVE_TAP4
- net Lower Active Balance Group/ACTIVE_TAP5 renamed sheet6209AAF7/ACTIVE_TAP5
- net Lower Active Balance Group/ACTIVE_TAP6 renamed GND_UPPER
Other:
- moved on the sheet: C?, F?, J?, Q?, R?, U?
