File: REVISION 1/211006_lmu_r0/file616BA637.sch (KiCad schematic (older format))
At the start: 20 parts

Commit message: LMU design init
Parts:
- removed C? (x8): C, symbol Device:C
- removed FB?: Ferrite_Bead_Small, symbol Device:Ferrite_Bead_Small
- removed R?: R, symbol Device:R
- removed U?: ADM3053, Package_SO:SOIC-20W_7.5x12.8mm_P1.27mm, symbol Interface_CAN_LIN:ADM3053
- added C? (x2): C, symbol Device:C
- added R?: R, symbol Device:R
- added U?: ISO1042DWVR, SOIC127P1150X280-8N, symbol ISO1042DWVR:ISO1042DWVR
Connections:
- net CAN_RX: now also U?.2 (RXD)
- net CAN_S: now also C?.1, R?.2, U?.5 (GND2)
- net CAN_TX: now also U?.3 (TXD)
- net at C?.1, D?.1 (K), L?.4: now also U?.6 (CANL)
- net at C?.1, D?.2 (K), L?.2: now also U?.7 (CANH)
- new net +3V3: C?.1, U?.1 (VCC1)
- new net +5V: C?.1, U?.8 (VCC2)
- new net GND: C?.2, C?.2, R?.1, U?.4 (GND1)
- no-connect marks 1 -> 0
Other:
- note added: "STPG"
