File: 211006_lmu_r0/Lower Active Balance Group.sch (KiCad schematic (older format))
At the start: 7 parts

Commit message: Updated BOM and footprints for non-hv components
Parts:
- gave numbers to parts that had none: 7
Changed lines of the file:
@@
 AR Path="/61619F34/61F7AB68/619B505D" Ref="U?"  Part="1"
 AR Path="/61619F34/62061D33/619B505D" Ref="U?"  Part="1"
-AR Path="/61619F34/6209AB17/619B505D" Ref="U?"  Part="1"
-F 0 "U?" H 8050 4970 50  0000 C CNN
+AR Path="/61619F34/6209AB17/619B505D" Ref="U5"  Part="1"
+F 0 "U5" H 8050 4970 50  0000 C CNN
 F 1 "LTC3300ILXE-2#PBF" H 8050 4879 50  0000 C CNN
 F 2 "QFP50P900X900X160-49N" H 8050 3400 50  0001 L BNN
@@
 AR Path="/61619F34/61F7AB68/6234DCC9" Ref="R?"  Part="1"
 AR Path="/61619F34/62061D33/6234DCC9" Ref="R?"  Part="1"
-AR Path="/61619F34/6209AB17/6234DCC9" Ref="R?"  Part="1"
-F 0 "R?" H 10320 4546 50  0000 L CNN
+AR Path="/61619F34/6209AB17/6234DCC9" Ref="R105"  Part="1"
+F 0 "R105" H 10320 4546 50  0000 L CNN
 F 1 "23.7k" H 10320 4455 50  0000 L CNN
 F 2 "" V 10180 4500 50  0001 C CNN
@@
 AR Path="/61619F34/61F7AB68/61F36DB3" Ref="R?"  Part="1"
 AR Path="/61619F34/62061D33/61F36DB3" Ref="R?"  Part="1"
-AR Path="/61619F34/6209AB17/61F36DB3" Ref="R?"  Part="1"
-F 0 "R?" H 10670 4546 50  0000 L CNN
+AR Path="/61619F34/6209AB17/61F36DB3" Ref="R106"  Part="1"
+F 0 "R106" H 10670 4546 50  0000 L CNN
 F 1 "33.2k" H 10670 4455 50  0000 L CNN
 F 2 "" V 10530 4500 50  0001 C CNN
@@
 	8950 3600 9150 3600
 $Comp
-L Device:D_Schottky D?
+L Device:D_Schottky D27
 U 1 1 6234DCCB
 P 9450 4900
-F 0 "D?" V 9404 4980 50  0000 L CNN
+F 0 "D27" V 9404 4980 50  0000 L CNN
 F 1 "D_Schottky" V 9495 4980 50  0000 L CNN
 F 2 "" H 9450 4900 50  0001 C CNN
@@
 C6
 $Comp
-L Device:R R?
+L Device:R R103
 U 1 1 6234DCCC
 P 9450 5200
-F 0 "R?" H 9520 5246 50  0000 L CNN
+F 0 "R103" H 9520 5246 50  0000 L CNN
 F 1 "R" H 9520 5155 50  0000 L CNN
 F 2 "" V 9380 5200 50  0001 C CNN
@@
 $EndComp
 $Comp
-L Device:C C?
+L Device:C C103
 U 1 1 6234DCCD
 P 9800 4550
-F 0 "C?" H 9915 4596 50  0000 L CNN
+F 0 "C103" H 9915 4596 50  0000 L CNN
 F 1 "100n" H 9915 4505 50  0000 L CNN
 F 2 "" H 9838 4400 50  0001 C CNN
@@
 AR Path="/61619F34/61F7AB68/6228C6A6" Ref="R?"  Part="1"
 AR Path="/61619F34/62061D33/6228C6A6" Ref="R?"  Part="1"
-AR Path="/61619F34/6209AB17/6228C6A6" Ref="R?"  Part="1"
-F 0 "R?" H 10120 3346 50  0000 L CNN
+AR Path="/61619F34/6209AB17/6228C6A6" Ref="R104"  Part="1"
+F 0 "R104" H 10120 3346 50  0000 L CNN
 F 1 "1M" H 10120 3255 50  0000 L CNN
 F 2 "" V 9980 3300 50  0001 C CNN

Commit message: Cleaned up last components missing footprint refs
Parts:
- C103: footprint (none) -> Capacitor_SMD:C_1206_3216Metric_Pad1.33x1.80mm_HandSolder
- R104, R105, R106: footprint (none) -> Resistor_SMD:R_0603_1608Metric_Pad0.98x0.95mm_HandSolder
Changed lines of the file:
@@
 F 0 "R105" H 10320 4546 50  0000 L CNN
 F 1 "23.7k" H 10320 4455 50  0000 L CNN
-F 2 "" V 10180 4500 50  0001 C CNN
+F 2 "Resistor_SMD:R_0603_1608Metric_Pad0.98x0.95mm_HandSolder" V 10180 4500 50  0001 C CNN
 F 3 "~" H 10250 4500 50  0001 C CNN
 	1    10250 4500
@@
 F 0 "R106" H 10670 4546 50  0000 L CNN
 F 1 "33.2k" H 10670 4455 50  0000 L CNN
-F 2 "" V 10530 4500 50  0001 C CNN
+F 2 "Resistor_SMD:R_0603_1608Metric_Pad0.98x0.95mm_HandSolder" V 10530 4500 50  0001 C CNN
 F 3 "~" H 10600 4500 50  0001 C CNN
 	1    10600 4500
@@
 F 0 "C103" H 9915 4596 50  0000 L CNN
 F 1 "100n" H 9915 4505 50  0000 L CNN
-F 2 "" H 9838 4400 50  0001 C CNN
+F 2 "Capacitor_SMD:C_1206_3216Metric_Pad1.33x1.80mm_HandSolder" H 9838 4400 50  0001 C CNN
 F 3 "~" H 9800 4550 50  0001 C CNN
 	1    9800 4550
@@
 F 0 "R104" H 10120 3346 50  0000 L CNN
 F 1 "1M" H 10120 3255 50  0000 L CNN
-F 2 "" V 9980 3300 50  0001 C CNN
+F 2 "Resistor_SMD:R_0603_1608Metric_Pad0.98x0.95mm_HandSolder" V 9980 3300 50  0001 C CNN
 F 3 "~" H 10050 3300 50  0001 C CNN
 	1    10050 3300

Commit message: Updated with Mouser links for BOM
Parts:
- C103: value 100n -> 100nF
- R103: value R -> 6.81R
- R104: value 1M -> 1MR
- R105: value 23.7k -> 23.7kR
- R106: value 33.2k -> 33.2kR
Changed lines of the file:
@@
 AR Path="/61619F34/6209AB17/6234DCC9" Ref="R105"  Part="1"
 F 0 "R105" H 10320 4546 50  0000 L CNN
-F 1 "23.7k" H 10320 4455 50  0000 L CNN
+F 1 "23.7kR" H 10320 4455 50  0000 L CNN
 F 2 "Resistor_SMD:R_0603_1608Metric_Pad0.98x0.95mm_HandSolder" V 10180 4500 50  0001 C CNN
 F 3 "~" H 10250 4500 50  0001 C CNN
@@
 AR Path="/61619F34/6209AB17/61F36DB3" Ref="R106"  Part="1"
 F 0 "R106" H 10670 4546 50  0000 L CNN
-F 1 "33.2k" H 10670 4455 50  0000 L CNN
+F 1 "33.2kR" H 10670 4455 50  0000 L CNN
 F 2 "Resistor_SMD:R_0603_1608Metric_Pad0.98x0.95mm_HandSolder" V 10530 4500 50  0001 C CNN
 F 3 "~" H 10600 4500 50  0001 C CNN
@@
 P 9450 5200
 F 0 "R103" H 9520 5246 50  0000 L CNN
-F 1 "R" H 9520 5155 50  0000 L CNN
+F 1 "6.81R" H 9520 5155 50  0000 L CNN
 F 2 "" V 9380 5200 50  0001 C CNN
 F 3 "~" H 9450 5200 50  0001 C CNN
@@
 P 9800 4550
 F 0 "C103" H 9915 4596 50  0000 L CNN
-F 1 "100n" H 9915 4505 50  0000 L CNN
+F 1 "100nF" H 9915 4505 50  0000 L CNN
 F 2 "Capacitor_SMD:C_1206_3216Metric_Pad1.33x1.80mm_HandSolder" H 9838 4400 50  0001 C CNN
 F 3 "~" H 9800 4550 50  0001 C CNN
@@
 AR Path="/61619F34/6209AB17/6228C6A6" Ref="R104"  Part="1"
 F 0 "R104" H 10120 3346 50  0000 L CNN
-F 1 "1M" H 10120 3255 50  0000 L CNN
+F 1 "1MR" H 10120 3255 50  0000 L CNN
 F 2 "Resistor_SMD:R_0603_1608Metric_Pad0.98x0.95mm_HandSolder" V 9980 3300 50  0001 C CNN
 F 3 "~" H 10050 3300 50  0001 C CNN
