File: 211006_lmu_r0/Lower Address Selection.sch (KiCad schematic (older format))
At the start: 8 parts

Commit message: Updated BOM and footprints for non-hv components
Parts:
- removed R? (x3): R, symbol Device:R
- added R187, R188, R193: R, symbol Device:R
- gave numbers to parts that had none: 5
Connections:
- net A0: now also R187.2, R188.1
- net A3: now also R193.2
- net GND_REF: now also R188.2
- net VCC_REF: now also R187.1, R193.1
Changed lines of the file:
@@
 $Comp
 L Device:R R?
-U 1 1 61FF994E
+U 1 1 61F42E78
 P 5000 3650
-AR Path="/61619F34/61FF949C/61FF994E" Ref="R?"  Part="1"
-AR Path="/61619F34/620A15AD/61FF994E" Ref="R?"  Part="1"
-AR Path="/61619F34/620DEAEE/61FF994E" Ref="R?"  Part="1"
-AR Path="/61619F34/62127D2E/61FF994E" Ref="R?"  Part="1"
-AR Path="/61619F34/62135562/61FF994E" Ref="R?"  Part="1"
-AR Path="/61619F34/62140E50/61FF994E" Ref="R?"  Part="1"
-AR Path="/61619F34/6215FBD7/61FF994E" Ref="R?"  Part="1"
-F 0 "R?" H 5070 3696 50  0000 L CNN
+AR Path="/61619F34/61FF949C/61F42E78" Ref="R?"  Part="1"
+AR Path="/61619F34/620A15AD/61F42E78" Ref="R?"  Part="1"
+AR Path="/61619F34/620DEAEE/61F42E78" Ref="R?"  Part="1"
+AR Path="/61619F34/62127D2E/61F42E78" Ref="R187"  Part="1"
+AR Path="/61619F34/62135562/61F42E78" Ref="R?"  Part="1"
+AR Path="/61619F34/62140E50/61F42E78" Ref="R?"  Part="1"
+AR Path="/61619F34/6215FBD7/61F42E78" Ref="R?"  Part="1"
+F 0 "R187" H 5070 3696 50  0000 L CNN
 F 1 "R" H 5070 3605 50  0000 L CNN
 F 2 "" V 4930 3650 50  0001 C CNN
@@
 $Comp
 L Device:R R?
-U 1 1 61FFA5B8
+U 1 1 61F42E79
 P 5000 3950
-AR Path="/61619F34/61FF949C/61FFA5B8" Ref="R?"  Part="1"
-AR Path="/61619F34/620A15AD/61FFA5B8" Ref="R?"  Part="1"
-AR Path="/61619F34/620DEAEE/61FFA5B8" Ref="R?"  Part="1"
-AR Path="/61619F34/62127D2E/61FFA5B8" Ref="R?"  Part="1"
-AR Path="/61619F34/62135562/61FFA5B8" Ref="R?"  Part="1"
-AR Path="/61619F34/62140E50/61FFA5B8" Ref="R?"  Part="1"
-AR Path="/61619F34/6215FBD7/61FFA5B8" Ref="R?"  Part="1"
-F 0 "R?" H 5070 3996 50  0000 L CNN
+AR Path="/61619F34/61FF949C/61F42E79" Ref="R?"  Part="1"
+AR Path="/61619F34/620A15AD/61F42E79" Ref="R?"  Part="1"
+AR Path="/61619F34/620DEAEE/61F42E79" Ref="R?"  Part="1"
+AR Path="/61619F34/62127D2E/61F42E79" Ref="R188"  Part="1"
+AR Path="/61619F34/62135562/61F42E79" Ref="R?"  Part="1"
+AR Path="/61619F34/62140E50/61F42E79" Ref="R?"  Part="1"
+AR Path="/61619F34/6215FBD7/61F42E79" Ref="R?"  Part="1"
+F 0 "R188" H 5070 3996 50  0000 L CNN
 F 1 "R" H 5070 3905 50  0000 L CNN
 F 2 "" V 4930 3950 50  0001 C CNN
@@
 AR Path="/61619F34/620A15AD/6234DD81" Ref="R?"  Part="1"
 AR Path="/61619F34/620DEAEE/6234DD81" Ref="R?"  Part="1"
-AR Path="/61619F34/62127D2E/6234DD81" Ref="R?"  Part="1"
+AR Path="/61619F34/62127D2E/6234DD81" Ref="R189"  Part="1"
 AR Path="/61619F34/62135562/6234DD81" Ref="R?"  Part="1"
 AR Path="/61619F34/62140E50/6234DD81" Ref="R?"  Part="1"
 AR Path="/61619F34/6215FBD7/6234DD81" Ref="R?"  Part="1"
-F 0 "R?" H 5420 3696 50  0000 L CNN
+F 0 "R189" H 5420 3696 50  0000 L CNN
 F 1 "R" H 5420 3605 50  0000 L CNN
 F 2 "" V 5280 3650 50  0001 C CNN
@@
 AR Path="/61619F34/620A15AD/6234DD82" Ref="R?"  Part="1"
 AR Path="/61619F34/620DEAEE/6234DD82" Ref="R?"  Part="1"
-AR Path="/61619F34/62127D2E/6234DD82" Ref="R?"  Part="1"
+AR Path="/61619F34/62127D2E/6234DD82" Ref="R190"  Part="1"
 AR Path="/61619F34/62135562/6234DD82" Ref="R?"  Part="1"
 AR Path="/61619F34/62140E50/6234DD82" Ref="R?"  Part="1"
 AR Path="/61619F34/6215FBD7/6234DD82" Ref="R?"  Part="1"
-F 0 "R?" H 5420 3996 50  0000 L CNN
+F 0 "R190" H 5420 3996 50  0000 L CNN
 F 1 "R" H 5420 3905 50  0000 L CNN
 F 2 "" V 5280 3950 50  0001 C CNN
@@
 AR Path="/61619F34/620A15AD/61FFB654" Ref="R?"  Part="1"
 AR Path="/61619F34/620DEAEE/61FFB654" Ref="R?"  Part="1"
-AR Path="/61619F34/62127D2E/61FFB654" Ref="R?"  Part="1"
+AR Path="/61619F34/62127D2E/61FFB654" Ref="R191"  Part="1"
 AR Path="/61619F34/62135562/61FFB654" Ref="R?"  Part="1"
 AR Path="/61619F34/62140E50/61FFB654" Ref="R?"  Part="1"
 AR Path="/61619F34/6215FBD7/61FFB654" Ref="R?"  Part="1"
-F 0 "R?" H 5720 3696 50  0000 L CNN
+F 0 "R191" H 5720 3696 50  0000 L CNN
 F 1 "R" H 5720 3605 50  0000 L CNN
 F 2 "" V 5580 3650 50  0001 C CNN
@@
 AR Path="/61619F34/620A15AD/61FFB65A" Ref="R?"  Part="1"
 AR Path="/61619F34/620DEAEE/61FFB65A" Ref="R?"  Part="1"
-AR Path="/61619F34/62127D2E/61FFB65A" Ref="R?"  Part="1"
+AR Path="/61619F34/62127D2E/61FFB65A" Ref="R192"  Part="1"
 AR Path="/61619F34/62135562/61FFB65A" Ref="R?"  Part="1"
 AR Path="/61619F34/62140E50/61FFB65A" Ref="R?"  Part="1"
 AR Path="/61619F34/6215FBD7/61FFB65A" Ref="R?"  Part="1"
-F 0 "R?" H 5720 3996 50  0000 L CNN
+F 0 "R192" H 5720 3996 50  0000 L CNN
 F 1 "R" H 5720 3905 50  0000 L CNN
 F 2 "" V 5580 3950 50  0001 C CNN
@@
 $Comp
 L Device:R R?
-U 1 1 61FFBB96
+U 1 1 61F42E7C
 P 5950 3650
-AR Path="/61619F34/61FF949C/61FFBB96" Ref="R?"  Part="1"
-AR Path="/61619F34/620A15AD/61FFBB96" Ref="R?"  Part="1"
-AR Path="/61619F34/620DEAEE/61FFBB96" Ref="R?"  Part="1"
-AR Path="/61619F34/62127D2E/61FFBB96" Ref="R?"  Part="1"
-AR Path="/61619F34/62135562/61FFBB96" Ref="R?"  Part="1"
-AR Path="/61619F34/62140E50/61FFBB96" Ref="R?"  Part="1"
-AR Path="/61619F34/6215FBD7/61FFBB96" Ref="R?"  Part="1"
-F 0 "R?" H 6020 3696 50  0000 L CNN
+AR Path="/61619F34/61FF949C/61F42E7C" Ref="R?"  Part="1"
+AR Path="/61619F34/620A15AD/61F42E7C" Ref="R?"  Part="1"
+AR Path="/61619F34/620DEAEE/61F42E7C" Ref="R?"  Part="1"
+AR Path="/61619F34/62127D2E/61F42E7C" Ref="R193"  Part="1"
+AR Path="/61619F34/62135562/61F42E7C" Ref="R?"  Part="1"
+AR Path="/61619F34/62140E50/61F42E7C" Ref="R?"  Part="1"
+AR Path="/61619F34/6215FBD7/61F42E7C" Ref="R?"  Part="1"
+F 0 "R193" H 6020 3696 50  0000 L CNN
 F 1 "R" H 6020 3605 50  0000 L CNN
 F 2 "" V 5880 3650 50  0001 C CNN
@@
 AR Path="/61619F34/620A15AD/61FFBB9C" Ref="R?"  Part="1"
 AR Path="/61619F34/620DEAEE/61FFBB9C" Ref="R?"  Part="1"
-AR Path="/61619F34/62127D2E/61FFBB9C" Ref="R?"  Part="1"
+AR Path="/61619F34/62127D2E/61FFBB9C" Ref="R194"  Part="1"
 AR Path="/61619F34/62135562/61FFBB9C" Ref="R?"  Part="1"
 AR Path="/61619F34/62140E50/61FFBB9C" Ref="R?"  Part="1"
 AR Path="/61619F34/6215FBD7/61FFBB9C" Ref="R?"  Part="1"
-F 0 "R?" H 6020 3996 50  0000 L CNN
+F 0 "R194" H 6020 3996 50  0000 L CNN
 F 1 "R" H 6020 3905 50  0000 L CNN
 F 2 "" V 5880 3950 50  0001 C CNN

Commit message: Added most footprint requirements in HV
Parts:
- R187, R188, R189, R190, R191, R192, R193, R194: value R -> 50k; footprint (none) -> Resistor_SMD:R_0603_1608Metric_Pad0.98x0.95mm_HandSolder
Connections:
- net A0: now also R188.2; no longer R188.1
- net A1: now also R190.2; no longer R190.1
- net A2: now also R192.2; no longer R192.1
- net A3: now also R194.2; no longer R194.1
- net GND_REF: now also R188.1, R190.1, R192.1, R194.1; no longer R188.2, R190.2, R192.2, R194.2

Commit message: Updated with Mouser links for BOM
Parts:
- R111: renamed from R187; value 50k -> 50kR
- R112: renamed from R188; value 50k -> 50kR
- R113: renamed from R189; value 50k -> 50kR
- R114: renamed from R190; value 50k -> 50kR
- R115: renamed from R191; value 50k -> 50kR
- R116: renamed from R192; value 50k -> 50kR
- R117: renamed from R193; value 50k -> 50kR
- R118: renamed from R194; value 50k -> 50kR
Changed lines of the file:
@@
 AR Path="/61619F34/620A15AD/61F42E78" Ref="R?"  Part="1"
 AR Path="/61619F34/620DEAEE/61F42E78" Ref="R?"  Part="1"
-AR Path="/61619F34/62127D2E/61F42E78" Ref="R187"  Part="1"
+AR Path="/61619F34/62127D2E/61F42E78" Ref="R111"  Part="1"
 AR Path="/61619F34/62135562/61F42E78" Ref="R?"  Part="1"
 AR Path="/61619F34/62140E50/61F42E78" Ref="R?"  Part="1"
 AR Path="/61619F34/6215FBD7/61F42E78" Ref="R?"  Part="1"
-F 0 "R187" H 4950 3950 50  0000 L CNN
-F 1 "50k" H 4950 3850 50  0000 L CNN
+F 0 "R111" H 4950 3950 50  0000 L CNN
+F 1 "50kR" H 4950 3850 50  0000 L CNN
 F 2 "Resistor_SMD:R_0603_1608Metric_Pad0.98x0.95mm_HandSolder" V 4930 3650 50  0001 C CNN
 F 3 "~" H 5000 3650 50  0001 C CNN
@@
 AR Path="/61619F34/620A15AD/621350AF" Ref="R?"  Part="1"
 AR Path="/61619F34/620DEAEE/621350AF" Ref="R?"  Part="1"
-AR Path="/61619F34/62127D2E/621350AF" Ref="R189"  Part="1"
+AR Path="/61619F34/62127D2E/621350AF" Ref="R113"  Part="1"
 AR Path="/61619F34/62135562/621350AF" Ref="R?"  Part="1"
 AR Path="/61619F34/62140E50/621350AF" Ref="R?"  Part="1"
 AR Path="/61619F34/6215FBD7/621350AF" Ref="R?"  Part="1"
-F 0 "R189" H 5300 3950 50  0000 L CNN
-F 1 "50k" H 5300 3850 50  0000 L CNN
+F 0 "R113" H 5300 3950 50  0000 L CNN
+F 1 "50kR" H 5300 3850 50  0000 L CNN
 F 2 "Resistor_SMD:R_0603_1608Metric_Pad0.98x0.95mm_HandSolder" V 5280 3650 50  0001 C CNN
 F 3 "~" H 5350 3650 50  0001 C CNN
@@
 AR Path="/61619F34/620A15AD/62135560" Ref="R?"  Part="1"
 AR Path="/61619F34/620DEAEE/62135560" Ref="R?"  Part="1"
-AR Path="/61619F34/62127D2E/62135560" Ref="R191"  Part="1"
+AR Path="/61619F34/62127D2E/62135560" Ref="R115"  Part="1"
 AR Path="/61619F34/62135562/62135560" Ref="R?"  Part="1"
 AR Path="/61619F34/62140E50/62135560" Ref="R?"  Part="1"
 AR Path="/61619F34/6215FBD7/62135560" Ref="R?"  Part="1"
-F 0 "R191" H 5600 3950 50  0000 L CNN
-F 1 "50k" H 5600 3850 50  0000 L CNN
+F 0 "R115" H 5600 3950 50  0000 L CNN
+F 1 "50kR" H 5600 3850 50  0000 L CNN
 F 2 "Resistor_SMD:R_0603_1608Metric_Pad0.98x0.95mm_HandSolder" V 5580 3650 50  0001 C CNN
 F 3 "~" H 5650 3650 50  0001 C CNN
@@
 AR Path="/61619F34/620A15AD/62135A9A" Ref="R?"  Part="1"
 AR Path="/61619F34/620DEAEE/62135A9A" Ref="R?"  Part="1"
-AR Path="/61619F34/62127D2E/62135A9A" Ref="R193"  Part="1"
+AR Path="/61619F34/62127D2E/62135A9A" Ref="R117"  Part="1"
 AR Path="/61619F34/62135562/62135A9A" Ref="R?"  Part="1"
 AR Path="/61619F34/62140E50/62135A9A" Ref="R?"  Part="1"
 AR Path="/61619F34/6215FBD7/62135A9A" Ref="R?"  Part="1"
-F 0 "R193" H 5900 3950 50  0000 L CNN
-F 1 "50k" H 5900 3850 50  0000 L CNN
+F 0 "R117" H 5900 3950 50  0000 L CNN
+F 1 "50kR" H 5900 3850 50  0000 L CNN
 F 2 "Resistor_SMD:R_0603_1608Metric_Pad0.98x0.95mm_HandSolder" V 5880 3650 50  0001 C CNN
 F 3 "~" H 5950 3650 50  0001 C CNN
@@
 AR Path="/61619F34/620A15AD/62135D35" Ref="R?"  Part="1"
 AR Path="/61619F34/620DEAEE/62135D35" Ref="R?"  Part="1"
-AR Path="/61619F34/62127D2E/62135D35" Ref="R188"  Part="1"
+AR Path="/61619F34/62127D2E/62135D35" Ref="R112"  Part="1"
 AR Path="/61619F34/62135562/62135D35" Ref="R?"  Part="1"
 AR Path="/61619F34/62140E50/62135D35" Ref="R?"  Part="1"
 AR Path="/61619F34/6215FBD7/62135D35" Ref="R?"  Part="1"
-F 0 "R188" H 4950 4250 50  0000 L CNN
-F 1 "50k" H 4950 4150 50  0000 L CNN
+F 0 "R112" H 4950 4250 50  0000 L CNN
+F 1 "50kR" H 4950 4150 50  0000 L CNN
 F 2 "Resistor_SMD:R_0603_1608Metric_Pad0.98x0.95mm_HandSolder" V 4930 3950 50  0001 C CNN
 F 3 "~" H 5000 3950 50  0001 C CNN
@@
 AR Path="/61619F34/620A15AD/62136854" Ref="R?"  Part="1"
 AR Path="/61619F34/620DEAEE/62136854" Ref="R?"  Part="1"
-AR Path="/61619F34/62127D2E/62136854" Ref="R190"  Part="1"
+AR Path="/61619F34/62127D2E/62136854" Ref="R114"  Part="1"
 AR Path="/61619F34/62135562/62136854" Ref="R?"  Part="1"
 AR Path="/61619F34/62140E50/62136854" Ref="R?"  Part="1"
 AR Path="/61619F34/6215FBD7/62136854" Ref="R?"  Part="1"
-F 0 "R190" H 5300 4250 50  0000 L CNN
-F 1 "50k" H 5300 4150 50  0000 L CNN
+F 0 "R114" H 5300 4250 50  0000 L CNN
+F 1 "50kR" H 5300 4150 50  0000 L CNN
 F 2 "Resistor_SMD:R_0603_1608Metric_Pad0.98x0.95mm_HandSolder" V 5280 3950 50  0001 C CNN
 F 3 "~" H 5350 3950 50  0001 C CNN
@@
 AR Path="/61619F34/620A15AD/62136BCC" Ref="R?"  Part="1"
 AR Path="/61619F34/620DEAEE/62136BCC" Ref="R?"  Part="1"
-AR Path="/61619F34/62127D2E/62136BCC" Ref="R192"  Part="1"
+AR Path="/61619F34/62127D2E/62136BCC" Ref="R116"  Part="1"
 AR Path="/61619F34/62135562/62136BCC" Ref="R?"  Part="1"
 AR Path="/61619F34/62140E50/62136BCC" Ref="R?"  Part="1"
 AR Path="/61619F34/6215FBD7/62136BCC" Ref="R?"  Part="1"
-F 0 "R192" H 5600 4250 50  0000 L CNN
-F 1 "50k" H 5600 4150 50  0000 L CNN
+F 0 "R116" H 5600 4250 50  0000 L CNN
+F 1 "50kR" H 5600 4150 50  0000 L CNN
 F 2 "Resistor_SMD:R_0603_1608Metric_Pad0.98x0.95mm_HandSolder" V 5580 3950 50  0001 C CNN
 F 3 "~" H 5650 3950 50  0001 C CNN
@@
 AR Path="/61619F34/620A15AD/62136E89" Ref="R?"  Part="1"
 AR Path="/61619F34/620DEAEE/62136E89" Ref="R?"  Part="1"
-AR Path="/61619F34/62127D2E/62136E89" Ref="R194"  Part="1"
+AR Path="/61619F34/62127D2E/62136E89" Ref="R118"  Part="1"
 AR Path="/61619F34/62135562/62136E89" Ref="R?"  Part="1"
 AR Path="/61619F34/62140E50/62136E89" Ref="R?"  Part="1"
 AR Path="/61619F34/6215FBD7/62136E89" Ref="R?"  Part="1"
-F 0 "R194" H 5900 4250 50  0000 L CNN
-F 1 "50k" H 5900 4150 50  0000 L CNN
+F 0 "R118" H 5900 4250 50  0000 L CNN
+F 1 "50kR" H 5900 4150 50  0000 L CNN
 F 2 "Resistor_SMD:R_0603_1608Metric_Pad0.98x0.95mm_HandSolder" V 5880 3950 50  0001 C CNN
 F 3 "~" H 5950 3950 50  0001 C CNN
