File: 211006_lmu_r0/Upper Address Selection.sch (KiCad schematic (older format))
At the start: 8 parts

Commit message: Updated BOM and footprints for non-hv components
Parts:
- gave numbers to parts that had none: 8
Changed lines of the file:
@@
 $EndDescr
 $Comp
-L Device:R R?
+L Device:R R179
 U 1 1 6234DD24
 P 5000 3650
-AR Path="/61619F34/61FF949C/6234DD24" Ref="R?"  Part="1"
+AR Path="/61619F34/61FF949C/6234DD24" Ref="R179"  Part="1"
 AR Path="/61619F34/620A15AD/6234DD24" Ref="R?"  Part="1"
 AR Path="/61619F34/620DEAEE/6234DD24" Ref="R?"  Part="1"
@@
 AR Path="/61619F34/62140E50/6234DD24" Ref="R?"  Part="1"
 AR Path="/61619F34/6215FBD7/6234DD24" Ref="R?"  Part="1"
-F 0 "R?" H 5070 3696 50  0000 L CNN
+F 0 "R179" H 5070 3696 50  0000 L CNN
 F 1 "R" H 5070 3605 50  0000 L CNN
 F 2 "" V 4930 3650 50  0001 C CNN
@@
 $EndComp
 $Comp
-L Device:R R?
+L Device:R R180
 U 1 1 6234DD25
 P 5000 3950
-AR Path="/61619F34/61FF949C/6234DD25" Ref="R?"  Part="1"
+AR Path="/61619F34/61FF949C/6234DD25" Ref="R180"  Part="1"
 AR Path="/61619F34/620A15AD/6234DD25" Ref="R?"  Part="1"
 AR Path="/61619F34/620DEAEE/6234DD25" Ref="R?"  Part="1"
@@
 AR Path="/61619F34/62140E50/6234DD25" Ref="R?"  Part="1"
 AR Path="/61619F34/6215FBD7/6234DD25" Ref="R?"  Part="1"
-F 0 "R?" H 5070 3996 50  0000 L CNN
+F 0 "R180" H 5070 3996 50  0000 L CNN
 F 1 "R" H 5070 3905 50  0000 L CNN
 F 2 "" V 4930 3950 50  0001 C CNN
@@
 $EndComp
 $Comp
-L Device:R R?
+L Device:R R181
 U 1 1 61FFAD0C
 P 5350 3650
-AR Path="/61619F34/61FF949C/61FFAD0C" Ref="R?"  Part="1"
+AR Path="/61619F34/61FF949C/61FFAD0C" Ref="R181"  Part="1"
 AR Path="/61619F34/620A15AD/61FFAD0C" Ref="R?"  Part="1"
 AR Path="/61619F34/620DEAEE/61FFAD0C" Ref="R?"  Part="1"
@@
 AR Path="/61619F34/62140E50/61FFAD0C" Ref="R?"  Part="1"
 AR Path="/61619F34/6215FBD7/61FFAD0C" Ref="R?"  Part="1"
-F 0 "R?" H 5420 3696 50  0000 L CNN
+F 0 "R181" H 5420 3696 50  0000 L CNN
 F 1 "R" H 5420 3605 50  0000 L CNN
 F 2 "" V 5280 3650 50  0001 C CNN
@@
 $EndComp
 $Comp
-L Device:R R?
+L Device:R R182
 U 1 1 61FFAD12
 P 5350 3950
-AR Path="/61619F34/61FF949C/61FFAD12" Ref="R?"  Part="1"
+AR Path="/61619F34/61FF949C/61FFAD12" Ref="R182"  Part="1"
 AR Path="/61619F34/620A15AD/61FFAD12" Ref="R?"  Part="1"
 AR Path="/61619F34/620DEAEE/61FFAD12" Ref="R?"  Part="1"
@@
 AR Path="/61619F34/62140E50/61FFAD12" Ref="R?"  Part="1"
 AR Path="/61619F34/6215FBD7/61FFAD12" Ref="R?"  Part="1"
-F 0 "R?" H 5420 3996 50  0000 L CNN
+F 0 "R182" H 5420 3996 50  0000 L CNN
 F 1 "R" H 5420 3905 50  0000 L CNN
 F 2 "" V 5280 3950 50  0001 C CNN
@@
 $EndComp
 $Comp
-L Device:R R?
+L Device:R R183
 U 1 1 6234DD28
 P 5650 3650
-AR Path="/61619F34/61FF949C/6234DD28" Ref="R?"  Part="1"
+AR Path="/61619F34/61FF949C/6234DD28" Ref="R183"  Part="1"
 AR Path="/61619F34/620A15AD/6234DD28" Ref="R?"  Part="1"
 AR Path="/61619F34/620DEAEE/6234DD28" Ref="R?"  Part="1"
@@
 AR Path="/61619F34/62140E50/6234DD28" Ref="R?"  Part="1"
 AR Path="/61619F34/6215FBD7/6234DD28" Ref="R?"  Part="1"
-F 0 "R?" H 5720 3696 50  0000 L CNN
+F 0 "R183" H 5720 3696 50  0000 L CNN
 F 1 "R" H 5720 3605 50  0000 L CNN
 F 2 "" V 5580 3650 50  0001 C CNN
@@
 $EndComp
 $Comp
-L Device:R R?
+L Device:R R184
 U 1 1 6234DD29
 P 5650 3950
-AR Path="/61619F34/61FF949C/6234DD29" Ref="R?"  Part="1"
+AR Path="/61619F34/61FF949C/6234DD29" Ref="R184"  Part="1"
 AR Path="/61619F34/620A15AD/6234DD29" Ref="R?"  Part="1"
 AR Path="/61619F34/620DEAEE/6234DD29" Ref="R?"  Part="1"
@@
 AR Path="/61619F34/62140E50/6234DD29" Ref="R?"  Part="1"
 AR Path="/61619F34/6215FBD7/6234DD29" Ref="R?"  Part="1"
-F 0 "R?" H 5720 3996 50  0000 L CNN
+F 0 "R184" H 5720 3996 50  0000 L CNN
 F 1 "R" H 5720 3905 50  0000 L CNN
 F 2 "" V 5580 3950 50  0001 C CNN
@@
 $EndComp
 $Comp
-L Device:R R?
+L Device:R R185
 U 1 1 6234DD2A
 P 5950 3650
-AR Path="/61619F34/61FF949C/6234DD2A" Ref="R?"  Part="1"
+AR Path="/61619F34/61FF949C/6234DD2A" Ref="R185"  Part="1"
 AR Path="/61619F34/620A15AD/6234DD2A" Ref="R?"  Part="1"
 AR Path="/61619F34/620DEAEE/6234DD2A" Ref="R?"  Part="1"
@@
 AR Path="/61619F34/62140E50/6234DD2A" Ref="R?"  Part="1"
 AR Path="/61619F34/6215FBD7/6234DD2A" Ref="R?"  Part="1"
-F 0 "R?" H 6020 3696 50  0000 L CNN
+F 0 "R185" H 6020 3696 50  0000 L CNN
 F 1 "R" H 6020 3605 50  0000 L CNN
 F 2 "" V 5880 3650 50  0001 C CNN
@@
 $EndComp
 $Comp
-L Device:R R?
+L Device:R R186
 U 1 1 6234DD2B
 P 5950 3950
-AR Path="/61619F34/61FF949C/6234DD2B" Ref="R?"  Part="1"
+AR Path="/61619F34/61FF949C/6234DD2B" Ref="R186"  Part="1"
 AR Path="/61619F34/620A15AD/6234DD2B" Ref="R?"  Part="1"
 AR Path="/61619F34/620DEAEE/6234DD2B" Ref="R?"  Part="1"
@@
 AR Path="/61619F34/62140E50/6234DD2B" Ref="R?"  Part="1"
 AR Path="/61619F34/6215FBD7/6234DD2B" Ref="R?"  Part="1"
-F 0 "R?" H 6020 3996 50  0000 L CNN
+F 0 "R186" H 6020 3996 50  0000 L CNN
 F 1 "R" H 6020 3905 50  0000 L CNN
 F 2 "" V 5880 3950 50  0001 C CNN

Commit message: Cleaned up last components missing footprint refs
Parts:
- R179, R180, R181, R182, R183, R184, R185, R186: footprint (none) -> Resistor_SMD:R_0603_1608Metric_Pad0.98x0.95mm_HandSolder
Changed lines of the file:
@@
 $Descr A4 11693 8268
 encoding utf-8
-Sheet 30 35
+Sheet 28 35
 Title ""
 Date ""
@@
 F 0 "R179" H 5070 3696 50  0000 L CNN
 F 1 "R" H 5070 3605 50  0000 L CNN
-F 2 "" V 4930 3650 50  0001 C CNN
+F 2 "Resistor_SMD:R_0603_1608Metric_Pad0.98x0.95mm_HandSolder" V 4930 3650 50  0001 C CNN
 F 3 "~" H 5000 3650 50  0001 C CNN
 	1    5000 3650
@@
 F 0 "R180" H 5070 3996 50  0000 L CNN
 F 1 "R" H 5070 3905 50  0000 L CNN
-F 2 "" V 4930 3950 50  0001 C CNN
+F 2 "Resistor_SMD:R_0603_1608Metric_Pad0.98x0.95mm_HandSolder" V 4930 3950 50  0001 C CNN
 F 3 "~" H 5000 3950 50  0001 C CNN
 	1    5000 3950
@@
 F 0 "R181" H 5420 3696 50  0000 L CNN
 F 1 "R" H 5420 3605 50  0000 L CNN
-F 2 "" V 5280 3650 50  0001 C CNN
+F 2 "Resistor_SMD:R_0603_1608Metric_Pad0.98x0.95mm_HandSolder" V 5280 3650 50  0001 C CNN
 F 3 "~" H 5350 3650 50  0001 C CNN
 	1    5350 3650
@@
 F 0 "R182" H 5420 3996 50  0000 L CNN
 F 1 "R" H 5420 3905 50  0000 L CNN
-F 2 "" V 5280 3950 50  0001 C CNN
+F 2 "Resistor_SMD:R_0603_1608Metric_Pad0.98x0.95mm_HandSolder" V 5280 3950 50  0001 C CNN
 F 3 "~" H 5350 3950 50  0001 C CNN
 	1    5350 3950
@@
 F 0 "R183" H 5720 3696 50  0000 L CNN
 F 1 "R" H 5720 3605 50  0000 L CNN
-F 2 "" V 5580 3650 50  0001 C CNN
+F 2 "Resistor_SMD:R_0603_1608Metric_Pad0.98x0.95mm_HandSolder" V 5580 3650 50  0001 C CNN
 F 3 "~" H 5650 3650 50  0001 C CNN
 	1    5650 3650
@@
 F 0 "R184" H 5720 3996 50  0000 L CNN
 F 1 "R" H 5720 3905 50  0000 L CNN
-F 2 "" V 5580 3950 50  0001 C CNN
+F 2 "Resistor_SMD:R_0603_1608Metric_Pad0.98x0.95mm_HandSolder" V 5580 3950 50  0001 C CNN
 F 3 "~" H 5650 3950 50  0001 C CNN
 	1    5650 3950
@@
 F 0 "R185" H 6020 3696 50  0000 L CNN
 F 1 "R" H 6020 3605 50  0000 L CNN
-F 2 "" V 5880 3650 50  0001 C CNN
+F 2 "Resistor_SMD:R_0603_1608Metric_Pad0.98x0.95mm_HandSolder" V 5880 3650 50  0001 C CNN
 F 3 "~" H 5950 3650 50  0001 C CNN
 	1    5950 3650
@@
 F 0 "R186" H 6020 3996 50  0000 L CNN
 F 1 "R" H 6020 3905 50  0000 L CNN
-F 2 "" V 5880 3950 50  0001 C CNN
+F 2 "Resistor_SMD:R_0603_1608Metric_Pad0.98x0.95mm_HandSolder" V 5880 3950 50  0001 C CNN
 F 3 "~" H 5950 3950 50  0001 C CNN
 	1    5950 3950

Commit message: Updated with Mouser links for BOM
Parts:
- R103: renamed from R179; value R -> DNP 50k
- R104: renamed from R180; value R -> DNP 50k
- R105: renamed from R181; value R -> DNP 50k
- R106: renamed from R182; value R -> DNP 50k
- R107: renamed from R183; value R -> DNP 50k
- R108: renamed from R184; value R -> DNP 50k
- R109: renamed from R185; value R -> DNP 50k
- R110: renamed from R186; value R -> DNP 50k
Changed lines of the file:
@@
 $Descr A4 11693 8268
 encoding utf-8
-Sheet 28 35
+Sheet 21 35
 Title ""
 Date ""
@@
 $EndDescr
 $Comp
-L Device:R R179
+L Device:R R103
 U 1 1 6234DD24
 P 5000 3650
-AR Path="/61619F34/61FF949C/6234DD24" Ref="R179"  Part="1"
+AR Path="/61619F34/61FF949C/6234DD24" Ref="R103"  Part="1"
 AR Path="/61619F34/620A15AD/6234DD24" Ref="R?"  Part="1"
 AR Path="/61619F34/620DEAEE/6234DD24" Ref="R?"  Part="1"
@@
 AR Path="/61619F34/62140E50/6234DD24" Ref="R?"  Part="1"
 AR Path="/61619F34/6215FBD7/6234DD24" Ref="R?"  Part="1"
-F 0 "R179" H 5070 3696 50  0000 L CNN
-F 1 "R" H 5070 3605 50  0000 L CNN
+F 0 "R103" H 4850 4000 50  0000 L CNN
+F 1 "DNP 50k" H 4850 3900 50  0000 L CNN
 F 2 "Resistor_SMD:R_0603_1608Metric_Pad0.98x0.95mm_HandSolder" V 4930 3650 50  0001 C CNN
 F 3 "~" H 5000 3650 50  0001 C CNN
@@
 $EndComp
 $Comp
-L Device:R R180
+L Device:R R104
 U 1 1 6234DD25
 P 5000 3950
-AR Path="/61619F34/61FF949C/6234DD25" Ref="R180"  Part="1"
+AR Path="/61619F34/61FF949C/6234DD25" Ref="R104"  Part="1"
 AR Path="/61619F34/620A15AD/6234DD25" Ref="R?"  Part="1"
 AR Path="/61619F34/620DEAEE/6234DD25" Ref="R?"  Part="1"
@@
 AR Path="/61619F34/62140E50/6234DD25" Ref="R?"  Part="1"
 AR Path="/61619F34/6215FBD7/6234DD25" Ref="R?"  Part="1"
-F 0 "R180" H 5070 3996 50  0000 L CNN
-F 1 "R" H 5070 3905 50  0000 L CNN
+F 0 "R104" H 4850 3700 50  0000 L CNN
+F 1 "DNP 50k" H 4850 3600 50  0000 L CNN
 F 2 "Resistor_SMD:R_0603_1608Metric_Pad0.98x0.95mm_HandSolder" V 4930 3950 50  0001 C CNN
 F 3 "~" H 5000 3950 50  0001 C CNN
@@
 $EndComp
 $Comp
-L Device:R R181
+L Device:R R105
 U 1 1 61FFAD0C
 P 5350 3650
-AR Path="/61619F34/61FF949C/61FFAD0C" Ref="R181"  Part="1"
+AR Path="/61619F34/61FF949C/61FFAD0C" Ref="R105"  Part="1"
 AR Path="/61619F34/620A15AD/61FFAD0C" Ref="R?"  Part="1"
 AR Path="/61619F34/620DEAEE/61FFAD0C" Ref="R?"  Part="1"
@@
 AR Path="/61619F34/62140E50/61FFAD0C" Ref="R?"  Part="1"
 AR Path="/61619F34/6215FBD7/61FFAD0C" Ref="R?"  Part="1"
-F 0 "R181" H 5420 3696 50  0000 L CNN
-F 1 "R" H 5420 3605 50  0000 L CNN
+F 0 "R105" H 5200 4000 50  0000 L CNN
+F 1 "DNP 50k" H 5200 3900 50  0000 L CNN
 F 2 "Resistor_SMD:R_0603_1608Metric_Pad0.98x0.95mm_HandSolder" V 5280 3650 50  0001 C CNN
 F 3 "~" H 5350 3650 50  0001 C CNN
@@
 $EndComp
 $Comp
-L Device:R R182
+L Device:R R106
 U 1 1 61FFAD12
 P 5350 3950
-AR Path="/61619F34/61FF949C/61FFAD12" Ref="R182"  Part="1"
+AR Path="/61619F34/61FF949C/61FFAD12" Ref="R106"  Part="1"
 AR Path="/61619F34/620A15AD/61FFAD12" Ref="R?"  Part="1"
 AR Path="/61619F34/620DEAEE/61FFAD12" Ref="R?"  Part="1"
@@
 AR Path="/61619F34/62140E50/61FFAD12" Ref="R?"  Part="1"
 AR Path="/61619F34/6215FBD7/61FFAD12" Ref="R?"  Part="1"
-F 0 "R182" H 5420 3996 50  0000 L CNN
-F 1 "R" H 5420 3905 50  0000 L CNN
+F 0 "R106" H 5250 3700 50  0000 L CNN
+F 1 "DNP 50k" H 5250 3600 50  0000 L CNN
 F 2 "Resistor_SMD:R_0603_1608Metric_Pad0.98x0.95mm_HandSolder" V 5280 3950 50  0001 C CNN
 F 3 "~" H 5350 3950 50  0001 C CNN
@@
 $EndComp
 $Comp
-L Device:R R183
+L Device:R R107
 U 1 1 6234DD28
 P 5650 3650
-AR Path="/61619F34/61FF949C/6234DD28" Ref="R183"  Part="1"
+AR Path="/61619F34/61FF949C/6234DD28" Ref="R107"  Part="1"
 AR Path="/61619F34/620A15AD/6234DD28" Ref="R?"  Part="1"
 AR Path="/61619F34/620DEAEE/6234DD28" Ref="R?"  Part="1"
@@
 AR Path="/61619F34/62140E50/6234DD28" Ref="R?"  Part="1"
 AR Path="/61619F34/6215FBD7/6234DD28" Ref="R?"  Part="1"
-F 0 "R183" H 5720 3696 50  0000 L CNN
-F 1 "R" H 5720 3605 50  0000 L CNN
+F 0 "R107" H 5550 4000 50  0000 L CNN
+F 1 "DNP 50k" H 5550 3900 50  0000 L CNN
 F 2 "Resistor_SMD:R_0603_1608Metric_Pad0.98x0.95mm_HandSolder" V 5580 3650 50  0001 C CNN
 F 3 "~" H 5650 3650 50  0001 C CNN
@@
 $EndComp
 $Comp
-L Device:R R184
+L Device:R R108
 U 1 1 6234DD29
 P 5650 3950
-AR Path="/61619F34/61FF949C/6234DD29" Ref="R184"  Part="1"
+AR Path="/61619F34/61FF949C/6234DD29" Ref="R108"  Part="1"
 AR Path="/61619F34/620A15AD/6234DD29" Ref="R?"  Part="1"
 AR Path="/61619F34/620DEAEE/6234DD29" Ref="R?"  Part="1"
@@
 AR Path="/61619F34/62140E50/6234DD29" Ref="R?"  Part="1"
 AR Path="/61619F34/6215FBD7/6234DD29" Ref="R?"  Part="1"
-F 0 "R184" H 5720 3996 50  0000 L CNN
-F 1 "R" H 5720 3905 50  0000 L CNN
+F 0 "R108" H 5600 3700 50  0000 L CNN
+F 1 "DNP 50k" H 5600 3600 50  0000 L CNN
 F 2 "Resistor_SMD:R_0603_1608Metric_Pad0.98x0.95mm_HandSolder" V 5580 3950 50  0001 C CNN
 F 3 "~" H 5650 3950 50  0001 C CNN
@@
 $EndComp
 $Comp
-L Device:R R185
+L Device:R R109
 U 1 1 6234DD2A
 P 5950 3650
-AR Path="/61619F34/61FF949C/6234DD2A" Ref="R185"  Part="1"
+AR Path="/61619F34/61FF949C/6234DD2A" Ref="R109"  Part="1"
 AR Path="/61619F34/620A15AD/6234DD2A" Ref="R?"  Part="1"
 AR Path="/61619F34/620DEAEE/6234DD2A" Ref="R?"  Part="1"
@@
 AR Path="/61619F34/62140E50/6234DD2A" Ref="R?"  Part="1"
 AR Path="/61619F34/6215FBD7/6234DD2A" Ref="R?"  Part="1"
-F 0 "R185" H 6020 3696 50  0000 L CNN
-F 1 "R" H 6020 3605 50  0000 L CNN
+F 0 "R109" H 5900 4000 50  0000 L CNN
+F 1 "DNP 50k" H 5900 3900 50  0000 L CNN
 F 2 "Resistor_SMD:R_0603_1608Metric_Pad0.98x0.95mm_HandSolder" V 5880 3650 50  0001 C CNN
 F 3 "~" H 5950 3650 50  0001 C CNN
@@
 $EndComp
 $Comp
-L Device:R R186
+L Device:R R110
 U 1 1 6234DD2B
 P 5950 3950
-AR Path="/61619F34/61FF949C/6234DD2B" Ref="R186"  Part="1"
+AR Path="/61619F34/61FF949C/6234DD2B" Ref="R110"  Part="1"
 AR Path="/61619F34/620A15AD/6234DD2B" Ref="R?"  Part="1"
 AR Path="/61619F34/620DEAEE/6234DD2B" Ref="R?"  Part="1"
@@
 AR Path="/61619F34/62140E50/6234DD2B" Ref="R?"  Part="1"
 AR Path="/61619F34/6215FBD7/6234DD2B" Ref="R?"  Part="1"
-F 0 "R186" H 6020 3996 50  0000 L CNN
-F 1 "R" H 6020 3905 50  0000 L CNN
+F 0 "R110" H 5950 3700 50  0000 L CNN
+F 1 "DNP 50k" H 5950 3600 50  0000 L CNN
 F 2 "Resistor_SMD:R_0603_1608Metric_Pad0.98x0.95mm_HandSolder" V 5880 3950 50  0001 C CNN
 F 3 "~" H 5950 3950 50  0001 C CNN
