File: 211006_lmu_r0/file615D6DD2.sch (KiCad schematic (older format))
At the start: 26 parts, among them J11 Conn_ARM_JTAG_SWD_10, J12 Conn_01x03, SW1 SW_Push, SW2 SW_SPST, U9 STM32F103C8Tx, Y1 Crystal_GND23

Commit message: Updated with Mouser links for BOM
Parts:
- C182: value 10n -> 10nF
- C183: value 1u -> 1uF
- C184, C185, C186: value 100n -> 100nF
- D40: value LED (Blue) TX -> LED (Blue); Manufacturer (none) -> Lumex; Mouser Part Number (none) -> SML-LX0805USBC-TR; Mouser URL (none) -> https://au.mouser.com/ProductDetail/Lumex/SML-LX0805USBC-TR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; Part Number (none) -> SML-LX0805USBC-TR
- D41: value LED (Red) LED0 -> LED (Red); Manufacturer (none) -> AMS OSRAM; Mouser Part Number (none) -> 720-LSR976-NR-1; Mouser URL (none) -> https://au.mouser.com/ProductDetail/ams-OSRAM/LS-R976-NR-1-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; Part Number (none) -> LS R976-NR-1-0-20-R18
- D42: value LED (Blue) RX -> LED (Blue); Manufacturer (none) -> Lumex; Mouser Part Number (none) -> SML-LX0805USBC-TR; Mouser URL (none) -> https://au.mouser.com/ProductDetail/Lumex/SML-LX0805USBC-TR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; Part Number (none) -> SML-LX0805USBC-TR
- D43, D44: Manufacturer (none) -> AMS OSRAM; Mouser Part Number (none) -> 720-LOR976-PS-1; Mouser URL (none) -> https://au.mouser.com/ProductDetail/ams-OSRAM/LO-R976-PS-1-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; Part Number (none) -> LO R976-PS-1-0-20-R18
- FB1: value Ferrite_Bead -> Ferrite Bead; Manufacturer TDK Corportation -> TDK; Mouser Part Number (none) -> 810-MMZ0603S102HT000; Mouser URL (none) -> https://au.mouser.com/ProductDetail/TDK/MMZ0603S102HT000?qs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; Part Number MMZ2012Y202BTD25 -> MMZ0603S102HT000
- R242, R243, R244, R245, R246: value 2.2k -> 2.2kR
- R247: value 50k -> 50kR
- TP158: renamed from TP153; Manufacturer (none) -> -; Mouser Part Number (none) -> -; Mouser URL (none) -> -; Part Number (none) -> -
- TP159: renamed from TP154; Manufacturer (none) -> -; Mouser Part Number (none) -> -; Mouser URL (none) -> -; Part Number (none) -> -
- TP160: renamed from TP155; Manufacturer (none) -> -; Mouser Part Number (none) -> -; Mouser URL (none) -> -; Part Number (none) -> -
- U9: Manufacturer (none) -> ST Microelectronics; Mouser Part Number (none) -> NOT AVAILABLE!; Mouser URL (none) -> NOT AVAILABLE!; Part Number (none) -> STM32F103C8Tx
- Y1: value Crystal_GND23 -> 16MHz; footprint (none) -> Crystal:Crystal_SMD_3225-4Pin_3.2x2.5mm_HandSoldering; Manufacturer (none) -> ABRACON; Mouser Part Number (none) -> 815-M8AIG-16-12-2ZT3; Mouser URL (none) -> https://au.mouser.com/ProductDetail/ABRACON/ABM8AIG-16000MH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; Part Number (none) -> ABM8AIG-16.000MHZ-12-2Z-T3
Changed lines of the file:
@@
 P 7050 2400
 F 0 "FB1" V 7200 2450 50  0000 C CNN
-F 1 "Ferrite_Bead" V 7300 2450 50  0000 C CNN
+F 1 "Ferrite Bead" V 7300 2450 50  0000 C CNN
 F 2 "Inductor_SMD:L_0603_1608Metric_Pad1.05x0.95mm_HandSolder" V 6980 2400 50  0001 C CNN
 F 3 "~" H 7050 2400 50  0001 C CNN
-F 4 "MMZ2012Y202BTD25 " V 7050 2400 50  0001 C CNN "Part Number"
-F 5 "TDK Corportation" V 7050 2400 50  0001 C CNN "Manufacturer"
+F 4 "MMZ0603S102HT000" V 7050 2400 50  0001 C CNN "Part Number"
+F 5 "TDK" V 7050 2400 50  0001 C CNN "Manufacturer"
+F 6 "810-MMZ0603S102HT000" H 7050 2400 50  0001 C CNN "Mouser Part Number"
+F 7 "https://au.mouser.com/ProductDetail/TDK/MMZ0603S102HT000?qs=sGAEpiMZZMukHu%252BjC5l7YXmIAtxpPm1GoBQpx1Hc8%2F0%3D" H 7050 2400 50  0001 C CNN "Mouser URL"
 	1    7050 2400
 	0    1    1    0
@@
 P 7550 2400
 F 0 "C183" H 7450 2800 50  0000 L CNN
-F 1 "1u" H 7450 2700 50  0000 L CNN
+F 1 "1uF" H 7450 2700 50  0000 L CNN
 F 2 "Capacitor_SMD:C_0805_2012Metric_Pad1.18x1.45mm_HandSolder" H 7588 2250 50  0001 C CNN
 F 3 "~" H 7550 2400 50  0001 C CNN
@@
 F 2 "Package_QFP:LQFP-48_7x7mm_P0.5mm" H 5700 2500 50  0001 R CNN
 F 3 "http://www.st.com/st-web-ui/static/active/en/resource/technical/document/datasheet/CD00161566.pdf" H 6300 3900 50  0001 C CNN
+F 4 "STM32F103C8Tx" H 6300 3900 50  0001 C CNN "Part Number"
+F 5 "ST Microelectronics" H 6300 3900 50  0001 C CNN "Manufacturer"
+F 6 "NOT AVAILABLE!" H 6300 3900 50  0001 C CNN "Mouser Part Number"
+F 7 "NOT AVAILABLE!" H 6300 3900 50  0001 C CNN "Mouser URL"
 	1    6300 3900
 	1    0    0    -1
@@
 P 3350 2750
 F 0 "C182" H 3465 2796 50  0000 L CNN
-F 1 "10n" H 3465 2705 50  0000 L CNN
+F 1 "10nF" H 3465 2705 50  0000 L CNN
 F 2 "Capacitor_SMD:C_0603_1608Metric_Pad1.08x0.95mm_HandSolder" H 3388 2600 50  0001 C CNN
 F 3 "~" H 3350 2750 50  0001 C CNN
@@
 P 3350 2450
 F 0 "R247" H 3420 2496 50  0000 L CNN
-F 1 "50k" H 3420 2405 50  0000 L CNN
+F 1 "50kR" H 3420 2405 50  0000 L CNN
 F 2 "Resistor_SMD:R_0603_1608Metric_Pad0.98x0.95mm_HandSolder" V 3280 2450 50  0001 C CNN
 F 3 "~" H 3350 2450 50  0001 C CNN
@@
 P 4500 3050
 F 0 "Y1" V 4750 2900 50  0000 L CNN
-F 1 "Crystal_GND23" V 4850 2900 50  0000 L CNN
-F 2 "" H 4500 3050 50  0001 C CNN
+F 1 "16MHz" V 4850 2900 50  0000 L CNN
+F 2 "Crystal:Crystal_SMD_3225-4Pin_3.2x2.5mm_HandSoldering" H 4500 3050 50  0001 C CNN
 F 3 "~" H 4500 3050 50  0001 C CNN
+F 4 "ABRACON" H 4500 3050 50  0001 C CNN "Manufacturer"
+F 5 "815-M8AIG-16-12-2ZT3" H 4500 3050 50  0001 C CNN "Mouser Part Number"
+F 6 "https://au.mouser.com/ProductDetail/ABRACON/ABM8AIG-16000MHZ-12-2Z-T3?qs=gG6m684uYP7glnqUpaQmDA%3D%3D" H 4500 3050 50  0001 C CNN "Mouser URL"
+F 7 "ABM8AIG-16.000MHZ-12-2Z-T3" H 4500 3050 50  0001 C CNN "Part Number"
 	1    4500 3050
 	0    1    1    0
@@
 	6900 5100 7400 5100
 $Comp
-L Connector:TestPoint TP153
+L Connector:TestPoint TP158
 U 1 1 616033D7
 P 3000 2600
-F 0 "TP153" H 3058 2718 50  0000 L CNN
+F 0 "TP158" H 3058 2718 50  0000 L CNN
 F 1 "TestPoint" H 3058 2627 50  0000 L CNN
 F 2 "TestPoint:TestPoint_Pad_D1.0mm" H 3200 2600 50  0001 C CNN
 F 3 "~" H 3200 2600 50  0001 C CNN
+F 4 "-" H 3000 2600 50  0001 C CNN "Part Number"
+F 5 "-" H 3000 2600 50  0001 C CNN "Manufacturer"
+F 6 "-" H 3000 2600 50  0001 C CNN "Mouser Part Number"
+F 7 "-" H 3000 2600 50  0001 C CNN "Mouser URL"
 	1    3000 2600
 	1    0    0    -1
@@
 	6900 4200 7400 4200
 $Comp
-L Connector:TestPoint TP154
+L Connector:TestPoint TP159
 U 1 1 6162689C
 P 3200 1000
-F 0 "TP154" V 3154 1188 50  0000 L CNN
+F 0 "TP159" V 3154 1188 50  0000 L CNN
 F 1 "TestPoint" V 3245 1188 50  0000 L CNN
 F 2 "TestPoint:TestPoint_Pad_D1.0mm" H 3400 1000 50  0001 C CNN
 F 3 "~" H 3400 1000 50  0001 C CNN
+F 4 "-" H 3200 1000 50  0001 C CNN "Part Number"
+F 5 "-" H 3200 1000 50  0001 C CNN "Manufacturer"
+F 6 "-" H 3200 1000 50  0001 C CNN "Mouser Part Number"
+F 7 "-" H 3200 1000 50  0001 C CNN "Mouser URL"
 	1    3200 1000
 	0    1    1    0
 $EndComp
 $Comp
-L Connector:TestPoint TP155
+L Connector:TestPoint TP160
 U 1 1 6162866E
 P 3200 1100
-F 0 "TP155" V 3154 1288 50  0000 L CNN
+F 0 "TP160" V 3154 1288 50  0000 L CNN
 F 1 "TestPoint" V 3245 1288 50  0000 L CNN
 F 2 "TestPoint:TestPoint_Pad_D1.0mm" H 3400 1100 50  0001 C CNN
 F 3 "~" H 3400 1100 50  0001 C CNN
+F 4 "-" H 3200 1100 50  0001 C CNN "Part Number"
+F 5 "-" H 3200 1100 50  0001 C CNN "Manufacturer"
+F 6 "-" H 3200 1100 50  0001 C CNN "Mouser Part Number"
+F 7 "-" H 3200 1100 50  0001 C CNN "Mouser URL"
 	1    3200 1100
 	0    1    1    0
@@
 P 1800 5550
 F 0 "D40" V 1350 6150 50  0000 R CNN
-F 1 "LED (Blue) TX" V 1250 6150 50  0000 R CNN
+F 1 "LED (Blue)" V 1250 6150 50  0000 R CNN
 F 2 "LED_SMD:LED_0805_2012Metric_Pad1.15x1.40mm_HandSolder" H 1800 5550 50  0001 C CNN
 F 3 "~" H 1800 5550 50  0001 C CNN
+F 4 "Lumex" H 1800 5550 50  0001 C CNN "Manufacturer"
+F 5 "SML-LX0805USBC-TR" H 1800 5550 50  0001 C CNN "Mouser Part Number"
+F 6 "https://au.mouser.com/ProductDetail/Lumex/SML-LX0805USBC-TR?qs=jywnEC9mS4F%2FCvyk4BNITw%3D%3D" H 1800 5550 50  0001 C CNN "Mouser URL"
+F 7 "SML-LX0805USBC-TR" H 1800 5550 50  0001 C CNN "Part Number"
 	1    1800 5550
 	0    -1   -1   0
@@
 P 1800 5250
 F 0 "R242" H 1870 5296 50  0000 L CNN
-F 1 "2.2k" H 1870 5205 50  0000 L CNN
+F 1 "2.2kR" H 1870 5205 50  0000 L CNN
 F 2 "Resistor_SMD:R_0603_1608Metric_Pad0.98x0.95mm_HandSolder" V 1730 5250 50  0001 C CNN
 F 3 "~" H 1800 5250 50  0001 C CNN
@@
 P 7900 2400
 F 0 "C184" H 7800 2800 50  0000 L CNN
-F 1 "100n" H 7800 2700 50  0000 L CNN
+F 1 "100nF" H 7800 2700 50  0000 L CNN
 F 2 "Capacitor_SMD:C_0603_1608Metric_Pad1.08x0.95mm_HandSolder" H 7938 2250 50  0001 C CNN
 F 3 "~" H 7900 2400 50  0001 C CNN
@@
 P 8250 2400
 F 0 "C185" H 8150 2800 50  0000 L CNN
-F 1 "100n" H 8150 2700 50  0000 L CNN
+F 1 "100nF" H 8150 2700 50  0000 L CNN
 F 2 "Capacitor_SMD:C_0603_1608Metric_Pad1.08x0.95mm_HandSolder" H 8288 2250 50  0001 C CNN
 F 3 "~" H 8250 2400 50  0001 C CNN
@@
 P 8600 2400
 F 0 "C186" H 8500 2800 50  0000 L CNN
-F 1 "100n" H 8500 2700 50  0000 L CNN
+F 1 "100nF" H 8500 2700 50  0000 L CNN
 F 2 "Capacitor_SMD:C_0603_1608Metric_Pad1.08x0.95mm_HandSolder" H 8638 2250 50  0001 C CNN
 F 3 "~" H 8600 2400 50  0001 C CNN
@@
 P 2200 5250
 F 0 "R244" H 2270 5296 50  0000 L CNN
-F 1 "2.2k" H 2270 5205 50  0000 L CNN
+F 1 "2.2kR" H 2270 5205 50  0000 L CNN
 F 2 "Resistor_SMD:R_0603_1608Metric_Pad0.98x0.95mm_HandSolder" V 2130 5250 50  0001 C CNN
 F 3 "~" H 2200 5250 50  0001 C CNN
@@
 P 2600 5250
 F 0 "R245" H 2670 5296 50  0000 L CNN
-F 1 "2.2k" H 2670 5205 50  0000 L CNN
+F 1 "2.2kR" H 2670 5205 50  0000 L CNN
 F 2 "Resistor_SMD:R_0603_1608Metric_Pad0.98x0.95mm_HandSolder" V 2530 5250 50  0001 C CNN
 F 3 "~" H 2600 5250 50  0001 C CNN
@@
 P 2950 5250
 F 0 "R246" H 3020 5296 50  0000 L CNN
-F 1 "2.2k" H 3020 5205 50  0000 L CNN
+F 1 "2.2kR" H 3020 5205 50  0000 L CNN
 F 2 "Resistor_SMD:R_0603_1608Metric_Pad0.98x0.95mm_HandSolder" V 2880 5250 50  0001 C CNN
 F 3 "~" H 2950 5250 50  0001 C CNN
@@
 P 2200 5550
 F 0 "D42" V 1750 5900 50  0000 R CNN
-F 1 "LED (Blue) RX" V 1650 5900 50  0000 R CNN
+F 1 "LED (Blue)" V 1650 5900 50  0000 R CNN
 F 2 "LED_SMD:LED_0805_2012Metric_Pad1.15x1.40mm_HandSolder" H 2200 5550 50  0001 C CNN
 F 3 "~" H 2200 5550 50  0001 C CNN
+F 4 "Lumex" H 2200 5550 50  0001 C CNN "Manufacturer"
+F 5 "SML-LX0805USBC-TR" H 2200 5550 50  0001 C CNN "Mouser Part Number"
+F 6 "https://au.mouser.com/ProductDetail/Lumex/SML-LX0805USBC-TR?qs=jywnEC9mS4F%2FCvyk4BNITw%3D%3D" H 2200 5550 50  0001 C CNN "Mouser URL"
+F 7 "SML-LX0805USBC-TR" H 2200 5550 50  0001 C CNN "Part Number"
 	1    2200 5550
 	0    -1   -1   0
@@
 F 2 "LED_SMD:LED_0805_2012Metric_Pad1.15x1.40mm_HandSolder" H 2600 5550 50  0001 C CNN
 F 3 "~" H 2600 5550 50  0001 C CNN
+F 4 "AMS OSRAM" H 2600 5550 50  0001 C CNN "Manufacturer"
+F 5 "720-LOR976-PS-1" H 2600 5550 50  0001 C CNN "Mouser Part Number"
+F 6 "https://au.mouser.com/ProductDetail/ams-OSRAM/LO-R976-PS-1-0-20-R18?qs=p6VZ%252BklCkRQY6bKwpfgF7g%3D%3D" H 2600 5550 50  0001 C CNN "Mouser URL"
+F 7 "LO R976-PS-1-0-20-R18" H 2600 5550 50  0001 C CNN "Part Number"
 	1    2600 5550
 	0    -1   -1   0
@@
 F 2 "LED_SMD:LED_0805_2012Metric_Pad1.15x1.40mm_HandSolder" H 2950 5550 50  0001 C CNN
 F 3 "~" H 2950 5550 50  0001 C CNN
+F 4 "AMS OSRAM" H 2950 5550 50  0001 C CNN "Manufacturer"
+F 5 "720-LOR976-PS-1" H 2950 5550 50  0001 C CNN "Mouser Part Number"
+F 6 "https://au.mouser.com/ProductDetail/ams-OSRAM/LO-R976-PS-1-0-20-R18?qs=p6VZ%252BklCkRQY6bKwpfgF7g%3D%3D" H 2950 5550 50  0001 C CNN "Mouser URL"
+F 7 "LO R976-PS-1-0-20-R18" H 2950 5550 50  0001 C CNN "Part Number"
 	1    2950 5550
 	0    -1   -1   0
@@
 P 1850 3350
 F 0 "R243" H 1920 3396 50  0000 L CNN
-F 1 "2.2k" H 1920 3305 50  0000 L CNN
+F 1 "2.2kR" H 1920 3305 50  0000 L CNN
 F 2 "Resistor_SMD:R_0603_1608Metric_Pad0.98x0.95mm_HandSolder" V 1780 3350 50  0001 C CNN
 F 3 "~" H 1850 3350 50  0001 C CNN
@@
 P 1850 3650
 F 0 "D41" V 1850 4350 50  0000 R CNN
-F 1 "LED (Red) LED0" V 1750 4350 50  0000 R CNN
+F 1 "LED (Red)" V 1750 4350 50  0000 R CNN
 F 2 "LED_SMD:LED_0805_2012Metric_Pad1.15x1.40mm_HandSolder" H 1850 3650 50  0001 C CNN
 F 3 "~" H 1850 3650 50  0001 C CNN
+F 4 "AMS OSRAM" H 1850 3650 50  0001 C CNN "Manufacturer"
+F 5 "720-LSR976-NR-1" H 1850 3650 50  0001 C CNN "Mouser Part Number"
+F 6 "https://au.mouser.com/ProductDetail/ams-OSRAM/LS-R976-NR-1-0-20-R18?qs=sGAEpiMZZMt82OzCyDsLFGbrp1fQkD8H8bij58Oys9s%3D" H 1850 3650 50  0001 C CNN "Mouser URL"
+F 7 "LS R976-NR-1-0-20-R18" H 1850 3650 50  0001 C CNN "Part Number"
 	1    1850 3650
 	0    -1   -1   0
