File: 211006_lmu_r0/file616BA637.sch (KiCad schematic (older format))
At the start: 13 parts

Commit message: Updated BOM and footprints for non-hv components
Parts:
- removed C? (x4): C, symbol Device:C
- removed R?: R, symbol Device:R
- added C? (x3): DNP 10p, Capacitor_SMD:C_0603_1608Metric_Pad1.08x0.95mm_HandSolder, symbol Device:C
- added C?: 100n, Capacitor_SMD:C_0603_1608Metric_Pad1.08x0.95mm_HandSolder, symbol Device:C
- added R?: 60, Resistor_SMD:R_0805_2012Metric_Pad1.20x1.40mm_HandSolder, symbol Device:R
- C12: renamed from C?; value C -> 100n; footprint (none) -> Capacitor_SMD:C_0603_1608Metric_Pad1.08x0.95mm_HandSolder
- C7: renamed from C?; value C -> 10n; footprint (none) -> Capacitor_SMD:C_0603_1608Metric_Pad1.08x0.95mm_HandSolder
- C8: renamed from C?; value C -> DNP 10p; footprint (none) -> Capacitor_SMD:C_0603_1608Metric_Pad1.08x0.95mm_HandSolder
- L2: renamed from L?; footprint (none) -> Inductor_SMD:L_CommonModeChoke_Coilcraft_1812CAN; Manufacturer (none) -> EPCOS - TDK; Part Number (none) -> 0ZCF0100AF2A
- R3: renamed from R?; value R -> 60; footprint (none) -> Resistor_SMD:R_0805_2012Metric_Pad1.20x1.40mm_HandSolder
- R5: renamed from R?; value R -> 0; footprint (none) -> Resistor_SMD:R_0805_2012Metric_Pad1.20x1.40mm_HandSolder
- gave numbers to parts that had none: 2
Connections:
- net +3V3: now also C?.1
- net CAN_L: now also C?.1, R?.2
- net CAN_S: now also C?.2, C?.2, C?.2
- net GND: now also C?.2
- net at D5.1 (K), L2.4, U2.6 (CANL): now also C?.1
- net at D5.2 (K), L2.2, U2.7 (CANH): now also C?.1
- net at C7.2, R3.2: now also R?.1
Changed lines of the file:
@@
 $EndDescr
 $Comp
-L Power_Protection:NUP2105L D?
+L Power_Protection:NUP2105L D5
 U 1 1 616BCB8F
 P 5000 4100
-F 0 "D?" H 5205 4146 50  0000 L CNN
+F 0 "D5" H 5205 4146 50  0000 L CNN
 F 1 "NUP2105L" H 5205 4055 50  0000 L CNN
 F 2 "Package_TO_SOT_SMD:SOT-23" H 5225 4050 50  0001 L CNN
@@
 CAN_RX
 $Comp
-L Device:R R?
-U 1 1 616C53CC
-P 2200 3500
-F 0 "R?" H 2270 3546 50  0000 L CNN
-F 1 "R" H 2270 3455 50  0000 L CNN
-F 2 "" V 2130 3500 50  0001 C CNN
-F 3 "~" H 2200 3500 50  0001 C CNN
-	1    2200 3500
-	1    0    0    -1
-$EndComp
-$Comp
-L Device:R R?
-U 1 1 616C5950
-P 2200 3900
-F 0 "R?" H 2270 3946 50  0000 L CNN
-F 1 "R" H 2270 3855 50  0000 L CNN
-F 2 "" V 2130 3900 50  0001 C CNN
-F 3 "~" H 2200 3900 50  0001 C CNN
-	1    2200 3900
-	1    0    0    -1
-$EndComp
-$Comp
-L Device:C C?
+L Device:C C7
 U 1 1 616C5DE2
 P 2450 3700
-F 0 "C?" V 2198 3700 50  0000 C CNN
-F 1 "C" V 2289 3700 50  0000 C CNN
-F 2 "" H 2488 3550 50  0001 C CNN
+F 0 "C7" V 2198 3700 50  0000 C CNN
+F 1 "10n" V 2289 3700 50  0000 C CNN
+F 2 "Capacitor_SMD:C_0603_1608Metric_Pad1.08x0.95mm_HandSolder" H 2488 3550 50  0001 C CNN
 F 3 "~" H 2450 3700 50  0001 C CNN
 	1    2450 3700
@@
 Connection ~ 2200 3700
 $Comp
-L Device:L_Core_Ferrite_Coupled L?
+L Device:L_Core_Ferrite_Coupled L2
 U 1 1 616C7456
 P 3750 3700
-F 0 "L?" H 3750 3981 50  0000 C CNN
+F 0 "L2" H 3750 3981 50  0000 C CNN
 F 1 "L_Core_Ferrite_Coupled" H 3750 3890 50  0000 C CNN
-F 2 "" H 3750 3700 50  0001 C CNN
+F 2 "Inductor_SMD:L_CommonModeChoke_Coilcraft_1812CAN" H 3750 3700 50  0001 C CNN
 F 3 "~" H 3750 3700 50  0001 C CNN
+F 4 "0ZCF0100AF2A" H 3750 3700 50  0001 C CNN "Part Number"
+F 5 "EPCOS - TDK" H 3750 3700 50  0001 C CNN "Manufacturer"
 	1    3750 3700
 	1    0    0    -1
@@
 	2650 3550 2650 3350
 Wire Wire Line
-	2650 3350 2200 3350
-Wire Wire Line
-	2200 4050 2650 4050
-Wire Wire Line
 	2650 4050 2650 3850
 Wire Wire Line
 	3950 3550 4100 3550
-Wire Wire Line
-	3950 3850 4350 3850
-$Comp
-L Device:C C?
-U 1 1 616DF522
-P 4350 4050
-F 0 "C?" H 4465 4096 50  0000 L CNN
-F 1 "C" H 4465 4005 50  0000 L CNN
-F 2 "" H 4388 3900 50  0001 C CNN
-F 3 "~" H 4350 4050 50  0001 C CNN
-	1    4350 4050
-	1    0    0    -1
-$EndComp
-$Comp
-L Device:C C?
-U 1 1 616DFB8B
-P 4100 4050
-F 0 "C?" H 4215 4096 50  0000 L CNN
-F 1 "C" H 4215 4005 50  0000 L CNN
-F 2 "" H 4138 3900 50  0001 C CNN
-F 3 "~" H 4100 4050 50  0001 C CNN
-	1    4100 4050
-	1    0    0    -1
-$EndComp
-$Comp
-L Device:C C?
-U 1 1 616DFD5A
-P 3500 4050
-F 0 "C?" H 3615 4096 50  0000 L CNN
-F 1 "C" H 3615 4005 50  0000 L CNN
-F 2 "" H 3538 3900 50  0001 C CNN
-F 3 "~" H 3500 4050 50  0001 C CNN
-	1    3500 4050
-	1    0    0    -1
-$EndComp
-$Comp
-L Device:C C?
+$Comp
+L Device:C C8
 U 1 1 616E025C
 P 3250 4050
-F 0 "C?" H 3365 4096 50  0000 L CNN
-F 1 "C" H 3365 4005 50  0000 L CNN
-F 2 "" H 3288 3900 50  0001 C CNN
+F 0 "C8" H 3000 3650 50  0000 L CNN
+F 1 "DNP 10p" H 3000 3550 50  0000 L CNN
+F 2 "Capacitor_SMD:C_0603_1608Metric_Pad1.08x0.95mm_HandSolder" H 3288 3900 50  0001 C CNN
 F 3 "~" H 3250 4050 50  0001 C CNN
 	1    3250 4050
@@
 $EndComp
 Wire Wire Line
-	2200 3350 2000 3350
-Connection ~ 2200 3350
-Wire Wire Line
-	2200 4050 2000 4050
-Connection ~ 2200 4050
-Wire Wire Line
 	3500 3900 3500 3850
 Connection ~ 3500 3850
@@
 Wire Wire Line
 	4100 3550 5100 3550
-Wire Wire Line
-	4350 3900 4350 3850
-Connection ~ 4350 3850
-Wire Wire Line
-	4350 3850 4900 3850
 Text HLabel 2000 3350 0    50   Input ~ 0
 CAN_H
@@
 	5000 4300 5000 4350
 Wire Wire Line
-	4350 4200 4350 4350
-Connection ~ 4350 4350
-Wire Wire Line
-	4350 4350 5000 4350
-Wire Wire Line
 	4100 4200 4100 4350
 Connection ~ 4100 4350
 Wire Wire Line
-	4100 4350 4350 4350
-Wire Wire Line
 	3500 4200 3500 4350
 Connection ~ 3500 4350
@@
 	3250 4350 3500 4350
 $Comp
-L ISO1042DWVR:ISO1042DWVR U?
+L ISO1042DWVR:ISO1042DWVR U2
 U 1 1 6164A289
 P 6900 3700
-F 0 "U?" H 6900 4117 50  0000 C CNN
+F 0 "U2" H 6900 4117 50  0000 C CNN
 F 1 "ISO1042DWVR" H 6900 4026 50  0000 C CNN
 F 2 "SOIC127P1150X280-8N" H 6600 3250 50  0001 L BNN
@@
 $EndComp
 $Comp
-L +3v3_iso:+3V3_ISO #PWR?
+L +3v3_iso:+3V3_ISO #PWR0110
 U 1 1 6164CF50
 P 7850 3550
-F 0 "#PWR?" H 7850 3400 50  0001 C CNN
+F 0 "#PWR0110" H 7850 3400 50  0001 C CNN
 F 1 "+3V3_ISO" H 7865 3723 50  0000 C CNN
 F 2 "" H 7850 3550 50  0001 C CNN
@@
 $EndComp
 $Comp
-L power:+5V #PWR?
+L power:+5V #PWR0111
 U 1 1 6164E3CD
 P 6350 3550
-F 0 "#PWR?" H 6350 3400 50  0001 C CNN
+F 0 "#PWR0111" H 6350 3400 50  0001 C CNN
 F 1 "+5V" H 6365 3723 50  0000 C CNN
 F 2 "" H 6350 3550 50  0001 C CNN
@@
 $EndComp
 $Comp
-L gnd_iso:GND_ISO #PWR?
+L gnd_iso:GND_ISO #PWR0112
 U 1 1 6164EDB4
 P 7850 3850
-F 0 "#PWR?" H 7850 3600 50  0001 C CNN
+F 0 "#PWR0112" H 7850 3600 50  0001 C CNN
 F 1 "GND_ISO" H 7855 3677 50  0000 C CNN
 F 2 "" H 7850 3850 50  0001 C CNN
@@
 	5600 3550 5100 3550
 $Comp
-L power:GND #PWR?
+L power:GND #PWR0113
 U 1 1 6164F300
 P 6550 4400
-F 0 "#PWR?" H 6550 4150 50  0001 C CNN
+F 0 "#PWR0113" H 6550 4150 50  0001 C CNN
 F 1 "GND" H 6555 4227 50  0000 C CNN
 F 2 "" H 6550 4400 50  0001 C CNN
@@
 	6100 3850 6500 3850
 $Comp
-L Device:R R?
+L Device:R R5
 U 1 1 616603F3
 P 6250 4350
-F 0 "R?" H 6320 4396 50  0000 L CNN
-F 1 "R" H 6320 4305 50  0000 L CNN
-F 2 "" V 6180 4350 50  0001 C CNN
+F 0 "R5" H 6320 4396 50  0000 L CNN
+F 1 "0" H 6320 4305 50  0000 L CNN
+F 2 "Resistor_SMD:R_0805_2012Metric_Pad1.20x1.40mm_HandSolder" V 6180 4350 50  0001 C CNN
 F 3 "~" H 6250 4350 50  0001 C CNN
 	1    6250 4350
@@
 	6500 3550 6350 3550
 $Comp
-L Device:C C?
+L Device:C C12
 U 1 1 61661D34
 P 6000 3250
-F 0 "C?" H 6115 3296 50  0000 L CNN
-F 1 "C" H 6115 3205 50  0000 L CNN
-F 2 "" H 6038 3100 50  0001 C CNN
+F 0 "C12" H 6115 3296 50  0000 L CNN
+F 1 "100n" H 6115 3205 50  0000 L CNN
+F 2 "Capacitor_SMD:C_0603_1608Metric_Pad1.08x0.95mm_HandSolder" H 6038 3100 50  0001 C CNN
 F 3 "~" H 6000 3250 50  0001 C CNN
 	1    6000 3250
@@
 $EndComp
 $Comp
-L power:+5V #PWR?
+L power:+5V #PWR0114
 U 1 1 6166218D
 P 6000 3100
-F 0 "#PWR?" H 6000 2950 50  0001 C CNN
+F 0 "#PWR0114" H 6000 2950 50  0001 C CNN
 F 1 "+5V" H 6015 3273 50  0000 C CNN
 F 2 "" H 6000 3100 50  0001 C CNN
@@
 $EndComp
 $Comp
-L power:GND #PWR?
+L power:GND #PWR0115
 U 1 1 61662537
 P 6000 3400
-F 0 "#PWR?" H 6000 3150 50  0001 C CNN
+F 0 "#PWR0115" H 6000 3150 50  0001 C CNN
 F 1 "GND" H 6005 3227 50  0000 C CNN
 F 2 "" H 6000 3400 50  0001 C CNN
@@
 	1    0    0    -1
 $EndComp
-$Comp
-L Device:C C?
-U 1 1 61665BA8
-P 7850 3700
-F 0 "C?" H 7965 3746 50  0000 L CNN
-F 1 "C" H 7965 3655 50  0000 L CNN
-F 2 "" H 7888 3550 50  0001 C CNN
-F 3 "~" H 7850 3700 50  0001 C CNN
-	1    7850 3700
-	1    0    0    -1
-$EndComp
-Connection ~ 7850 3850
 Wire Wire Line
 	7850 3550 7300 3550
-Connection ~ 7850 3550
 Wire Wire Line
 	2600 3700 2850 3700
@@
 Text Notes 6150 4250 0    50   ~ 0
 STPG
+$Comp
+L Device:C C?
+U 1 1 61F47A53
+P 3500 4050
+F 0 "C?" H 3400 3650 50  0000 L CNN
+F 1 "DNP 10p" H 3400 3550 50  0000 L CNN
+F 2 "Capacitor_SMD:C_0603_1608Metric_Pad1.08x0.95mm_HandSolder" H 3538 3900 50  0001 C CNN
+F 3 "~" H 3500 4050 50  0001 C CNN
+	1    3500 4050
+	1    0    0    -1
+$EndComp
+$Comp
+L Device:C C?
+U 1 1 61F48147
+P 4100 4050
+F 0 "C?" H 3900 3650 50  0000 L CNN
+F 1 "DNP 10p" H 3900 3550 50  0000 L CNN
+F 2 "Capacitor_SMD:C_0603_1608Metric_Pad1.08x0.95mm_HandSolder" H 4138 3900 50  0001 C CNN
+F 3 "~" H 4100 4050 50  0001 C CNN
+	1    4100 4050
+	1    0    0    -1
+$EndComp
+Wire Wire Line
+	4100 4350 4350 4350
+Wire Wire Line
+	4350 4350 5000 4350
+Connection ~ 4350 4350
+Wire Wire Line
+	4350 4200 4350 4350
+Wire Wire Line
+	4350 3850 4900 3850
+Wire Wire Line
+	3950 3850 4350 3850
+Connection ~ 4350 3850
+Wire Wire Line
+	4350 3900 4350 3850
+$Comp
+L Device:C C?
+U 1 1 61F486D2
+P 4350 4050
+F 0 "C?" H 4300 3650 50  0000 L CNN
+F 1 "DNP 10p" H 4300 3550 50  0000 L CNN
+F 2 "Capacitor_SMD:C_0603_1608Metric_Pad1.08x0.95mm_HandSolder" H 4388 3900 50  0001 C CNN
+F 3 "~" H 4350 4050 50  0001 C CNN
+	1    4350 4050
+	1    0    0    -1
+$EndComp
+Wire Wire Line
+	2200 3350 2000 3350
+Wire Wire Line
+	2650 3350 2200 3350
+Connection ~ 2200 3350
+$Comp
+L Device:R R3
+U 1 1 616C53CC
+P 2200 3500
+F 0 "R3" H 2270 3546 50  0000 L CNN
+F 1 "60" H 2270 3455 50  0000 L CNN
+F 2 "Resistor_SMD:R_0805_2012Metric_Pad1.20x1.40mm_HandSolder" V 2130 3500 50  0001 C CNN
+F 3 "~" H 2200 3500 50  0001 C CNN
+	1    2200 3500
+	1    0    0    -1
+$EndComp
+Wire Wire Line
+	2000 4050 2200 4050
+$Comp
+L Device:R R?
+U 1 1 61F4B3FE
+P 2200 3900
+F 0 "R?" H 2270 3946 50  0000 L CNN
+F 1 "60" H 2270 3855 50  0000 L CNN
+F 2 "Resistor_SMD:R_0805_2012Metric_Pad1.20x1.40mm_HandSolder" V 2130 3900 50  0001 C CNN
+F 3 "~" H 2200 3900 50  0001 C CNN
+	1    2200 3900
+	1    0    0    -1
+$EndComp
+Connection ~ 2200 4050
+Wire Wire Line
+	2200 4050 2650 4050
+$Comp
+L Device:C C?
+U 1 1 61F4B7AE
+P 7850 3700
+F 0 "C?" H 7965 3746 50  0000 L CNN
+F 1 "100n" H 7965 3655 50  0000 L CNN
+F 2 "Capacitor_SMD:C_0603_1608Metric_Pad1.08x0.95mm_HandSolder" H 7888 3550 50  0001 C CNN
+F 3 "~" H 7850 3700 50  0001 C CNN
+	1    7850 3700
+	1    0    0    -1
+$EndComp
+Connection ~ 7850 3550
+Connection ~ 7850 3850
 $EndSCHEMATC

Commit message: Added most footprint requirements in HV
Parts:
- gave numbers to parts that had none: 5
Changed lines of the file:
@@
 $EndComp
 $Comp
-L +3v3_iso:+3V3_ISO #PWR0110
+L +3v3_iso:+3V3_ISO #PWR014
 U 1 1 6164CF50
 P 7850 3550
-F 0 "#PWR0110" H 7850 3400 50  0001 C CNN
+F 0 "#PWR014" H 7850 3400 50  0001 C CNN
 F 1 "+3V3_ISO" H 7865 3723 50  0000 C CNN
 F 2 "" H 7850 3550 50  0001 C CNN
@@
 $EndComp
 $Comp
-L power:+5V #PWR0111
+L power:+5V #PWR012
 U 1 1 6164E3CD
 P 6350 3550
-F 0 "#PWR0111" H 6350 3400 50  0001 C CNN
+F 0 "#PWR012" H 6350 3400 50  0001 C CNN
 F 1 "+5V" H 6365 3723 50  0000 C CNN
 F 2 "" H 6350 3550 50  0001 C CNN
@@
 $EndComp
 $Comp
-L gnd_iso:GND_ISO #PWR0112
+L gnd_iso:GND_ISO #PWR015
 U 1 1 6164EDB4
 P 7850 3850
-F 0 "#PWR0112" H 7850 3600 50  0001 C CNN
+F 0 "#PWR015" H 7850 3600 50  0001 C CNN
 F 1 "GND_ISO" H 7855 3677 50  0000 C CNN
 F 2 "" H 7850 3850 50  0001 C CNN
@@
 	5600 3550 5100 3550
 $Comp
-L power:GND #PWR0113
+L power:GND #PWR013
 U 1 1 6164F300
 P 6550 4400
-F 0 "#PWR0113" H 6550 4150 50  0001 C CNN
+F 0 "#PWR013" H 6550 4150 50  0001 C CNN
 F 1 "GND" H 6555 4227 50  0000 C CNN
 F 2 "" H 6550 4400 50  0001 C CNN
@@
 $EndComp
 $Comp
-L power:+5V #PWR0114
+L power:+5V #PWR010
 U 1 1 6166218D
 P 6000 3100
-F 0 "#PWR0114" H 6000 2950 50  0001 C CNN
+F 0 "#PWR010" H 6000 2950 50  0001 C CNN
 F 1 "+5V" H 6015 3273 50  0000 C CNN
 F 2 "" H 6000 3100 50  0001 C CNN
@@
 $EndComp
 $Comp
-L power:GND #PWR0115
+L power:GND #PWR011
 U 1 1 61662537
 P 6000 3400
-F 0 "#PWR0115" H 6000 3150 50  0001 C CNN
+F 0 "#PWR011" H 6000 3150 50  0001 C CNN
 F 1 "GND" H 6005 3227 50  0000 C CNN
 F 2 "" H 6000 3400 50  0001 C CNN
@@
 STPG
 $Comp
-L Device:C C?
+L Device:C C9
 U 1 1 61F47A53
 P 3500 4050
-F 0 "C?" H 3400 3650 50  0000 L CNN
+F 0 "C9" H 3400 3650 50  0000 L CNN
 F 1 "DNP 10p" H 3400 3550 50  0000 L CNN
 F 2 "Capacitor_SMD:C_0603_1608Metric_Pad1.08x0.95mm_HandSolder" H 3538 3900 50  0001 C CNN
@@
 $EndComp
 $Comp
-L Device:C C?
+L Device:C C10
 U 1 1 61F48147
 P 4100 4050
-F 0 "C?" H 3900 3650 50  0000 L CNN
+F 0 "C10" H 3900 3650 50  0000 L CNN
 F 1 "DNP 10p" H 3900 3550 50  0000 L CNN
 F 2 "Capacitor_SMD:C_0603_1608Metric_Pad1.08x0.95mm_HandSolder" H 4138 3900 50  0001 C CNN
@@
 	4350 3900 4350 3850
 $Comp
-L Device:C C?
+L Device:C C11
 U 1 1 61F486D2
 P 4350 4050
-F 0 "C?" H 4300 3650 50  0000 L CNN
+F 0 "C11" H 4300 3650 50  0000 L CNN
 F 1 "DNP 10p" H 4300 3550 50  0000 L CNN
 F 2 "Capacitor_SMD:C_0603_1608Metric_Pad1.08x0.95mm_HandSolder" H 4388 3900 50  0001 C CNN
@@
 	2000 4050 2200 4050
 $Comp
-L Device:R R?
+L Device:R R4
 U 1 1 61F4B3FE
 P 2200 3900
-F 0 "R?" H 2270 3946 50  0000 L CNN
+F 0 "R4" H 2270 3946 50  0000 L CNN
 F 1 "60" H 2270 3855 50  0000 L CNN
 F 2 "Resistor_SMD:R_0805_2012Metric_Pad1.20x1.40mm_HandSolder" V 2130 3900 50  0001 C CNN
@@
 	2200 4050 2650 4050
 $Comp
-L Device:C C?
+L Device:C C13
 U 1 1 61F4B7AE
 P 7850 3700
-F 0 "C?" H 7965 3746 50  0000 L CNN
+F 0 "C13" H 7965 3746 50  0000 L CNN
 F 1 "100n" H 7965 3655 50  0000 L CNN
 F 2 "Capacitor_SMD:C_0603_1608Metric_Pad1.08x0.95mm_HandSolder" H 7888 3550 50  0001 C CNN

Commit message: Updated with Mouser links for BOM
Parts:
- C10, C11, C8, C9: value DNP 10p -> DNP 10pF
- C12, C13: value 100n -> 100nF
- C7: value 10n -> 10nF
- D5: Manufacturer (none) -> ON Semiconductor; Mouser Part Number (none) -> 863-SZNUP2105LT1G; Mouser URL (none) -> https://au.mouser.com/ProductDetail/onsemi/SZNUP2105LT1G?qs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; Part Number (none) -> NUP2105L
- L2: value L_Core_Ferrite_Coupled -> 0ZCF0100AF2A; Mouser Part Number (none) -> 871-B82787C104H2; Mouser URL (none) -> https://au.mouser.com/ProductDetail/EPCOS-TDK/B82787C0104H0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; Part Number 0ZCF0100AF2A -> B82787C0104H002
- R3, R4: value 60 -> 60R
- R5: value 0 -> 0R
- U2: Manufacturer (none) -> Texas Instruments; Mouser Part Number (none) -> NOT AVAILABLE!; Mouser URL (none) -> NOT AVAILABLE!; Part Number (none) -> ISO1042DWVR
Changed lines of the file:
@@
 F 2 "Package_TO_SOT_SMD:SOT-23" H 5225 4050 50  0001 L CNN
 F 3 "http://www.onsemi.com/pub_link/Collateral/NUP2105L-D.PDF" H 5125 4225 50  0001 C CNN
+F 4 "NUP2105L" H 5000 4100 50  0001 C CNN "Part Number"
+F 5 "ON Semiconductor" H 5000 4100 50  0001 C CNN "Manufacturer"
+F 6 "863-SZNUP2105LT1G" H 5000 4100 50  0001 C CNN "Mouser Part Number"
+F 7 "https://au.mouser.com/ProductDetail/onsemi/SZNUP2105LT1G?qs=PJJcWtbOkNWqqZbXH80dfQ%3D%3D" H 5000 4100 50  0001 C CNN "Mouser URL"
 	1    5000 4100
 	1    0    0    -1
@@
 P 2450 3700
 F 0 "C7" V 2198 3700 50  0000 C CNN
-F 1 "10n" V 2289 3700 50  0000 C CNN
+F 1 "10nF" V 2289 3700 50  0000 C CNN
 F 2 "Capacitor_SMD:C_0603_1608Metric_Pad1.08x0.95mm_HandSolder" H 2488 3550 50  0001 C CNN
 F 3 "~" H 2450 3700 50  0001 C CNN
@@
 P 3750 3700
 F 0 "L2" H 3750 3981 50  0000 C CNN
-F 1 "L_Core_Ferrite_Coupled" H 3750 3890 50  0000 C CNN
+F 1 "0ZCF0100AF2A" H 3750 3890 50  0000 C CNN
 F 2 "Inductor_SMD:L_CommonModeChoke_Coilcraft_1812CAN" H 3750 3700 50  0001 C CNN
 F 3 "~" H 3750 3700 50  0001 C CNN
-F 4 "0ZCF0100AF2A" H 3750 3700 50  0001 C CNN "Part Number"
+F 4 "B82787C0104H002" H 3750 3700 50  0001 C CNN "Part Number"
 F 5 "EPCOS - TDK" H 3750 3700 50  0001 C CNN "Manufacturer"
+F 6 "871-B82787C104H2" H 3750 3700 50  0001 C CNN "Mouser Part Number"
+F 7 "https://au.mouser.com/ProductDetail/EPCOS-TDK/B82787C0104H002?qs=C9xViIFka8ni2PxKXbJHjQ%3D%3D" H 3750 3700 50  0001 C CNN "Mouser URL"
 	1    3750 3700
 	1    0    0    -1
@@
 P 3250 4050
 F 0 "C8" H 3000 3650 50  0000 L CNN
-F 1 "DNP 10p" H 3000 3550 50  0000 L CNN
+F 1 "DNP 10pF" H 3000 3550 50  0000 L CNN
 F 2 "Capacitor_SMD:C_0603_1608Metric_Pad1.08x0.95mm_HandSolder" H 3288 3900 50  0001 C CNN
 F 3 "~" H 3250 4050 50  0001 C CNN
@@
 F 2 "SOIC127P1150X280-8N" H 6600 3250 50  0001 L BNN
 F 3 "" H 6900 3700 50  0001 L BNN
+F 4 "ISO1042DWVR" H 6900 3700 50  0001 C CNN "Part Number"
+F 5 "Texas Instruments" H 6900 3700 50  0001 C CNN "Manufacturer"
+F 6 "NOT AVAILABLE!" H 6900 3700 50  0001 C CNN "Mouser Part Number"
+F 7 "NOT AVAILABLE!" H 6900 3700 50  0001 C CNN "Mouser URL"
 	1    6900 3700
 	1    0    0    -1
@@
 P 6250 4350
 F 0 "R5" H 6320 4396 50  0000 L CNN
-F 1 "0" H 6320 4305 50  0000 L CNN
+F 1 "0R" H 6320 4305 50  0000 L CNN
 F 2 "Resistor_SMD:R_0805_2012Metric_Pad1.20x1.40mm_HandSolder" V 6180 4350 50  0001 C CNN
 F 3 "~" H 6250 4350 50  0001 C CNN
@@
 P 6000 3250
 F 0 "C12" H 6115 3296 50  0000 L CNN
-F 1 "100n" H 6115 3205 50  0000 L CNN
+F 1 "100nF" H 6115 3205 50  0000 L CNN
 F 2 "Capacitor_SMD:C_0603_1608Metric_Pad1.08x0.95mm_HandSolder" H 6038 3100 50  0001 C CNN
 F 3 "~" H 6000 3250 50  0001 C CNN
@@
 P 3500 4050
 F 0 "C9" H 3400 3650 50  0000 L CNN
-F 1 "DNP 10p" H 3400 3550 50  0000 L CNN
+F 1 "DNP 10pF" H 3400 3550 50  0000 L CNN
 F 2 "Capacitor_SMD:C_0603_1608Metric_Pad1.08x0.95mm_HandSolder" H 3538 3900 50  0001 C CNN
 F 3 "~" H 3500 4050 50  0001 C CNN
@@
 P 4100 4050
 F 0 "C10" H 3900 3650 50  0000 L CNN
-F 1 "DNP 10p" H 3900 3550 50  0000 L CNN
+F 1 "DNP 10pF" H 3900 3550 50  0000 L CNN
 F 2 "Capacitor_SMD:C_0603_1608Metric_Pad1.08x0.95mm_HandSolder" H 4138 3900 50  0001 C CNN
 F 3 "~" H 4100 4050 50  0001 C CNN
@@
 P 4350 4050
 F 0 "C11" H 4300 3650 50  0000 L CNN
-F 1 "DNP 10p" H 4300 3550 50  0000 L CNN
+F 1 "DNP 10pF" H 4300 3550 50  0000 L CNN
 F 2 "Capacitor_SMD:C_0603_1608Metric_Pad1.08x0.95mm_HandSolder" H 4388 3900 50  0001 C CNN
 F 3 "~" H 4350 4050 50  0001 C CNN
@@
 P 2200 3500
 F 0 "R3" H 2270 3546 50  0000 L CNN
-F 1 "60" H 2270 3455 50  0000 L CNN
+F 1 "60R" H 2270 3455 50  0000 L CNN
 F 2 "Resistor_SMD:R_0805_2012Metric_Pad1.20x1.40mm_HandSolder" V 2130 3500 50  0001 C CNN
 F 3 "~" H 2200 3500 50  0001 C CNN
@@
 P 2200 3900
 F 0 "R4" H 2270 3946 50  0000 L CNN
-F 1 "60" H 2270 3855 50  0000 L CNN
+F 1 "60R" H 2270 3855 50  0000 L CNN
 F 2 "Resistor_SMD:R_0805_2012Metric_Pad1.20x1.40mm_HandSolder" V 2130 3900 50  0001 C CNN
 F 3 "~" H 2200 3900 50  0001 C CNN
@@
 P 7850 3700
 F 0 "C13" H 7965 3746 50  0000 L CNN
-F 1 "100n" H 7965 3655 50  0000 L CNN
+F 1 "100nF" H 7965 3655 50  0000 L CNN
 F 2 "Capacitor_SMD:C_0603_1608Metric_Pad1.08x0.95mm_HandSolder" H 7888 3550 50  0001 C CNN
 F 3 "~" H 7850 3700 50  0001 C CNN
