File: 211006_lmu_r0/file6196A5FB.sch (KiCad schematic (older format))
At the start: 7 parts

Commit message: Updated BOM and footprints for non-hv components
Parts:
- gave numbers to parts that had none: 7
Changed lines of the file:
@@
 P 8050 3400
 AR Path="/6196A5FC/6234DCC8" Ref="U?"  Part="1"
-AR Path="/61619F34/6161AC01/6234DCC8" Ref="U?"  Part="1"
+AR Path="/61619F34/6161AC01/6234DCC8" Ref="U4"  Part="1"
 AR Path="/61619F34/6161D6CD/6234DCC8" Ref="U?"  Part="1"
 AR Path="/61619F34/61F7AB68/6234DCC8" Ref="U?"  Part="1"
 AR Path="/61619F34/62061D33/6234DCC8" Ref="U?"  Part="1"
 AR Path="/61619F34/6209AB17/6234DCC8" Ref="U?"  Part="1"
-F 0 "U?" H 8050 4970 50  0000 C CNN
+F 0 "U4" H 8050 4970 50  0000 C CNN
 F 1 "LTC3300ILXE-2#PBF" H 8050 4879 50  0000 C CNN
 F 2 "QFP50P900X900X160-49N" H 8050 3400 50  0001 L BNN
@@
 	6700 4500 7150 4500
 $Comp
-L Device:R R?
+L Device:R R29
 U 1 1 61F30A1E
 P 10250 4500
-AR Path="/61619F34/6161AC01/61F30A1E" Ref="R?"  Part="1"
+AR Path="/61619F34/6161AC01/61F30A1E" Ref="R29"  Part="1"
 AR Path="/61619F34/61F7AB68/61F30A1E" Ref="R?"  Part="1"
 AR Path="/61619F34/62061D33/61F30A1E" Ref="R?"  Part="1"
 AR Path="/61619F34/6209AB17/61F30A1E" Ref="R?"  Part="1"
-F 0 "R?" H 10320 4546 50  0000 L CNN
+F 0 "R29" H 10320 4546 50  0000 L CNN
 F 1 "23.7k" H 10320 4455 50  0000 L CNN
 F 2 "" V 10180 4500 50  0001 C CNN
@@
 	10250 4300 10250 4350
 $Comp
-L Device:R R?
+L Device:R R30
 U 1 1 6234DCCA
 P 10600 4500
-AR Path="/61619F34/6161AC01/6234DCCA" Ref="R?"  Part="1"
+AR Path="/61619F34/6161AC01/6234DCCA" Ref="R30"  Part="1"
 AR Path="/61619F34/61F7AB68/6234DCCA" Ref="R?"  Part="1"
 AR Path="/61619F34/62061D33/6234DCCA" Ref="R?"  Part="1"
 AR Path="/61619F34/6209AB17/6234DCCA" Ref="R?"  Part="1"
-F 0 "R?" H 10670 4546 50  0000 L CNN
+F 0 "R30" H 10670 4546 50  0000 L CNN
 F 1 "33.2k" H 10670 4455 50  0000 L CNN
 F 2 "" V 10530 4500 50  0001 C CNN
@@
 	8950 3600 9150 3600
 $Comp
-L Device:D_Schottky D?
+L Device:D_Schottky D14
 U 1 1 6222295F
 P 9450 4900
-F 0 "D?" V 9404 4980 50  0000 L CNN
+F 0 "D14" V 9404 4980 50  0000 L CNN
 F 1 "D_Schottky" V 9495 4980 50  0000 L CNN
 F 2 "" H 9450 4900 50  0001 C CNN
@@
 C6
 $Comp
-L Device:R R?
+L Device:R R27
 U 1 1 622462AA
 P 9450 5200
-F 0 "R?" H 9520 5246 50  0000 L CNN
+F 0 "R27" H 9520 5246 50  0000 L CNN
 F 1 "R" H 9520 5155 50  0000 L CNN
 F 2 "" V 9380 5200 50  0001 C CNN
@@
 $EndComp
 $Comp
-L Device:C C?
+L Device:C C30
 U 1 1 62253C9B
 P 9800 4550
-F 0 "C?" H 9915 4596 50  0000 L CNN
+F 0 "C30" H 9915 4596 50  0000 L CNN
 F 1 "100n" H 9915 4505 50  0000 L CNN
 F 2 "" H 9838 4400 50  0001 C CNN
@@
 	9450 5500 9650 5500
 $Comp
-L Device:R R?
+L Device:R R28
 U 1 1 6234DCCE
 P 10050 3300
-AR Path="/61619F34/6161AC01/6234DCCE" Ref="R?"  Part="1"
+AR Path="/61619F34/6161AC01/6234DCCE" Ref="R28"  Part="1"
 AR Path="/61619F34/61F7AB68/6234DCCE" Ref="R?"  Part="1"
 AR Path="/61619F34/62061D33/6234DCCE" Ref="R?"  Part="1"
 AR Path="/61619F34/6209AB17/6234DCCE" Ref="R?"  Part="1"
-F 0 "R?" H 10120 3346 50  0000 L CNN
+F 0 "R28" H 10120 3346 50  0000 L CNN
 F 1 "1M" H 10120 3255 50  0000 L CNN
 F 2 "" V 9980 3300 50  0001 C CNN

Commit message: Added most footprint requirements in HV
Parts:
- C30: footprint (none) -> Capacitor_SMD:C_0603_1608Metric_Pad1.08x0.95mm_HandSolder
- R27: value R -> 6.81; footprint (none) -> Resistor_SMD:R_0603_1608Metric_Pad0.98x0.95mm_HandSolder
- R28, R29, R30: footprint (none) -> Resistor_SMD:R_0603_1608Metric_Pad0.98x0.95mm_HandSolder
Changed lines of the file:
@@
 F 0 "R29" H 10320 4546 50  0000 L CNN
 F 1 "23.7k" H 10320 4455 50  0000 L CNN
-F 2 "" V 10180 4500 50  0001 C CNN
+F 2 "Resistor_SMD:R_0603_1608Metric_Pad0.98x0.95mm_HandSolder" V 10180 4500 50  0001 C CNN
 F 3 "~" H 10250 4500 50  0001 C CNN
 	1    10250 4500
@@
 F 0 "R30" H 10670 4546 50  0000 L CNN
 F 1 "33.2k" H 10670 4455 50  0000 L CNN
-F 2 "" V 10530 4500 50  0001 C CNN
+F 2 "Resistor_SMD:R_0603_1608Metric_Pad0.98x0.95mm_HandSolder" V 10530 4500 50  0001 C CNN
 F 3 "~" H 10600 4500 50  0001 C CNN
 	1    10600 4500
@@
 P 9450 5200
 F 0 "R27" H 9520 5246 50  0000 L CNN
-F 1 "R" H 9520 5155 50  0000 L CNN
-F 2 "" V 9380 5200 50  0001 C CNN
+F 1 "6.81" H 9520 5155 50  0000 L CNN
+F 2 "Resistor_SMD:R_0603_1608Metric_Pad0.98x0.95mm_HandSolder" V 9380 5200 50  0001 C CNN
 F 3 "~" H 9450 5200 50  0001 C CNN
 	1    9450 5200
@@
 F 0 "C30" H 9915 4596 50  0000 L CNN
 F 1 "100n" H 9915 4505 50  0000 L CNN
-F 2 "" H 9838 4400 50  0001 C CNN
+F 2 "Capacitor_SMD:C_0603_1608Metric_Pad1.08x0.95mm_HandSolder" H 9838 4400 50  0001 C CNN
 F 3 "~" H 9800 4550 50  0001 C CNN
 	1    9800 4550
@@
 F 0 "R28" H 10120 3346 50  0000 L CNN
 F 1 "1M" H 10120 3255 50  0000 L CNN
-F 2 "" V 9980 3300 50  0001 C CNN
+F 2 "Resistor_SMD:R_0603_1608Metric_Pad0.98x0.95mm_HandSolder" V 9980 3300 50  0001 C CNN
 F 3 "~" H 10050 3300 50  0001 C CNN
 	1    10050 3300

Commit message: Cleaned up last components missing footprint refs
Parts:
- D14: footprint (none) -> Diode_SMD:D_SOD-123F; Part Number (none) -> CMMSH2-40
Changed lines of the file:
@@
 F 0 "D14" V 9404 4980 50  0000 L CNN
 F 1 "D_Schottky" V 9495 4980 50  0000 L CNN
-F 2 "" H 9450 4900 50  0001 C CNN
+F 2 "Diode_SMD:D_SOD-123F" H 9450 4900 50  0001 C CNN
 F 3 "~" H 9450 4900 50  0001 C CNN
+F 4 "CMMSH2-40" V 9450 4900 50  0001 C CNN "Part Number"
 	1    9450 4900
 	0    1    1    0

Commit message: Updated with Mouser links for BOM
Parts:
- C30: value 100n -> 100nF
- D14: value D_Schottky -> CMMSH2-40; Manufacturer (none) -> Central Semiconductor; Mouser Part Number (none) -> 610-CMMSH2-40TR; Mouser URL (none) -> https://au.mouser.com/ProductDetail/Central-Semiconductor/C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
- R27: value 6.81 -> 6.81R
- R28: value 1M -> 1MR
- R29: value 23.7k -> 23.7kR
- R30: value 33.2k -> 33.2kR
- U4: MANUFACTURER Linear Technology -> (none); MP LTC3300ILXE-2#PBF -> (none); Manufacturer (none) -> Linear Technology; Mouser Part Number (none) -> NOT AVAILABLE!; Mouser URL (none) -> NOT AVAILABLE!; PACKAGE LQFP-48 Linear Technology -> (none); Part Number (none) -> LTC3300ILXE-2#PBF; STANDARD IPC-7351B -> (none)
Changed lines of the file:
@@
 AR Path="/61619F34/62061D33/6234DCC8" Ref="U?"  Part="1"
 AR Path="/61619F34/6209AB17/6234DCC8" Ref="U?"  Part="1"
-F 0 "U4" H 8050 4970 50  0000 C CNN
+AR Path="/61619F34/61F88CA4/6234DCC8" Ref="U5"  Part="1"
+F 0 "U5" H 8050 4970 50  0000 C CNN
 F 1 "LTC3300ILXE-2#PBF" H 8050 4879 50  0000 C CNN
 F 2 "QFP50P900X900X160-49N" H 8050 3400 50  0001 L BNN
 F 3 "" H 8050 3400 50  0001 L BNN
-F 4 "LQFP-48 Linear Technology" H 8050 3400 50  0001 L BNN "PACKAGE"
+F 4 "" H 8050 3400 50  0001 L BNN "PACKAGE"
 F 5 "29275" H 8050 3400 50  0001 L BNN "SNAPEDA_PACKAGE_ID"
-F 6 "IPC-7351B" H 8050 3400 50  0001 L BNN "STANDARD"
+F 6 "" H 8050 3400 50  0001 L BNN "STANDARD"
 F 7 "10.07 USD" H 8050 3400 50  0001 L BNN "PRICE"
-F 8 "LTC3300ILXE-2#PBF" H 8050 3400 50  0001 L BNN "MP"
+F 8 "" H 8050 3400 50  0001 L BNN "MP"
 F 9 "A" H 8050 3400 50  0001 L BNN "PARTREV"
-F 10 "Linear Technology" H 8050 3400 50  0001 L BNN "MANUFACTURER"
+F 10 "" H 8050 3400 50  0001 L BNN "MANUFACTURER"
 F 11 "Unavailable" H 8050 3400 50  0001 L BNN "AVAILABILITY"
+F 12 "Linear Technology" H 8050 3400 50  0001 C CNN "Manufacturer"
+F 13 "LTC3300ILXE-2#PBF" H 8050 3400 50  0001 C CNN "Part Number"
+F 14 "NOT AVAILABLE!" H 8050 3400 50  0001 C CNN "Mouser Part Number"
+F 15 "NOT AVAILABLE!" H 8050 3400 50  0001 C CNN "Mouser URL"
 	1    8050 3400
 	1    0    0    -1
@@
 AR Path="/61619F34/62061D33/61F30A1E" Ref="R?"  Part="1"
 AR Path="/61619F34/6209AB17/61F30A1E" Ref="R?"  Part="1"
-F 0 "R29" H 10320 4546 50  0000 L CNN
-F 1 "23.7k" H 10320 4455 50  0000 L CNN
+AR Path="/61619F34/61F88CA4/61F30A1E" Ref="R129"  Part="1"
+F 0 "R129" H 10320 4546 50  0000 L CNN
+F 1 "23.7kR" H 10320 4455 50  0000 L CNN
 F 2 "Resistor_SMD:R_0603_1608Metric_Pad0.98x0.95mm_HandSolder" V 10180 4500 50  0001 C CNN
 F 3 "~" H 10250 4500 50  0001 C CNN
@@
 AR Path="/61619F34/62061D33/6234DCCA" Ref="R?"  Part="1"
 AR Path="/61619F34/6209AB17/6234DCCA" Ref="R?"  Part="1"
-F 0 "R30" H 10670 4546 50  0000 L CNN
-F 1 "33.2k" H 10670 4455 50  0000 L CNN
+AR Path="/61619F34/61F88CA4/6234DCCA" Ref="R130"  Part="1"
+F 0 "R130" H 10670 4546 50  0000 L CNN
+F 1 "33.2kR" H 10670 4455 50  0000 L CNN
 F 2 "Resistor_SMD:R_0603_1608Metric_Pad0.98x0.95mm_HandSolder" V 10530 4500 50  0001 C CNN
 F 3 "~" H 10600 4500 50  0001 C CNN
@@
 U 1 1 6222295F
 P 9450 4900
-F 0 "D14" V 9404 4980 50  0000 L CNN
-F 1 "D_Schottky" V 9495 4980 50  0000 L CNN
+AR Path="/61619F34/6161AC01/6222295F" Ref="D14"  Part="1"
+AR Path="/61619F34/61F88CA4/6222295F" Ref="D27"  Part="1"
+F 0 "D27" V 9404 4980 50  0000 L CNN
+F 1 "CMMSH2-40" V 9495 4980 50  0000 L CNN
 F 2 "Diode_SMD:D_SOD-123F" H 9450 4900 50  0001 C CNN
 F 3 "~" H 9450 4900 50  0001 C CNN
 F 4 "CMMSH2-40" V 9450 4900 50  0001 C CNN "Part Number"
+F 5 "Central Semiconductor" H 9450 4900 50  0001 C CNN "Manufacturer"
+F 6 "610-CMMSH2-40TR" H 9450 4900 50  0001 C CNN "Mouser Part Number"
+F 7 "https://au.mouser.com/ProductDetail/Central-Semiconductor/CMMSH2-40-TR-PBFREE?qs=OlC7AqGiEDmeZ8mWO7SnhA%3D%3D" H 9450 4900 50  0001 C CNN "Mouser URL"
 	1    9450 4900
 	0    1    1    0
@@
 U 1 1 622462AA
 P 9450 5200
-F 0 "R27" H 9520 5246 50  0000 L CNN
-F 1 "6.81" H 9520 5155 50  0000 L CNN
+AR Path="/61619F34/6161AC01/622462AA" Ref="R27"  Part="1"
+AR Path="/61619F34/61F88CA4/622462AA" Ref="R127"  Part="1"
+F 0 "R127" H 9520 5246 50  0000 L CNN
+F 1 "6.81R" H 9520 5155 50  0000 L CNN
 F 2 "Resistor_SMD:R_0603_1608Metric_Pad0.98x0.95mm_HandSolder" V 9380 5200 50  0001 C CNN
 F 3 "~" H 9450 5200 50  0001 C CNN
@@
 U 1 1 62253C9B
 P 9800 4550
-F 0 "C30" H 9915 4596 50  0000 L CNN
-F 1 "100n" H 9915 4505 50  0000 L CNN
+AR Path="/61619F34/6161AC01/62253C9B" Ref="C30"  Part="1"
+AR Path="/61619F34/61F88CA4/62253C9B" Ref="C103"  Part="1"
+F 0 "C103" H 9915 4596 50  0000 L CNN
+F 1 "100nF" H 9915 4505 50  0000 L CNN
 F 2 "Capacitor_SMD:C_0603_1608Metric_Pad1.08x0.95mm_HandSolder" H 9838 4400 50  0001 C CNN
 F 3 "~" H 9800 4550 50  0001 C CNN
@@
 AR Path="/61619F34/62061D33/6234DCCE" Ref="R?"  Part="1"
 AR Path="/61619F34/6209AB17/6234DCCE" Ref="R?"  Part="1"
-F 0 "R28" H 10120 3346 50  0000 L CNN
-F 1 "1M" H 10120 3255 50  0000 L CNN
+AR Path="/61619F34/61F88CA4/6234DCCE" Ref="R128"  Part="1"
+F 0 "R128" H 10120 3346 50  0000 L CNN
+F 1 "1MR" H 10120 3255 50  0000 L CNN
 F 2 "Resistor_SMD:R_0603_1608Metric_Pad0.98x0.95mm_HandSolder" V 9980 3300 50  0001 C CNN
 F 3 "~" H 10050 3300 50  0001 C CNN

Commit message: minor BOM changes
Parts:
- U4: AVAILABILITY Unavailable -> (none)
Changed lines of the file:
@@
 F 9 "A" H 8050 3400 50  0001 L BNN "PARTREV"
 F 10 "" H 8050 3400 50  0001 L BNN "MANUFACTURER"
-F 11 "Unavailable" H 8050 3400 50  0001 L BNN "AVAILABILITY"
+F 11 "" H 8050 3400 50  0001 L BNN "AVAILABILITY"
 F 12 "Linear Technology" H 8050 3400 50  0001 C CNN "Manufacturer"
 F 13 "LTC3300ILXE-2#PBF" H 8050 3400 50  0001 C CNN "Part Number"
