File: 211006_lmu_r0/211006_lmu_r0.kicad_pcb (KiCad board)
At the start: 4 copper layers, 67.6 x 31.8 mm, 727 parts, among them J1 Conn_02x03_Odd_Even, J10 Conn_01x02, J11 Conn_ARM_JTAG_SWD_10, J12 Conn_01x03, J2 Conn_02x03_Odd_Even, J5 Conn_01x03, J6 Conn_01x03, J7 Conn_01x02, J8 Conn_01x02, J9 Conn_01x02, K1 G5V-2, Q1 CZT5551, Q10 SiR882DP, Q11 BSS308PE, Q12 SiR882DP, Q13 SiR882DP, Q14 BSS308PE, Q15 SiR882DP, Q16 SiR882DP, Q17 BSS308PE, Q18 SiR882DP, Q19 SiR882DP, Q2 BSS308PE, Q20 BSS308PE, Q21 SiR882DP, Q22 SiR882DP, Q23 BSS308PE, Q24 SiR882DP, Q25 SiR882DP, Q26 BSS308PE, Q27 SiR882DP, Q28 SiR882DP, Q29 BSS308PE, Q3 SiR882DP, Q30 SiR882DP, Q31 SiR882DP, Q32 BSS308PE, Q33 SiR882DP, Q34 SiR882DP, Q35 BSS308PE, Q36 SiR882DP, Q37 SiR882DP, Q38 BC817, Q4 SiR882DP, Q5 BSS308PE, Q6 SiR882DP, Q7 SiR882DP, Q8 BSS308PE, Q9 SiR882DP, SW1 SW_Push, SW2 SW_SPST, T1 750312504, T10 750312504, T11 750312504, T12 750312504, T2 750312504, T3 750312504, T4 750312504, T5 750312504, T6 750312504, T7 750312504, T8 750312504, T9 750312504, U1 R-78C5.0-1.0, U2 ISO1042DWVR, U3 LTC6811HG-2#PBF, U4 LTC3300ILXE-2#PBF, U5 LTC3300ILXE-2#PBF, U6 ISO7761DBQ, U7 ISO7761DBQ, U8 ISO7761DBQ, U9 STM32F103C8Tx, Y1 16MHz

Commit message: Close to completing front side of 4-module board
Parts:
- moved C49 198.0 mm to (159.8, 64.0), turned to 90 degrees
- moved R50 196.9 mm to (165.9, 69.3), turned to 90 degrees
- moved R48 195.0 mm to (141.8, 68.8), turned to 180 degrees
- moved C43 194.8 mm to (137.8, 64.0), turned to 90 degrees
- moved Q7 190.4 mm to (156.8, 83.0), turned to 180 degrees
- moved C44 187.8 mm to (140.3, 64.0), turned to 90 degrees
- moved C51 187.6 mm to (162.3, 64.0), turned to 90 degrees
- moved D17 185.7 mm to (136.8, 71.4), turned to -90 degrees
- moved C46 182.9 mm to (142.8, 64.0), turned to 90 degrees
- moved T2 181.6 mm to (151.3, 70.7), turned to -90 degrees
- moved Q5 181.0 mm to (136.4, 77.8), turned to -90 degrees
- moved C52 179.2 mm to (164.8, 64.0), turned to 90 degrees
- moved C53 178.0 mm to (172.7, 76.4), turned to 90 degrees
- moved C54 176.1 mm to (175.1, 76.5), turned to 90 degrees
- moved C50 175.9 mm to (162.0, 68.7), turned to -90 degrees
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Routing:
- net /Balance Interface V3/Upper Active Balance Group/ACTIVE_TAP5: track 28.7 -> 61.5 mm
- net Net-(Q7-Pad1): track 0.00 -> 23.3 mm, vias 0 -> 4
- net Net-(T2-Pad4): track 0.00 -> 17.4 mm
- net /Balance Interface V3/C12: track 5.73 -> 18.6 mm
- net /Balance Interface V3/Upper Active Balance Group/ACTIVE_TAP4: track 0.00 -> 11.5 mm
- net GND: track 9.45 -> 18.8 mm
- net /Balance Interface V3/Upper Active Balance Group/Active_Passive_Balance_Filter/BOOST: track 15.8 -> 24.3 mm
- net Net-(C47-Pad1): track 0.00 -> 7.06 mm
- net Net-(C48-Pad1): track 0.00 -> 5.08 mm
- net Net-(C35-Pad1): track 9.05 -> 13.4 mm
- net Net-(D18-Pad2): track 0.00 -> 3.04 mm
- net Net-(Q6-Pad1): track 0.00 -> 2.54 mm
- net Net-(Q4-Pad1): track 24.1 -> 25.6 mm
Other:
- outline, holes or cut-outs redrawn

Commit message: Installed and tested Replicate Layout plugin
Next to do: Finalise design of singular balancing module and then start layout of large board.
Things to update:
- Change orientation of FETs underneath coil, add vias and copper pour on opposite side for heat dissipation
- standardise all via stitching of all large traces to grid of small vias
- Route last few traces
- Ensure all traces coming of bottom side of "module" - will help with routing all traces once modules are replicated
- Ensure no acid traps in routing layout, check all layers used
Parts:
- moved C73 249.4 mm to (173.9, 105.7), turned to 90 degrees
- moved R74 248.2 mm to (180.0, 111.0), turned to 90 degrees
- moved R72 246.9 mm to (155.9, 110.5), turned to 180 degrees
- moved C67 246.8 mm to (151.9, 105.7), turned to 90 degrees
- moved R77 241.8 mm to (173.6, 119.1), turned to -90 degrees
- moved Q13 241.2 mm to (170.9, 124.7), turned to 180 degrees
- moved TP67 241.1 mm to (173.6, 116.5)
- moved C68 239.8 mm to (154.4, 105.7), turned to 90 degrees
- moved C75 239.1 mm to (176.4, 105.7), turned to 90 degrees
- moved D21 237.5 mm to (150.9, 113.1), turned to -90 degrees
- moved C70 235.0 mm to (156.9, 105.7), turned to 90 degrees
- moved C71 233.6 mm to (157.9, 116.3), turned to 90 degrees
- moved Q11 233.0 mm to (150.3, 119.4), turned to -90 degrees
- moved T4 232.9 mm to (165.4, 112.3), turned to -90 degrees
- moved TP68 232.5 mm to (177.2, 122.0)
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Routing:
- net /Balance Interface V3/Upper Active Balance Group/ACTIVE_TAP3: track 0.00 -> 238.5 mm, vias 0 -> 8
- net /Balance Interface V3/Upper Active Balance Group/ACTIVE_TAP4: track 11.5 -> 171.1 mm, vias 0 -> 6
- net /Balance Interface V3/Upper Active Balance Group/ACTIVE_TAP2: track 0.00 -> 109.4 mm, vias 0 -> 4
- net /Balance Interface V3/Upper Active Balance Group/Active_Passive_Balance_Filter/BOOST: track 24.3 -> 103.2 mm
- net /Balance Interface V3/Upper Active Balance Group/ACTIVE_TAP5: track 61.5 -> 127.9 mm, vias 2 -> 4
- net 0V_ISO: track 11.0 -> 66.3 mm
- net Net-(Q13-Pad1): track 0.00 -> 51.2 mm, vias 0 -> 8
- net Net-(Q10-Pad1): track 0.00 -> 51.2 mm, vias 0 -> 8
- net /Balance Interface V3/S10: track 0.00 -> 49.0 mm
- net /Balance Interface V3/C9: track 0.00 -> 49.0 mm
- net GND: track 18.8 -> 66.1 mm
- net /Balance Interface V3/Upper Active Balance Group/SI4: track 0.00 -> 39.3 mm, vias 0 -> 4
- net /Balance Interface V3/Upper Active Balance Group/SI3: track 0.00 -> 39.3 mm, vias 0 -> 4
- net Net-(T4-Pad4): track 0.00 -> 34.8 mm
- net Net-(T3-Pad4): track 0.00 -> 34.8 mm
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
Commit message: Balance module design finalised
Parts:
- moved C84 173.4 mm to (365.7, 203.3), turned to 90 degrees
- moved C109 173.1 mm to (209.3, 205.2), turned to 90 degrees
- moved C121 173.1 mm to (261.4, 266.5), turned to 90 degrees
- moved C133 173.1 mm to (209.3, 297.1), turned to 90 degrees
- moved C145 173.1 mm to (313.6, 205.2), turned to 90 degrees
- moved C157 173.1 mm to (261.4, 235.9), turned to 90 degrees
- moved C169 173.1 mm to (209.3, 266.5), turned to 90 degrees
- moved C96 173.1 mm to (209.3, 327.8), turned to 90 degrees
- moved C45 68.5 mm to (216.6, 81.9), turned to 0 degrees
- moved TP46 66.9 mm to (233.4, 63.1)
- moved R62 66.5 mm to (103.7, 171.1)
- moved R74 66.5 mm to (152.5, 171.7)
- moved TP38 65.9 mm to (208.8, 81.1)
- moved R52 65.5 mm to (231.8, 72.6)
- moved TP37 65.4 mm to (205.8, 81.5)
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Routing:
- net /Balance Interface V3/Upper Active Balance Group/ACTIVE_TAP3: track 238.5 -> 0.00 mm, vias 8 -> 0
- net /Balance Interface V3/Upper Active Balance Group/ACTIVE_TAP4: track 171.1 -> 0.00 mm, vias 6 -> 0
- net /Balance Interface V3/Upper Active Balance Group/ACTIVE_TAP2: track 109.4 -> 0.00 mm, vias 4 -> 0
- net /Balance Interface V3/Upper Active Balance Group/ACTIVE_TAP5: track 127.9 -> 54.9 mm, vias 4 -> 2
- net /Balance Interface V3/Upper Active Balance Group/Active_Passive_Balance_Filter/BOOST: track 103.2 -> 30.4 mm
- net Net-(Q13-Pad1): track 51.2 -> 0.00 mm, vias 8 -> 0
- net Net-(Q10-Pad1): track 51.2 -> 0.00 mm, vias 8 -> 0
- net 0V_ISO: track 66.3 -> 15.0 mm
- net /Balance Interface V3/S10: track 49.0 -> 0.00 mm
- net /Balance Interface V3/C9: track 49.0 -> 0.00 mm
- net Net-(Q7-Pad1): track 48.9 -> 0.00 mm, vias 8 -> 0
- net /Balance Interface V3/Upper Active Balance Group/SI4: track 39.3 -> 0.00 mm, vias 4 -> 0
- net /Balance Interface V3/Upper Active Balance Group/SI3: track 39.3 -> 0.00 mm, vias 4 -> 0
- net Net-(T4-Pad4): track 34.8 -> 0.00 mm
- net Net-(T3-Pad4): track 34.8 -> 0.00 mm
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- added copper zone on B.Cu, net Net-(C35-Pad1)
- added copper zone on F.Cu, net Net-(C35-Pad1)
- added copper zone on B.Cu, net Net-(C36-Pad1)
- added copper zone on F.Cu, net Net-(C36-Pad1)
Other:
- board size 67.6 x 31.8 mm -> 344.7 x 286 mm

Commit message: Fixed missed component in module
Parts:
- moved T6 312.7 mm to (215.4, 114.2), turned to -90 degrees
- moved C43 278.6 mm to (-70.8, 51.1)
- moved C44 278.6 mm to (-68.3, 51.1)
- moved C45 278.6 mm to (-61.8, 73.5)
- moved C46 278.6 mm to (-65.8, 51.1)
- moved C47 278.6 mm to (-64.8, 61.7)
- moved C49 278.6 mm to (-48.8, 51.1)
- moved C50 278.6 mm to (-46.5, 55.8)
- moved C51 278.6 mm to (-46.3, 51.1)
- moved C52 278.6 mm to (-43.8, 51.1)
- moved C53 278.6 mm to (-46.2, 60.6)
- moved C54 278.6 mm to (-44.6, 60.6)
- moved D17 278.6 mm to (-71.8, 58.5)
- moved D18 278.6 mm to (-66.6, 58.8)
- moved Q5 278.6 mm to (-72.3, 64.8)
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Routing:
- net Net-(C36-Pad1): track 1.50 -> 2.94 mm, vias 9 -> 10
- net Net-(C36-Pad2): track 3.05 -> 4.26 mm
- net /Balance Interface V3/Upper Active Balance Group/Active_Passive_Balance_Filter/BOOST: track 30.4 -> 31.5 mm
Other:
- board size 344.7 x 286 mm -> 240 x 130 mm

Commit message: Module replication successful
Parts:
- moved C128 363.0 mm to (223.8, 45.0), turned to 90 degrees
- moved C129 362.5 mm to (226.3, 45.0), turned to 90 degrees
- moved C131 362.0 mm to (228.8, 45.0), turned to 90 degrees
- moved C134 359.7 mm to (245.8, 45.0), turned to 90 degrees
- moved C136 359.5 mm to (248.3, 45.0), turned to 90 degrees
- moved C137 359.3 mm to (250.8, 45.0), turned to 90 degrees
- moved R160 355.5 mm to (227.8, 49.8), turned to 180 degrees
- moved TP123 354.4 mm to (249.6, 48.5), turned to 0 degrees
- moved D32 352.9 mm to (222.8, 52.4), turned to -90 degrees
- moved C135 352.9 mm to (248.1, 49.7), turned to -90 degrees
- moved TP124 352.5 mm to (250.6, 49.9), turned to 0 degrees
- moved R163 352.2 mm to (245.8, 50.4), turned to 90 degrees
- moved D33 351.4 mm to (228.0, 52.6), turned to 0 degrees
- moved T9 351.3 mm to (237.3, 51.6), turned to -90 degrees
- moved R166 349.5 mm to (248.6, 52.0), turned to 180 degrees
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Routing:
- net GND: track 34.4 -> 330.0 mm, vias 0 -> 4
- net /Balance Interface V3/sheet61F88C83/V-: track 0.00 -> 261.5 mm, vias 0 -> 2
- net /Balance Interface V3/sheet61F88C83/Active_Passive_Balance_Filter/BOOST: track 0.00 -> 188.9 mm
- net 0V_ISO: track 15.3 -> 183.5 mm
- net /Balance Interface V3/Upper Active Balance Group/Active_Passive_Balance_Filter/BOOST: track 31.5 -> 188.9 mm
- net /Balance Interface V3/sheet61F88C83/ACTIVE_TAP5: track 0.00 -> 123.3 mm, vias 0 -> 4
- net /Balance Interface V3/sheet61F88C83/ACTIVE_TAP4: track 0.00 -> 123.3 mm, vias 0 -> 4
- net /Balance Interface V3/Upper Active Balance Group/ACTIVE_TAP2: track 0.00 -> 123.3 mm, vias 0 -> 4
- net /Balance Interface V3/sheet61F88C83/ACTIVE_TAP3: track 0.00 -> 123.3 mm, vias 0 -> 4
- net /Balance Interface V3/Upper Active Balance Group/ACTIVE_TAP3: track 0.00 -> 123.3 mm, vias 0 -> 4
- net /Balance Interface V3/Upper Active Balance Group/ACTIVE_TAP1: track 0.00 -> 123.3 mm, vias 0 -> 4
- net /Balance Interface V3/sheet61F88C83/ACTIVE_TAP2: track 0.00 -> 123.3 mm, vias 0 -> 4
- net /Balance Interface V3/sheet61F88C83/ACTIVE_TAP1: track 0.00 -> 123.3 mm, vias 0 -> 4
- net /Balance Interface V3/Upper Active Balance Group/ACTIVE_TAP4: track 0.00 -> 123.3 mm, vias 0 -> 4
- net /Balance Interface V3/Upper Active Balance Group/ACTIVE_TAP5: track 54.9 -> 123.3 mm, vias 2 -> 4
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- added copper zone on B.Cu, net Net-(C108-Pad1)
- added copper zone on F.Cu, net Net-(C108-Pad1)
- added copper zone on B.Cu, net Net-(C109-Pad1)
- added copper zone on F.Cu, net Net-(C109-Pad1)
- added copper zone on B.Cu, net Net-(C120-Pad1)
- added copper zone on F.Cu, net Net-(C120-Pad1)
- added copper zone on B.Cu, net Net-(C121-Pad1)
- added copper zone on F.Cu, net Net-(C121-Pad1)
- added copper zone on B.Cu, net Net-(C132-Pad1)
- added copper zone on F.Cu, net Net-(C132-Pad1)
- added copper zone on B.Cu, net Net-(C133-Pad1)
- added copper zone on F.Cu, net Net-(C133-Pad1)
- added copper zone on B.Cu, net Net-(C144-Pad1)
- added copper zone on F.Cu, net Net-(C144-Pad1)
- added copper zone on B.Cu, net Net-(C145-Pad1)
- added copper zone on F.Cu, net Net-(C145-Pad1)
- added copper zone on B.Cu, net Net-(C156-Pad1)
- added copper zone on F.Cu, net Net-(C156-Pad1)
- added copper zone on B.Cu, net Net-(C157-Pad1)
- added copper zone on F.Cu, net Net-(C157-Pad1)
- added copper zone on B.Cu, net Net-(C168-Pad1)
- added copper zone on F.Cu, net Net-(C168-Pad1)
- added copper zone on B.Cu, net Net-(C169-Pad1)
- added copper zone on F.Cu, net Net-(C169-Pad1)
- added copper zone on B.Cu, net Net-(C47-Pad1)
- added copper zone on F.Cu, net Net-(C47-Pad1)
- added copper zone on B.Cu, net Net-(C48-Pad1)
- added copper zone on F.Cu, net Net-(C48-Pad1)
- added copper zone on B.Cu, net Net-(C59-Pad1)
- added copper zone on F.Cu, net Net-(C59-Pad1)
- added copper zone on B.Cu, net Net-(C60-Pad1)
- added copper zone on F.Cu, net Net-(C60-Pad1)
- added copper zone on B.Cu, net Net-(C71-Pad1)
- added copper zone on F.Cu, net Net-(C71-Pad1)
- added copper zone on B.Cu, net Net-(C72-Pad1)
- added copper zone on F.Cu, net Net-(C72-Pad1)
- added copper zone on B.Cu, net Net-(C83-Pad1)
- added copper zone on F.Cu, net Net-(C83-Pad1)
- added copper zone on B.Cu, net Net-(C84-Pad1)
- added copper zone on F.Cu, net Net-(C84-Pad1)
- added copper zone on B.Cu, net Net-(C95-Pad1)
- added copper zone on F.Cu, net Net-(C95-Pad1)
- added copper zone on B.Cu, net Net-(C96-Pad1)
- added copper zone on F.Cu, net Net-(C96-Pad1)
