File: 211006_lmu_r0/211006_lmu_r0.kicad_pcb (KiCad board)
At the start: 4 copper layers, 250 x 145.5 mm, 740 parts, among them IC1 ADS7038QRTERQ1, J1 Conn_02x03_Odd_Even, J10 Conn_01x02, J11 Conn_ARM_JTAG_SWD_10, J12 Conn_01x03, J13 Conn_02x03_Odd_Even, J14 Conn_01x02, J15 Conn_01x02, J16 Conn_01x02, J17 Conn_01x02, J18 Conn_01x02, J19 Conn_01x02, J2 Conn_02x03_Odd_Even, J20 Conn_01x02, J21 Conn_01x02, J22 Conn_01x02, J23 Conn_01x02, J24 Conn_01x02, J25 Conn_01x02, J3 Conn_02x08_Odd_Even, J4 Conn_01x02, J5 Conn_01x03, J6 Conn_01x03, J7 Conn_01x02, J8 Conn_01x02, J9 Conn_01x02, K1 G5V-2, Q1 CZT5551, Q10 SiR882DP, Q11 BSS308PE, Q12 SiR882DP, Q13 SiR882DP, Q14 BSS308PE, Q15 SiR882DP, Q16 SiR882DP, Q17 BSS308PE, Q18 SiR882DP, Q19 SiR882DP, Q2 BSS308PE, Q20 BSS308PE, Q21 SiR882DP, Q22 SiR882DP, Q23 BSS308PE, Q24 SiR882DP, Q25 SiR882DP, Q26 BSS308PE, Q27 SiR882DP, Q28 SiR882DP, Q29 BSS308PE, Q3 SiR882DP, Q30 SiR882DP, Q31 SiR882DP, Q32 BSS308PE, Q33 SiR882DP, Q34 SiR882DP, Q35 BSS308PE, Q36 SiR882DP, Q37 SiR882DP, Q38 BC817, Q4 SiR882DP, Q5 BSS308PE, Q6 SiR882DP, Q7 SiR882DP, Q8 BSS308PE, Q9 SiR882DP, SW1 SW_Push, T1 750312504, T10 750312504, T11 750312504, T12 750312504, T2 750312504, T3 750312504, T4 750312504, T5 750312504, T6 750312504, T7 750312504, T8 750312504, T9 750312504, U1 R-78C5.0-1.0, U2 ISO1042DWVR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

Commit message: progress on PCB
Parts:
- R128: moved to B.Cu
- moved C137 268.4 mm to (189.4, 105.8), turned to 180 degrees
- moved C136 267.7 mm to (189.4, 108.3), turned to 180 degrees
- moved C134 267.0 mm to (189.4, 110.8), turned to 180 degrees
- moved C131 263.5 mm to (189.4, 127.5), turned to 180 degrees
- moved C129 263.1 mm to (189.4, 130.0), turned to 180 degrees
- moved C128 262.9 mm to (189.4, 132.5), turned to 180 degrees
- moved TP123 261.7 mm to (194.1, 106.4), turned to 90 degrees
- moved C135 261.2 mm to (194.1, 108.2), turned to 0 degrees
- moved R163 259.7 mm to (194.7, 110.5), turned to 180 degrees
- moved TP124 259.4 mm to (196.0, 105.4), turned to 90 degrees
- moved R166 258.1 mm to (196.4, 107.7), turned to -90 degrees
- moved R160 256.7 mm to (194.1, 128.4), turned to -90 degrees
- moved T9 255.7 mm to (196.0, 119.0), turned to 0 degrees
- moved C139 255.1 mm to (198.9, 106.3), turned to 180 degrees
- moved C138 254.6 mm to (198.9, 107.9), turned to 180 degrees
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Routing:
- net /Balance Interface V3/Upper Active Balance Group/ACTIVE_TAP5: track 124.3 -> 232.2 mm, vias 4 -> 7
- net /Balance Interface V3/V+: track 69.5 -> 168.8 mm, vias 2 -> 4
- net /Balance Interface V3/Upper Active Balance Group/ACTIVE_TAP4: track 124.3 -> 173.8 mm
- net /Balance Interface V3/VREG_LOWER: track 7.03 -> 27.8 mm, vias 5 -> 2
- net /Balance Interface V3/LOWER_ADDRESS/A1: track 1.25 -> 18.4 mm, vias 1 -> 2
- net /Balance Interface V3/LOWER_ADDRESS/A3: track 1.34 -> 17.7 mm, vias 1 -> 2
- net /Balance Interface V3/LOWER_ADDRESS/A0: track 3.51 -> 19.5 mm
- net /Balance Interface V3/LOWER_ADDRESS/A2: track 3.51 -> 17.8 mm
- net /Balance Interface V3/VREG_UPPER: track 32.6 -> 38.0 mm
- net /Balance Interface V3/Lower Active Balance Group/V-: track 144.3 -> 149.4 mm, vias 14 -> 15
- net /Balance Interface V3/Lower Active Balance Group/C6: track 0.00 -> 4.76 mm
- net Net-(C103-Pad2): track 0.00 -> 4.71 mm
- net /Balance Interface V3/WDT_LOWER: track 0.00 -> 3.36 mm, vias 0 -> 1
- net /Balance Interface V3/UPPER_ADDRESS/A3: track 14.1 -> 17.3 mm
- net Net-(C103-Pad1): track 0.00 -> 2.88 mm
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Other:
- board size 250 x 145.5 mm -> 258.2 x 145.5 mm

Commit message: updated pcb still need to find j11
Parts:
- removed C102, C115, C127, C139, C151, C163, C175, C42, C54, C66, C78, C90: DNP 10nF, Capacitor_SMD:C_0805_2012Metric_Pad1.18x1.45mm_HandSolder
- removed Q10, Q12, Q13, Q15, Q16, Q18, Q19, Q21, Q22, Q24, Q25, Q27, Q28, Q3, Q30, Q31, Q33, Q34, Q36, Q37, Q4, Q6, Q7, Q9: SiR882DP, Package_SO:PowerPAK_SO-8_Single
- removed TP107, TP110, TP118, TP121, TP129, TP132, TP140, TP143, TP151, TP154, TP30, TP33, TP41, TP44, TP52, TP55, TP63, TP66, TP74, TP77, TP85, TP88, TP96, TP99: TestPoint, TestPoint:TestPoint_Pad_D1.0mm
- added T13: BUK9K13-60EX, BUK9K17-60E:SOT1205, B.Cu at (330.9, -29.7)
- added T14: BUK9K13-60EX, BUK9K17-60E:SOT1205, B.Cu at (330.3, -53.8)
- added T15: BUK9K13-60EX, BUK9K17-60E:SOT1205, B.Cu at (308.3, -68.1)
- added T16: BUK9K13-60EX, BUK9K17-60E:SOT1205, B.Cu at (303.1, -55.3)
- added T17: BUK9K13-60EX, BUK9K17-60E:SOT1205, B.Cu at (276.7, -56.9)
- added T18: BUK9K13-60EX, BUK9K17-60E:SOT1205, B.Cu at (276.4, -31.0)
- added T19: BUK9K13-60EX, BUK9K17-60E:SOT1205, B.Cu at (187.7, -74.3)
- added T20: BUK9K13-60EX, BUK9K17-60E:SOT1205, B.Cu at (200.7, -46.2)
- added T21: BUK9K13-60EX, BUK9K17-60E:SOT1205, B.Cu at (189.0, -26.0)
- added T22: BUK9K13-60EX, BUK9K17-60E:SOT1205, B.Cu at (167.3, -26.0)
- added T23: BUK9K13-60EX, BUK9K17-60E:SOT1205, B.Cu at (145.4, -26.1)
- added T24: BUK9K13-60EX, BUK9K17-60E:SOT1205, B.Cu at (145.7, -49.7)
- C100, C104, C105, C106, C107, C108, C109, C110, C111, C112, C113, C116, C117, C118, C119, C120, C121, C122, C123, C124, C125, C128, C129, C130, C131, C132, C133, C134, C135, C136, C137, C140, C141, C142, C143, C144, C145, C146, C147, C148, C149, C152, C153, C154, C155, C156, C157, C158, C159, C160, C161, C164, C165, C166, C167, C168, C169, C170, C171, C172, C173, C31, C32, C33, C34, C35, C36, C37, C38, C39, C40, C43, C44, C45, C46, C47, C48, C49, C50, C51, C52, C55, C56, C57, C58, C59, C60, C61, C62, C63, C64, C67, C68, C69, C70, C71, C72, C73, C74, C75, C76, C79, C80, C81, C82, C83, C84, C85, C86, C87, C88, C91, C92, C93, C94, C95, C96, C97, C98, C99, R100, R101, R134, R135, R136, R137, R138, R139, R140, R141, R146, R147, R148, R149, R150, R151, R152, R153, R158, R159, R160, R161, R162, R163, R164, R165, R170, R171, R172, R173, R174, R175, R176, R177, R182, R183, R184, R185, R186, R187, R188, R189, R194, R195, R196, R197, R198, R199, R200, R201, R34, R35, R36, R37, R38, R39, R40, R41, R46, R47, R48, R49, R50, R51, R52, R53, R58, R59, R60, R61, R62, R63, R64, R65, R70, R71, R72, R73, R74, R75, R76, R77, R82, R83, R84, R85, R86, R87, R88, R89, R94, R95, R96, R97, R98, R99, TP101, TP102, TP103, TP105, TP108, TP109, TP112, TP113, TP114, TP116, TP119, TP120, TP123, TP124, TP125, TP127, TP130, TP131, TP134, TP135, TP136, TP138, TP141, TP142, TP145, TP146, TP147, TP149, TP152, TP153, TP156, TP157, TP26, TP28, TP31, TP32, TP35, TP36, TP37, TP39, TP42, TP43, TP46, TP47, TP48, TP50, TP53, TP54, TP57, TP58, TP59, TP61, TP64, TP65, TP68, TP69, TP70, TP72, TP75, TP76, TP79, TP80, TP81, TP83, TP86, TP87, TP90, TP91, TP92, TP94, TP97, TP98: moved to B.Cu
- C13, C2, C3, C6: moved to F.Cu
- C5: footprint Capacitor_SMD:C_0603_1608Metric_Pad1.08x0.95mm_HandSolder -> Capacitor_SMD:C_0805_2012Metric_Pad1.18x1.45mm_HandSolder; moved to F.Cu
- D15, D17, D19, D21, D23, D25, D28, D30, D32, D34, D36, D38: value SBR10U200P5-13 -> SDT15H100P5-7; moved to B.Cu
- IC1: value ADS7038QRTERQ1 -> ADS7028QRTERQ1
- U6, U7, U8: value ISO7761DBQ -> ADuM7641A; footprint Package_SO:SSOP-16_3.9x4.9mm_P0.635mm -> Package_SO:QSOP-20_3.9x8.7mm_P0.635mm
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Connections:
- net /Balance Interface V3/C0 renamed /Balance Interface/C0
- net /Balance Interface V3/C1 renamed /Balance Interface/C1
- net /Balance Interface V3/C10 renamed /Balance Interface/C10
- net /Balance Interface V3/C11 renamed /Balance Interface/C11
- net /Balance Interface V3/C12 renamed /Balance Interface/C12
- net /Balance Interface V3/C2 renamed /Balance Interface/C2
- net /Balance Interface V3/C3 renamed /Balance Interface/C3
- net /Balance Interface V3/C4 renamed /Balance Interface/C4
- net /Balance Interface V3/C5 renamed /Balance Interface/C5
- net /Balance Interface V3/C6 renamed /Balance Interface/C6
- net /Balance Interface V3/C7 renamed /Balance Interface/C7
- net /Balance Interface V3/C8 renamed /Balance Interface/C8
- net /Balance Interface V3/C9 renamed /Balance Interface/C9
- net /Balance Interface V3/CS renamed /Balance Interface/CS
- net /Balance Interface V3/DRIVE renamed /Balance Interface/DRIVE
- net /Balance Interface V3/DTEN renamed /Balance Interface/DTEN
- net /Balance Interface V3/ISOMD renamed /Balance Interface/ISOMD
- net /Balance Interface V3/LOWER_ADDRESS/A0 renamed /Balance Interface/LOWER_ADDRESS/A0
- net /Balance Interface V3/LOWER_ADDRESS/A1 renamed /Balance Interface/LOWER_ADDRESS/A1
- net /Balance Interface V3/LOWER_ADDRESS/A2 renamed /Balance Interface/LOWER_ADDRESS/A2
- net /Balance Interface V3/LOWER_ADDRESS/A3 renamed /Balance Interface/LOWER_ADDRESS/A3
- net /Balance Interface V3/Lower Active Balance Group/ACTIVE_TAP1 renamed /Balance Interface/Lower Active Balance Group/ACTIVE_TAP1
- net /Balance Interface V3/Lower Active Balance Group/ACTIVE_TAP2 renamed /Balance Interface/Lower Active Balance Group/ACTIVE_TAP2
- net /Balance Interface V3/Lower Active Balance Group/ACTIVE_TAP3 renamed /Balance Interface/Lower Active Balance Group/ACTIVE_TAP3
- net /Balance Interface V3/Lower Active Balance Group/ACTIVE_TAP4 renamed /Balance Interface/Lower Active Balance Group/ACTIVE_TAP4
- net /Balance Interface V3/Lower Active Balance Group/ACTIVE_TAP5 renamed /Balance Interface/Lower Active Balance Group/ACTIVE_TAP5
- net /Balance Interface V3/Lower Active Balance Group/Active_Passive_Balance_Filter/BOOST renamed /Balance Interface/Lower Active Balance Group/BOOST
- net /Balance Interface V3/Lower Active Balance Group/C1 renamed /Balance Interface/Lower Active Balance Group/C1
- net /Balance Interface V3/Lower Active Balance Group/C2 renamed /Balance Interface/Lower Active Balance Group/C2
- net /Balance Interface V3/Lower Active Balance Group/C3 renamed /Balance Interface/Lower Active Balance Group/C3
- net /Balance Interface V3/Lower Active Balance Group/C4 renamed /Balance Interface/Lower Active Balance Group/C4
- net /Balance Interface V3/Lower Active Balance Group/C5 renamed /Balance Interface/Lower Active Balance Group/C5
- net /Balance Interface V3/Lower Active Balance Group/C6 renamed /Balance Interface/Lower Active Balance Group/C6
- net /Balance Interface V3/Lower Active Balance Group/PG1 renamed /Balance Interface/Lower Active Balance Group/PG1
- net /Balance Interface V3/Lower Active Balance Group/PG2 renamed /Balance Interface/Lower Active Balance Group/PG2
- net /Balance Interface V3/Lower Active Balance Group/PG3 renamed /Balance Interface/Lower Active Balance Group/PG3
- net /Balance Interface V3/Lower Active Balance Group/PG4 renamed /Balance Interface/Lower Active Balance Group/PG4
- net /Balance Interface V3/Lower Active Balance Group/PG5 renamed /Balance Interface/Lower Active Balance Group/PG5
- net /Balance Interface V3/Lower Active Balance Group/PG6 renamed /Balance Interface/Lower Active Balance Group/PG6
- net /Balance Interface V3/Lower Active Balance Group/PI1 renamed /Balance Interface/Lower Active Balance Group/PI1
- net /Balance Interface V3/Lower Active Balance Group/PI2 renamed /Balance Interface/Lower Active Balance Group/PI2
- net /Balance Interface V3/Lower Active Balance Group/PI3 renamed /Balance Interface/Lower Active Balance Group/PI3
- net /Balance Interface V3/Lower Active Balance Group/PI4 renamed /Balance Interface/Lower Active Balance Group/PI4
- net /Balance Interface V3/Lower Active Balance Group/PI5 renamed /Balance Interface/Lower Active Balance Group/PI5
- net /Balance Interface V3/Lower Active Balance Group/PI6 renamed /Balance Interface/Lower Active Balance Group/PI6
- net /Balance Interface V3/Lower Active Balance Group/RTONP renamed /Balance Interface/Lower Active Balance Group/RTONP
- net /Balance Interface V3/Lower Active Balance Group/RTONS renamed /Balance Interface/Lower Active Balance Group/RTONS
- net /Balance Interface V3/Lower Active Balance Group/SG1 renamed /Balance Interface/Lower Active Balance Group/SG1
- net /Balance Interface V3/Lower Active Balance Group/SG2 renamed /Balance Interface/Lower Active Balance Group/SG2
- net /Balance Interface V3/Lower Active Balance Group/SG3 renamed /Balance Interface/Lower Active Balance Group/SG3
- net /Balance Interface V3/Lower Active Balance Group/SG4 renamed /Balance Interface/Lower Active Balance Group/SG4
- net /Balance Interface V3/Lower Active Balance Group/SG5 renamed /Balance Interface/Lower Active Balance Group/SG5
- net /Balance Interface V3/Lower Active Balance Group/SG6 renamed /Balance Interface/Lower Active Balance Group/SG6
- net /Balance Interface V3/Lower Active Balance Group/SI1 renamed /Balance Interface/Lower Active Balance Group/SI1
- net /Balance Interface V3/Lower Active Balance Group/SI2 renamed /Balance Interface/Lower Active Balance Group/SI2
- net /Balance Interface V3/Lower Active Balance Group/SI3 renamed /Balance Interface/Lower Active Balance Group/SI3
- net /Balance Interface V3/Lower Active Balance Group/SI4 renamed /Balance Interface/Lower Active Balance Group/SI4
- net /Balance Interface V3/Lower Active Balance Group/SI5 renamed /Balance Interface/Lower Active Balance Group/SI5
- net /Balance Interface V3/Lower Active Balance Group/SI6 renamed /Balance Interface/Lower Active Balance Group/SI6
- net /Balance Interface V3/Lower Active Balance Group/V- renamed /Balance Interface/Lower Active Balance Group/V-
- net /Balance Interface V3/PASSIVE_ADDRESS/A0 renamed /Balance Interface/PASSIVE_ADDRESS/A0
- net /Balance Interface V3/PASSIVE_ADDRESS/A1 renamed /Balance Interface/PASSIVE_ADDRESS/A1
- net /Balance Interface V3/PASSIVE_ADDRESS/A2 renamed /Balance Interface/PASSIVE_ADDRESS/A2
- net /Balance Interface V3/PASSIVE_ADDRESS/A3 renamed /Balance Interface/PASSIVE_ADDRESS/A3
- net /Balance Interface V3/S1 renamed /Balance Interface/S1
- net /Balance Interface V3/S10 renamed /Balance Interface/S10
- net /Balance Interface V3/S11 renamed /Balance Interface/S11
- net /Balance Interface V3/S12 renamed /Balance Interface/S12
- net /Balance Interface V3/S2 renamed /Balance Interface/S2
- net /Balance Interface V3/S3 renamed /Balance Interface/S3
- net /Balance Interface V3/S4 renamed /Balance Interface/S4
- net /Balance Interface V3/S5 renamed /Balance Interface/S5
- net /Balance Interface V3/S6 renamed /Balance Interface/S6
- net /Balance Interface V3/S7 renamed /Balance Interface/S7
- net /Balance Interface V3/S8 renamed /Balance Interface/S8
- net /Balance Interface V3/S9 renamed /Balance Interface/S9
- net /Balance Interface V3/SCK renamed /Balance Interface/SCK
- net /Balance Interface V3/SCKI_LOWER renamed /Balance Interface/SCKI_LOWER
- net /Balance Interface V3/SCKI_UPPER renamed /Balance Interface/SCKI_UPPER
- net /Balance Interface V3/TAP0 renamed /Balance Interface/TAP0
- net /Balance Interface V3/TAP1 renamed /Balance Interface/TAP1
- net /Balance Interface V3/TAP10 renamed /Balance Interface/TAP10
- net /Balance Interface V3/TAP11 renamed /Balance Interface/TAP11
- net /Balance Interface V3/TAP12 renamed /Balance Interface/TAP12
- net /Balance Interface V3/TAP2 renamed /Balance Interface/TAP2
- net /Balance Interface V3/TAP3 renamed /Balance Interface/TAP3
- net /Balance Interface V3/TAP4 renamed /Balance Interface/TAP4
- net /Balance Interface V3/TAP5 renamed /Balance Interface/TAP5
- net /Balance Interface V3/TAP6 renamed /Balance Interface/TAP6
- net /Balance Interface V3/TAP7 renamed /Balance Interface/TAP7
- net /Balance Interface V3/TAP8 renamed /Balance Interface/TAP8
- net /Balance Interface V3/TAP9 renamed /Balance Interface/TAP9
- net /Balance Interface V3/UPPER_ADDRESS/A0 renamed /Balance Interface/UPPER_ADDRESS/A0
- net /Balance Interface V3/UPPER_ADDRESS/A1 renamed /Balance Interface/UPPER_ADDRESS/A1
- net /Balance Interface V3/UPPER_ADDRESS/A2 renamed /Balance Interface/UPPER_ADDRESS/A2
- net /Balance Interface V3/UPPER_ADDRESS/A3 renamed /Balance Interface/UPPER_ADDRESS/A3
- net /Balance Interface V3/Upper Active Balance Group/ACTIVE_TAP1 renamed /Balance Interface/Upper Active Balance Group/ACTIVE_TAP1
- net /Balance Interface V3/Upper Active Balance Group/ACTIVE_TAP2 renamed /Balance Interface/Upper Active Balance Group/ACTIVE_TAP2
- net /Balance Interface V3/Upper Active Balance Group/ACTIVE_TAP3 renamed /Balance Interface/Upper Active Balance Group/ACTIVE_TAP3
- net /Balance Interface V3/Upper Active Balance Group/ACTIVE_TAP4 renamed /Balance Interface/Upper Active Balance Group/ACTIVE_TAP4
- net /Balance Interface V3/Upper Active Balance Group/ACTIVE_TAP5 renamed /Balance Interface/Upper Active Balance Group/ACTIVE_TAP5
- net /Balance Interface V3/Upper Active Balance Group/Active_Passive_Balance_Filter/BOOST renamed /Balance Interface/Upper Active Balance Group/BOOST
- net /Balance Interface V3/Upper Active Balance Group/C1 renamed /Balance Interface/Upper Active Balance Group/C1
- net /Balance Interface V3/Upper Active Balance Group/C2 renamed /Balance Interface/Upper Active Balance Group/C2
- net /Balance Interface V3/Upper Active Balance Group/C3 renamed /Balance Interface/Upper Active Balance Group/C3
- net /Balance Interface V3/Upper Active Balance Group/C4 renamed /Balance Interface/Upper Active Balance Group/C4
- net /Balance Interface V3/Upper Active Balance Group/C5 renamed /Balance Interface/Upper Active Balance Group/C5
- net /Balance Interface V3/Upper Active Balance Group/C6 renamed /Balance Interface/Upper Active Balance Group/C6
- net /Balance Interface V3/Upper Active Balance Group/PG1 renamed /Balance Interface/Upper Active Balance Group/PG1
- net /Balance Interface V3/Upper Active Balance Group/PG2 renamed /Balance Interface/Upper Active Balance Group/PG2
- net /Balance Interface V3/Upper Active Balance Group/PG3 renamed /Balance Interface/Upper Active Balance Group/PG3
- net /Balance Interface V3/Upper Active Balance Group/PG4 renamed /Balance Interface/Upper Active Balance Group/PG4
- net /Balance Interface V3/Upper Active Balance Group/PG5 renamed /Balance Interface/Upper Active Balance Group/PG5
- net /Balance Interface V3/Upper Active Balance Group/PG6 renamed /Balance Interface/Upper Active Balance Group/PG6
- net /Balance Interface V3/Upper Active Balance Group/PI1 renamed /Balance Interface/Upper Active Balance Group/PI1
- net /Balance Interface V3/Upper Active Balance Group/PI2 renamed /Balance Interface/Upper Active Balance Group/PI2
- net /Balance Interface V3/Upper Active Balance Group/PI3 renamed /Balance Interface/Upper Active Balance Group/PI3
- net /Balance Interface V3/Upper Active Balance Group/PI4 renamed /Balance Interface/Upper Active Balance Group/PI4
- net /Balance Interface V3/Upper Active Balance Group/PI5 renamed /Balance Interface/Upper Active Balance Group/PI5
- net /Balance Interface V3/Upper Active Balance Group/PI6 renamed /Balance Interface/Upper Active Balance Group/PI6
- net /Balance Interface V3/Upper Active Balance Group/RTONP renamed /Balance Interface/Upper Active Balance Group/RTONP
- net /Balance Interface V3/Upper Active Balance Group/RTONS renamed /Balance Interface/Upper Active Balance Group/RTONS
- net /Balance Interface V3/Upper Active Balance Group/SG1 renamed /Balance Interface/Upper Active Balance Group/SG1
- net /Balance Interface V3/Upper Active Balance Group/SG2 renamed /Balance Interface/Upper Active Balance Group/SG2
- net /Balance Interface V3/Upper Active Balance Group/SG3 renamed /Balance Interface/Upper Active Balance Group/SG3
- net /Balance Interface V3/Upper Active Balance Group/SG4 renamed /Balance Interface/Upper Active Balance Group/SG4
- net /Balance Interface V3/Upper Active Balance Group/SG5 renamed /Balance Interface/Upper Active Balance Group/SG5
- net /Balance Interface V3/Upper Active Balance Group/SG6 renamed /Balance Interface/Upper Active Balance Group/SG6
- net /Balance Interface V3/Upper Active Balance Group/SI1 renamed /Balance Interface/Upper Active Balance Group/SI1
- net /Balance Interface V3/Upper Active Balance Group/SI2 renamed /Balance Interface/Upper Active Balance Group/SI2
- net /Balance Interface V3/Upper Active Balance Group/SI3 renamed /Balance Interface/Upper Active Balance Group/SI3
- net /Balance Interface V3/Upper Active Balance Group/SI4 renamed /Balance Interface/Upper Active Balance Group/SI4
- net /Balance Interface V3/Upper Active Balance Group/SI5 renamed /Balance Interface/Upper Active Balance Group/SI5
- net /Balance Interface V3/Upper Active Balance Group/SI6 renamed /Balance Interface/Upper Active Balance Group/SI6
- net /Balance Interface V3/V+ renamed /Balance Interface/V+
- net /Balance Interface V3/V_TEMP_SENSOR_REF renamed /Balance Interface/V_TEMP_SENSOR_REF
- net /Balance Interface V3/WDT renamed /Balance Interface/WDT
- net /Balance Interface V3/WDT_LOWER renamed /Balance Interface/WDT_LOWER
- net /Balance Interface V3/WDT_UPPER renamed /Balance Interface/WDT_UPPER
- net /Balance Interface V3/nCSBI_LOWER renamed /Balance Interface/nCSBI_LOWER
- net /Balance Interface V3/nCSBI_UPPER renamed /Balance Interface/nCSBI_UPPER
- net /HV Isolation v2/CS1 renamed /Temperature Isolation/CS1
- net /HV Isolation v3/CS1 renamed /Lower Ground Isolation/CS1
- net /HV Isolation v3/CS1_ISO renamed /Lower Ground Isolation/CS1_ISO
- net /HV Isolation v4/CS1 renamed /Upper Ground Isolation/CS1
- net /HV Isolation v4/CS1_ISO renamed /Upper Ground Isolation/CS1_ISO
- net Net-(C10-Pad1) renamed /CAN/CAN_PRE_P
- net Net-(C11-Pad1) renamed /CAN/CAN_PRE_N
- C16 pad 1: /Balance Interface V3/VREG -> /Balance Interface/VREG
- C177 pad 1: /Balance Interface V3/VREG -> /Balance Interface/VREG
- C179 pad 1: /Balance Interface V3/VREG_UPPER -> /Balance Interface/VREG_UPPER
- C181 pad 1: /Balance Interface V3/VREG_LOWER -> /Balance Interface/VREG_LOWER
- C25 pad 1: /Balance Interface V3/VREG -> /Balance Interface/VREG
- IC1 pad 10: /Balance Interface V3/VREG -> /Balance Interface/VREG
- IC1 pad 12: /Balance Interface V3/IBIAS -> /Balance Interface/IBIAS
- IC1 pad 14: /Balance Interface V3/ICMP -> /Balance Interface/ICMP
- J1 pad 2: /VGND -> /CAN_P
- J1 pad 3: /CAN_P -> /CAN_N
- J1 pad 4: unconnected-(J1-Pad4) -> /VGND
- J1 pad 5: /CAN_N -> unconnected-(J1-Pad5)
- J13 pad 2: 3.3V_ISO -> Net-(J13-Pad2)
- J13 pad 3: Net-(J13-Pad3) -> 0V_ISO
- J13 pad 4: Net-(J13-Pad4) -> 3.3V_ISO
- J13 pad 5: 0V_ISO -> Net-(J13-Pad5)
- J2 pad 2: /VGND -> /CAN_P
- J2 pad 3: /CAN_P -> /CAN_N
- J2 pad 4: unconnected-(J2-Pad4) -> /VGND
- J2 pad 5: /CAN_N -> unconnected-(J2-Pad5)
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Routing:
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- added copper zone on B.Cu, net /Balance Interface/Lower Active Balance Group/ACTIVE_TAP1
- added copper zone on F.Cu, net /Balance Interface/Lower Active Balance Group/ACTIVE_TAP1
- added copper zone on B.Cu, net /Balance Interface/Lower Active Balance Group/ACTIVE_TAP2
- added copper zone on F.Cu, net /Balance Interface/Lower Active Balance Group/ACTIVE_TAP2
- added copper zone on B.Cu, net /Balance Interface/Lower Active Balance Group/ACTIVE_TAP3
- added copper zone on F.Cu, net /Balance Interface/Lower Active Balance Group/ACTIVE_TAP3
- added copper zone on B.Cu, net /Balance Interface/Lower Active Balance Group/ACTIVE_TAP4
- added copper zone on F.Cu, net /Balance Interface/Lower Active Balance Group/ACTIVE_TAP4
- added copper zone on B.Cu, net /Balance Interface/Lower Active Balance Group/ACTIVE_TAP5
- added copper zone on F.Cu, net /Balance Interface/Lower Active Balance Group/ACTIVE_TAP5
- added copper zone on B.Cu, net /Balance Interface/Lower Active Balance Group/BOOST
- added copper zone on F.Cu, net /Balance Interface/Lower Active Balance Group/BOOST
- added copper zone on B.Cu, net /Balance Interface/Upper Active Balance Group/ACTIVE_TAP1
- added copper zone on F.Cu, net /Balance Interface/Upper Active Balance Group/ACTIVE_TAP1
- added copper zone on B.Cu, net /Balance Interface/Upper Active Balance Group/ACTIVE_TAP2
- added copper zone on F.Cu, net /Balance Interface/Upper Active Balance Group/ACTIVE_TAP2
- added copper zone on B.Cu, net /Balance Interface/Upper Active Balance Group/ACTIVE_TAP3
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Other:
- board size 258.2 x 145.5 mm -> 210 x 75 mm

Commit message: fixed issues on higher cells, study into how to route
Parts:
- added C42: 1u, Capacitor_SMD:C_0805_2012Metric_Pad1.18x1.45mm_HandSolder, F.Cu at (302.5, -14.8)
- added C54: 1u, Capacitor_SMD:C_0805_2012Metric_Pad1.18x1.45mm_HandSolder, F.Cu at (64.2, -88.5)
- added C66: 100nF, Capacitor_SMD:C_0805_2012Metric_Pad1.18x1.45mm_HandSolder, F.Cu at (156.2, -42.5)
- added C78: 22uF, Capacitor_SMD:C_0805_2012Metric_Pad1.18x1.45mm_HandSolder, F.Cu at (156.2, -39.5)
- added D6: LED (Red), LED_SMD:LED_0805_2012Metric_Pad1.15x1.40mm_HandSolder, F.Cu at (161.0, -42.5)
- added PS2: R2S-0505, R2S-0505:CONV_R2S-0505, F.Cu at (147.0, -36.9)
- added R251: 2.2kR, Resistor_SMD:R_0603_1608Metric_Pad0.98x0.95mm_HandSolder, F.Cu at (155.9, -36.7)
- added R252: 0R DNP, Resistor_SMD:R_0603_1608Metric_Pad0.98x0.95mm_HandSolder, F.Cu at (171.3, -42.8)
- added TP30: TestPoint, TestPoint:TestPoint_Pad_D1.0mm, F.Cu at (160.1, -39.4)
- added TP33: TestPoint, TestPoint:TestPoint_Pad_D1.0mm, F.Cu at (155.3, -34.0)
- R103, R104, R105, R106, R107, R108, R109, R110, R111, R112, R113, R114, R115, R116, R117, R118, R129, R130, R29, R30: moved to B.Cu
- moved TP120 143.9 mm to (75.8, -119.0)
- moved TP131 143.5 mm to (54.8, -119.1)
- moved TP142 143.3 mm to (33.1, -119.2)
- moved C130 142.4 mm to (83.8, -109.8)
- moved R157 142.4 mm to (89.2, -107.1)
- moved R165 142.4 mm to (74.8, -113.4)
- moved TP116 142.4 mm to (80.7, -106.5)
- moved C128 142.4 mm to (83.3, -100.3)
- moved C129 142.4 mm to (80.8, -100.3)
- moved C131 142.4 mm to (78.3, -100.3)
- moved C132 142.4 mm to (86.1, -115.2)
- moved C133 142.4 mm to (70.8, -115.3)
- moved C134 142.4 mm to (75.8, -100.3)
- moved C135 142.4 mm to (78.6, -107.2)
- moved C136 142.4 mm to (73.3, -100.3)
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Connections:
- C110 pad 1: /Balance Interface/Lower Active Balance Group/V- -> GND_HV
- C111 pad 1: /Balance Interface/Lower Active Balance Group/V- -> GND_HV
- C112 pad 1: /Balance Interface/Lower Active Balance Group/V- -> GND_HV
- C113 pad 1: /Balance Interface/Lower Active Balance Group/V- -> GND_HV
- C122 pad 1: /Balance Interface/Lower Active Balance Group/V- -> GND_HV
- C123 pad 1: /Balance Interface/Lower Active Balance Group/V- -> GND_HV
- C124 pad 1: /Balance Interface/Lower Active Balance Group/V- -> GND_HV
- C125 pad 1: /Balance Interface/Lower Active Balance Group/V- -> GND_HV
- C126 pad 1: /Balance Interface/S4 -> /Balance Interface/C3
- C134 pad 1: /Balance Interface/Lower Active Balance Group/V- -> GND_HV
- C135 pad 1: /Balance Interface/Lower Active Balance Group/V- -> GND_HV
- C136 pad 1: /Balance Interface/Lower Active Balance Group/V- -> GND_HV
- C137 pad 1: /Balance Interface/Lower Active Balance Group/V- -> GND_HV
- C138 pad 2: /Balance Interface/S4 -> /Balance Interface/C3
- C146 pad 1: /Balance Interface/Lower Active Balance Group/V- -> GND_HV
- C147 pad 1: /Balance Interface/Lower Active Balance Group/V- -> GND_HV
- C148 pad 1: /Balance Interface/Lower Active Balance Group/V- -> GND_HV
- C149 pad 1: /Balance Interface/Lower Active Balance Group/V- -> GND_HV
- C158 pad 1: /Balance Interface/Lower Active Balance Group/V- -> GND_HV
- C159 pad 1: /Balance Interface/Lower Active Balance Group/V- -> GND_HV
- C16 pad 1: /Balance Interface/VREG -> 5V_HV
- C160 pad 1: /Balance Interface/Lower Active Balance Group/V- -> GND_HV
- C161 pad 1: /Balance Interface/Lower Active Balance Group/V- -> GND_HV
- C164 pad 1: /Balance Interface/Lower Active Balance Group/V- -> GND_HV
- C165 pad 1: /Balance Interface/Lower Active Balance Group/V- -> GND_HV
- C166 pad 1: /Balance Interface/Lower Active Balance Group/V- -> GND_HV
- C167 pad 1: /Balance Interface/Lower Active Balance Group/V- -> GND_HV
- C17 pad 1: GND_HV -> 0V_HV
- C170 pad 1: /Balance Interface/Lower Active Balance Group/V- -> GND_HV
- C171 pad 1: /Balance Interface/Lower Active Balance Group/V- -> GND_HV
- C172 pad 1: /Balance Interface/Lower Active Balance Group/V- -> GND_HV
- C173 pad 1: /Balance Interface/Lower Active Balance Group/V- -> GND_HV
- C177 pad 1: /Balance Interface/VREG -> +5V_HV
- C18 pad 1: GND_HV -> 0V_HV
- C19 pad 1: GND_HV -> 0V_HV
- C20 pad 1: GND_HV -> 0V_HV
- C21 pad 1: GND_HV -> 0V_HV
- C22 pad 1: GND_HV -> 0V_HV
- C23 pad 1: GND_HV -> 0V_HV
- C24 pad 1: GND_HV -> 0V_HV
- C25 pad 1: /Balance Interface/VREG -> +5V_HV
- C25 pad 2: GND_HV -> 0V_HV
- C26 pad 2: GND_HV -> 0V_HV
- C27 pad 2: GND_HV -> 0V_HV
- C28 pad 1: GND_HV -> 0V_HV
- C29 pad 2: GND_HV -> 0V_HV
- C53 pad 1: /Balance Interface/S10 -> /Balance Interface/C9
- C65 pad 2: /Balance Interface/S10 -> /Balance Interface/C9
- D38 pad 2: /Balance Interface/Lower Active Balance Group/V- -> GND_HV
- D38 pad 3: /Balance Interface/Lower Active Balance Group/V- -> GND_HV
- D39 pad 1: /Balance Interface/Lower Active Balance Group/V- -> GND_HV
- F14 pad 2: /Balance Interface/Lower Active Balance Group/V- -> GND_HV
- IC1 pad 10: /Balance Interface/VREG -> 5V_HV
- J3 pad 10: GND_HV -> 0V_HV
- J3 pad 11: GND_HV -> 0V_HV
- J3 pad 12: GND_HV -> 0V_HV
- J3 pad 13: GND_HV -> 0V_HV
- J3 pad 14: GND_HV -> 0V_HV
- J3 pad 15: GND_HV -> 0V_HV
- J3 pad 16: GND_HV -> 0V_HV
- J3 pad 9: GND_HV -> 0V_HV
- J5 pad 1: GND_HV -> 0V_HV
- J5 pad 3: /Balance Interface/VREG -> +5V_HV
- J6 pad 1: GND_HV -> 0V_HV
- J6 pad 3: /Balance Interface/VREG -> +5V_HV
- Q1 pad 3: /Balance Interface/VREG -> +5V_HV
- R10 pad 2: +5V_HV -> 5V_HV
- R119 pad 1: /Balance Interface/VREG -> +5V_HV
- R12 pad 2: +5V_HV -> 5V_HV
- R121 pad 1: /Balance Interface/VREG -> +5V_HV
- R123 pad 1: /Balance Interface/VREG -> +5V_HV
- R125 pad 1: /Balance Interface/VREG -> +5V_HV
- R127 pad 2: /Balance Interface/Lower Active Balance Group/C6 -> /Balance Interface/S6
- R129 pad 2: /Balance Interface/Lower Active Balance Group/V- -> GND_HV
- R130 pad 2: /Balance Interface/Lower Active Balance Group/V- -> GND_HV
- R139 pad 2: /Balance Interface/Lower Active Balance Group/V- -> GND_HV
- R14 pad 2: +5V_HV -> 5V_HV
- R151 pad 2: /Balance Interface/Lower Active Balance Group/V- -> GND_HV
- R16 pad 2: +5V_HV -> 5V_HV
- R163 pad 2: /Balance Interface/Lower Active Balance Group/V- -> GND_HV
- R166 pad 1: /Balance Interface/S4 -> /Balance Interface/C3
- R175 pad 2: /Balance Interface/Lower Active Balance Group/V- -> GND_HV
- R18 pad 2: +5V_HV -> 5V_HV
- R187 pad 2: /Balance Interface/Lower Active Balance Group/V- -> GND_HV
- R191 pad 1: /Balance Interface/Lower Active Balance Group/V- -> GND_HV
- R197 pad 2: /Balance Interface/Lower Active Balance Group/V- -> GND_HV
- R199 pad 2: /Balance Interface/Lower Active Balance Group/V- -> GND_HV
- R20 pad 2: +5V_HV -> 5V_HV
- R22 pad 1: /Balance Interface/VREG -> +5V_HV
- R24 pad 1: GND_HV -> 0V_HV
- R27 pad 2: /Balance Interface/Upper Active Balance Group/C6 -> /Balance Interface/S12
- R6 pad 2: +5V_HV -> 5V_HV
- R66 pad 1: /Balance Interface/S10 -> /Balance Interface/C9
- R8 pad 2: +5V_HV -> 5V_HV
- TP124 pad 1: /Balance Interface/S4 -> /Balance Interface/C3
- TP25 pad 1: /Balance Interface/VREG -> +5V_HV
- TP58 pad 1: /Balance Interface/S10 -> /Balance Interface/C9
- U3 pad 19: /Balance Interface/S4 -> /Balance Interface/C3
- U3 pad 30: GND_HV -> 0V_HV
- U3 pad 31: GND_HV -> 0V_HV
- U3 pad 37: /Balance Interface/VREG -> +5V_HV
- U3 pad 7: /Balance Interface/S10 -> /Balance Interface/C9
- U4 pad 24: /Balance Interface/Upper Active Balance Group/C1 -> /Balance Interface/C8
- U4 pad 27: /Balance Interface/Upper Active Balance Group/C2 -> /Balance Interface/C9
- U4 pad 30: /Balance Interface/Upper Active Balance Group/C3 -> /Balance Interface/S11
- U4 pad 39: /Balance Interface/Upper Active Balance Group/C6 -> /Balance Interface/S12
- U5 pad 15: /Balance Interface/Lower Active Balance Group/V- -> GND_HV
- U5 pad 21: /Balance Interface/Lower Active Balance Group/V- -> GND_HV
- U5 pad 24: /Balance Interface/Lower Active Balance Group/C1 -> /Balance Interface/C2
- U5 pad 27: /Balance Interface/Lower Active Balance Group/C2 -> /Balance Interface/C3
- U5 pad 30: /Balance Interface/Lower Active Balance Group/C3 -> /Balance Interface/S5
- U5 pad 39: /Balance Interface/Lower Active Balance Group/C6 -> /Balance Interface/S6
- U5 pad 49: /Balance Interface/Lower Active Balance Group/V- -> GND_HV
- U6 pad 14: /Balance Interface/VREG -> +5V_HV
- U6 pad 20: /Balance Interface/VREG -> +5V_HV
Routing:
- net GND_HV: track 0.00 -> 42.2 mm, vias 0 -> 18
- net /Balance Interface/Lower Active Balance Group/V-: track 23.6 -> 0.00 mm, vias 14 -> 0
- net /Balance Interface/VREG_LOWER: track 0.00 -> 20.3 mm, vias 0 -> 3
- net /Balance Interface/VREG_UPPER: track 0.00 -> 20.3 mm, vias 0 -> 3
- net /UPPER_GND: track 28.9 -> 47.5 mm, vias 20 -> 24
- net /Balance Interface/C9: track 6.78 -> 19.2 mm, vias 2 -> 5
- net /Balance Interface/C3: track 6.78 -> 19.2 mm, vias 2 -> 5
- net /Balance Interface/WDT_UPPER: track 0.00 -> 10.1 mm, vias 0 -> 1
- net /Balance Interface/WDT_LOWER: track 0.00 -> 10.1 mm, vias 0 -> 1
- net /Balance Interface/UPPER_ADDRESS/A3: track 0.00 -> 10.0 mm, vias 0 -> 1
- net /Balance Interface/LOWER_ADDRESS/A3: track 0.00 -> 10.0 mm, vias 0 -> 1
- net /Balance Interface/UPPER_ADDRESS/A2: track 0.00 -> 9.28 mm, vias 0 -> 1
- net /Balance Interface/LOWER_ADDRESS/A2: track 0.00 -> 9.28 mm, vias 0 -> 1
- net /Balance Interface/UPPER_ADDRESS/A1: track 0.00 -> 8.79 mm, vias 0 -> 1
- net /Balance Interface/LOWER_ADDRESS/A1: track 0.00 -> 8.79 mm, vias 0 -> 1
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Other:
- board outline removed

Commit message: refined in-out routing mechanism
Parts:
- removed J10, J8: Conn_01x02, Connector_PinHeader_2.54mm:PinHeader_1x02_P2.54mm_Vertical
- C101, C114, C126, C138, C150, C162, C174, C41, C53, C65, C77, C89, D16, D18, D20, D22, D24, D26, D29, D31, D33, D35, D37, D39, Q11, Q14, Q17, Q2, Q20, Q23, Q26, Q29, Q32, Q35, Q38, Q5, Q8, R102, R131, R132, R133, R142, R143, R144, R145, R154, R155, R156, R157, R166, R167, R168, R169, R178, R179, R180, R181, R190, R191, R192, R193, R202, R203, R204, R205, R31, R32, R33, R42, R43, R44, R45, R54, R55, R56, R57, R66, R67, R68, R69, R78, R79, R80, R81, R90, R91, R92, R93, TP104, TP115, TP126, TP137, TP148, TP27, TP38, TP49, TP60, TP71, TP82, TP93: moved to B.Cu
- TP101, TP102, TP103, TP105, TP112, TP113, TP114, TP116, TP123, TP124, TP125, TP127, TP134, TP135, TP136, TP138, TP145, TP146, TP147, TP149, TP156, TP157, TP26, TP28, TP35, TP36, TP37, TP39, TP46, TP47, TP48, TP50, TP57, TP58, TP59, TP61, TP68, TP69, TP70, TP72, TP79, TP80, TP81, TP83, TP90, TP91, TP92, TP94: moved to F.Cu
- moved TP142 269.3 mm to (150.8, 123.1), turned to 0 degrees
- moved C157 267.3 mm to (155.7, 119.4), turned to 90 degrees
- moved TP141 263.5 mm to (143.8, 123.1), turned to 0 degrees
- moved TP144 262.6 mm to (152.6, 117.5), turned to 0 degrees
- moved T23 262.4 mm to (147.3, 120.9), turned to 0 degrees
- moved TP153 261.6 mm to (173.0, 123.2), turned to 0 degrees
- moved C169 261.1 mm to (178.0, 119.5), turned to 90 degrees
- moved R189 260.1 mm to (151.7, 117.5), turned to 180 degrees
- moved R186 259.5 mm to (155.7, 114.9), turned to 90 degrees
- moved TP155 256.4 mm to (174.9, 117.6), turned to 0 degrees
- moved R187 254.4 mm to (150.0, 114.0), turned to 90 degrees
- moved TP152 254.2 mm to (166.0, 123.2), turned to 0 degrees
- moved T24 254.1 mm to (169.5, 121.0), turned to 0 degrees
- moved C156 254.1 mm to (140.6, 119.3), turned to 180 degrees
- moved R198 253.9 mm to (178.0, 115.0), turned to 90 degrees
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Connections:
- C126 pad 1: /Balance Interface/C3 -> /Balance Interface/C4
- C138 pad 2: /Balance Interface/C3 -> /Balance Interface/C4
- C53 pad 1: /Balance Interface/C9 -> /Balance Interface/C10
- C65 pad 2: /Balance Interface/C9 -> /Balance Interface/C10
- J9 pad 2: Net-(J10-Pad1) -> /SDN_IN
- K1 pad 9: Net-(J10-Pad1) -> /SDN_IN
- R157 pad 2: /Balance Interface/C4 -> /Balance Interface/S4
- R166 pad 1: /Balance Interface/C3 -> /Balance Interface/C4
- R57 pad 2: /Balance Interface/C10 -> /Balance Interface/S10
- R66 pad 1: /Balance Interface/C9 -> /Balance Interface/C10
- TP124 pad 1: /Balance Interface/C3 -> /Balance Interface/C4
- TP58 pad 1: /Balance Interface/C9 -> /Balance Interface/C10
- U3 pad 19: /Balance Interface/C3 -> /Balance Interface/S4
- U3 pad 7: /Balance Interface/C9 -> /Balance Interface/S10
- U4 pad 24: /Balance Interface/C8 -> /Balance Interface/C7
- U4 pad 27: /Balance Interface/C9 -> /Balance Interface/C8
- U4 pad 30: /Balance Interface/S11 -> /Balance Interface/C9
- U4 pad 33: /Balance Interface/Upper Active Balance Group/C4 -> /Balance Interface/C10
- U4 pad 36: /Balance Interface/Upper Active Balance Group/C5 -> /Balance Interface/S11
- U5 pad 24: /Balance Interface/C2 -> /Balance Interface/C1
- U5 pad 27: /Balance Interface/C3 -> /Balance Interface/C2
- U5 pad 30: /Balance Interface/S5 -> /Balance Interface/C3
- U5 pad 33: /Balance Interface/Lower Active Balance Group/C4 -> /Balance Interface/C4
- U5 pad 36: /Balance Interface/Lower Active Balance Group/C5 -> /Balance Interface/S5
Routing:
- net /Balance Interface/Lower Active Balance Group/ACTIVE_TAP5: track 11.0 -> 56.8 mm, vias 8 -> 2
- net /Balance Interface/Lower Active Balance Group/ACTIVE_TAP2: track 11.0 -> 56.8 mm, vias 8 -> 2
- net /Balance Interface/Upper Active Balance Group/ACTIVE_TAP2: track 11.0 -> 56.8 mm, vias 8 -> 2
- net /Balance Interface/Lower Active Balance Group/ACTIVE_TAP3: track 11.0 -> 56.8 mm, vias 8 -> 2
- net /Balance Interface/Lower Active Balance Group/ACTIVE_TAP1: track 11.0 -> 56.8 mm, vias 8 -> 2
- net /Balance Interface/Upper Active Balance Group/ACTIVE_TAP5: track 11.0 -> 56.8 mm, vias 8 -> 2
- net /Balance Interface/Upper Active Balance Group/ACTIVE_TAP3: track 11.0 -> 56.8 mm, vias 8 -> 2
- net /Balance Interface/Upper Active Balance Group/ACTIVE_TAP4: track 11.0 -> 56.8 mm, vias 8 -> 2
- net /Balance Interface/Upper Active Balance Group/ACTIVE_TAP1: track 11.0 -> 56.8 mm, vias 8 -> 2
- net /Balance Interface/Lower Active Balance Group/ACTIVE_TAP4: track 11.0 -> 56.8 mm, vias 8 -> 2
- net /Balance Interface/V+: track 5.30 -> 32.8 mm, vias 6 -> 2
- net /Balance Interface/Lower Active Balance Group/BOOST: track 45.0 -> 70.4 mm, vias 24 -> 6
- net /Balance Interface/Upper Active Balance Group/BOOST: track 45.0 -> 70.4 mm, vias 24 -> 6
- net /UPPER_GND: track 47.5 -> 71.3 mm, vias 24 -> 14
- net /Balance Interface/VREG_UPPER: track 20.3 -> 0.00 mm, vias 3 -> 0
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- removed copper zone on B.Cu, net /Balance Interface/Lower Active Balance Group/ACTIVE_TAP1
- removed copper zone on F.Cu, net /Balance Interface/Lower Active Balance Group/ACTIVE_TAP1
- removed copper zone on B.Cu, net /Balance Interface/Lower Active Balance Group/ACTIVE_TAP2
- removed copper zone on F.Cu, net /Balance Interface/Lower Active Balance Group/ACTIVE_TAP2
- removed copper zone on B.Cu, net /Balance Interface/Lower Active Balance Group/ACTIVE_TAP3
- removed copper zone on F.Cu, net /Balance Interface/Lower Active Balance Group/ACTIVE_TAP3
- removed copper zone on B.Cu, net /Balance Interface/Lower Active Balance Group/ACTIVE_TAP4
- removed copper zone on F.Cu, net /Balance Interface/Lower Active Balance Group/ACTIVE_TAP4
- removed copper zone on B.Cu, net /Balance Interface/Lower Active Balance Group/ACTIVE_TAP5
- removed copper zone on F.Cu, net /Balance Interface/Lower Active Balance Group/ACTIVE_TAP5
- removed copper zone on B.Cu, net /Balance Interface/Lower Active Balance Group/BOOST
- removed copper zone on F.Cu, net /Balance Interface/Lower Active Balance Group/BOOST
- removed copper zone on B.Cu, net /Balance Interface/Upper Active Balance Group/ACTIVE_TAP1
- removed copper zone on F.Cu, net /Balance Interface/Upper Active Balance Group/ACTIVE_TAP1
- removed copper zone on B.Cu, net /Balance Interface/Upper Active Balance Group/ACTIVE_TAP2
- removed copper zone on F.Cu, net /Balance Interface/Upper Active Balance Group/ACTIVE_TAP2
- removed copper zone on B.Cu, net /Balance Interface/Upper Active Balance Group/ACTIVE_TAP3
- removed copper zone on F.Cu, net /Balance Interface/Upper Active Balance Group/ACTIVE_TAP3
- removed copper zone on B.Cu, net /Balance Interface/Upper Active Balance Group/ACTIVE_TAP4
- removed copper zone on F.Cu, net /Balance Interface/Upper Active Balance Group/ACTIVE_TAP4
- removed copper zone on B.Cu, net /Balance Interface/Upper Active Balance Group/ACTIVE_TAP5
- removed copper zone on F.Cu, net /Balance Interface/Upper Active Balance Group/ACTIVE_TAP5
- removed copper zone on B.Cu, net /Balance Interface/Upper Active Balance Group/BOOST
- removed copper zone on F.Cu, net /Balance Interface/Upper Active Balance Group/BOOST
- removed copper zone on B.Cu, net /Balance Interface/V+
- removed copper zone on F.Cu, net /Balance Interface/V+
- removed copper zone on B.Cu, net /UPPER_GND
- removed copper zone on F.Cu, net /UPPER_GND
- removed copper zone on B.Cu, net Net-(C108-Pad1)
- removed copper zone on B.Cu, net Net-(C109-Pad1)
- removed copper zone on B.Cu, net Net-(C120-Pad1)
- removed copper zone on B.Cu, net Net-(C121-Pad1)
- removed copper zone on B.Cu, net Net-(C132-Pad1)
- removed copper zone on B.Cu, net Net-(C133-Pad1)
- removed copper zone on B.Cu, net Net-(C144-Pad1)
- removed copper zone on B.Cu, net Net-(C145-Pad1)
Other:
- board outline added: 134.8 x 111.9 mm
