File: 211006_lmu_r0/211006_lmu_r0.kicad_pcb (KiCad board)
At the start: 4 copper layers, 134.8 x 111.9 mm, 700 parts, among them IC1 ADS7028QRTERQ1, J1 Conn_02x03_Odd_Even, J11 Conn_ARM_JTAG_SWD_10, J12 Conn_01x03, J13 Conn_02x03_Odd_Even, J14 Conn_01x02, J15 Conn_01x02, J16 Conn_01x02, J17 Conn_01x02, J18 Conn_01x02, J19 Conn_01x02, J2 Conn_02x03_Odd_Even, J20 Conn_01x02, J21 Conn_01x02, J22 Conn_01x02, J23 Conn_01x02, J24 Conn_01x02, J25 Conn_01x02, J3 Conn_02x08_Odd_Even, J4 Conn_01x02, J5 Conn_01x03, J6 Conn_01x03, J7 Conn_01x02, J9 Conn_01x02, K1 G5V-2, Q1 CZT5551, Q11 BSS308PE, Q14 BSS308PE, Q17 BSS308PE, Q2 BSS308PE, Q20 BSS308PE, Q23 BSS308PE, Q26 BSS308PE, Q29 BSS308PE, Q32 BSS308PE, Q35 BSS308PE, Q38 BC817, Q5 BSS308PE, Q8 BSS308PE, SW1 SW_Push, T1 750312504, T10 750312504, T11 750312504, T12 750312504, T13 BUK9K13-60EX, T14 BUK9K13-60EX, T15 BUK9K13-60EX, T16 BUK9K13-60EX, T17 BUK9K13-60EX, T18 BUK9K13-60EX, T19 BUK9K13-60EX, T2 750312504, T20 BUK9K13-60EX, T21 BUK9K13-60EX, T22 BUK9K13-60EX, T23 BUK9K13-60EX, T24 BUK9K13-60EX, T3 750312504, T4 750312504, T5 750312504, T6 750312504, T7 750312504, T8 750312504, T9 750312504, U1 R-78C5.0-1.0, U2 ISO1042DWVR, U3 LTC6811HG-2#PBF, U4 LTC3300ILXE-2#PBF, U5 LTC3300ILXE-2#PBF, U6 ADuM7641A, U7 ADuM7641A, U8 ADuM7641A, U9 STM32F103C8Tx, Y1 Crystal_GND24

Commit message: little bit closer
Parts:
- removed TP104, TP115, TP126, TP137, TP148, TP27, TP38, TP49, TP60, TP71, TP82, TP93: TestPoint, TestPoint:TestPoint_Pad_D1.0mm
- added J8: Conn_01x02, Connector_PinHeader_2.54mm:PinHeader_1x02_P2.54mm_Vertical, F.Cu at (135.6, 110.4)
- moved TP56 14.4 mm to (128.2, 13.3)
- moved TP100 14.4 mm to (176.2, 73.8)
- moved TP111 14.4 mm to (152.8, 76.0)
- moved TP122 14.4 mm to (129.8, 78.2)
- moved TP144 14.4 mm to (138.2, 123.5)
- moved TP155 14.4 mm to (160.4, 125.8)
- moved TP34 14.4 mm to (176.1, 14.0)
- moved TP45 14.4 mm to (152.4, 13.8)
- moved TP67 14.4 mm to (113.1, 58.8)
- moved TP78 14.4 mm to (137.7, 58.4)
- moved TP89 14.4 mm to (162.5, 58.2)
- moved TP133 13.2 mm to (114.8, 121.3)
- moved TP127 11.4 mm to (114.8, 112.2)
- moved TP128 11.0 mm to (114.8, 115.5)
- moved TP134 10.1 mm to (114.8, 118.0)
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Connections:
- D6 pad 1: 0V_ISO -> 0V_HV
- R251 pad 1: 3.3V_ISO -> 5V_HV
Routing:
- net /Balance Interface/Lower Active Balance Group/ACTIVE_TAP3: track 116.2 -> 55.1 mm
- net /Balance Interface/Lower Active Balance Group/ACTIVE_TAP4: track 103.1 -> 55.1 mm
- net /UPPER_GND: track 71.3 -> 109.3 mm, vias 14 -> 20
- net /Balance Interface/Lower Active Balance Group/ACTIVE_TAP5: track 80.4 -> 55.1 mm
- net GND_HV: track 78.2 -> 96.8 mm, vias 17 -> 22
- net /Balance Interface/Lower Active Balance Group/ACTIVE_TAP2: track 121.4 -> 102.9 mm
- net Net-(T12-Pad4): track 0.00 -> 17.5 mm
- net Net-(T11-Pad4): track 0.00 -> 17.5 mm
- net Net-(T6-Pad4): track 0.00 -> 17.5 mm
- net Net-(T9-Pad4): track 0.00 -> 17.5 mm
- net Net-(T7-Pad4): track 0.00 -> 17.5 mm
- net Net-(T3-Pad4): track 0.00 -> 17.5 mm
- net Net-(T1-Pad4): track 0.00 -> 17.5 mm
- net Net-(T5-Pad4): track 0.00 -> 17.5 mm
- net Net-(T2-Pad4): track 0.00 -> 17.5 mm
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- added copper zone on B.Cu, net Net-(C108-Pad1)
- added copper zone on B.Cu, net Net-(C109-Pad1)
- added copper zone on B.Cu, net Net-(C120-Pad1)
- added copper zone on B.Cu, net Net-(C121-Pad1)
- added copper zone on B.Cu, net Net-(C132-Pad1)
- added copper zone on B.Cu, net Net-(C133-Pad1)
- added copper zone on B.Cu, net Net-(C144-Pad1)
- added copper zone on B.Cu, net Net-(C145-Pad1)
Other:
- board outline removed

Commit message: sorted header location
Parts:
- removed J14, J15, J16, J17, J18, J19, J20, J21, J22, J23, J24, J25: Conn_01x02, Connector_Molex:Molex_Mini-Fit_Jr_5566-02A_2x01_P4.20mm_Vertical
- added J10: LOWER_BANK, Connector_Phoenix_MSTB:PhoenixContact_MSTBVA_2,5_8-G-5,08_1x08_P5.08mm_Vertical, F.Cu at (189.5, 84.7)
- F10, F11, F12, F13, F14, F2, F3, F4, F5, F6, F7, F8, F9, R119, R120, R121, R122, R123, R124, R125, R126, R23, R24, TP10, TP11, TP12, TP13, TP14, TP15, TP16, TP17, TP18, TP19, TP20, TP8, TP9: moved to B.Cu
- J4: value Conn_01x02 -> UPPER_BANK; footprint Connector_Molex:Molex_Mini-Fit_Jr_5566-02A_2x01_P4.20mm_Vertical -> Connector_Phoenix_MSTB:PhoenixContact_MSTBVA_2,5_6-G_1x06_P5.00mm_Vertical
- K1: value G5V-2 -> G5V-2 DC-3
- R252: footprint Resistor_SMD:R_0603_1608Metric_Pad0.98x0.95mm_HandSolder -> Resistor_SMD:R_1206_3216Metric_Pad1.30x1.75mm_HandSolder
- moved R218 335.0 mm to (-39.8, 91.0), turned to 180 degrees
- moved R219 334.3 mm to (-39.8, 92.4), turned to 180 degrees
- moved R220 333.7 mm to (-39.8, 93.8), turned to 180 degrees
- moved R221 333.1 mm to (-39.8, 95.2), turned to 180 degrees
- moved R222 332.5 mm to (-39.8, 96.6), turned to 180 degrees
- moved R223 331.9 mm to (-39.8, 98.0), turned to 180 degrees
- moved R206 329.1 mm to (-39.8, 105.2), turned to 180 degrees
- moved R207 328.6 mm to (-39.8, 106.6), turned to 180 degrees
- moved R208 328.1 mm to (-39.8, 108.0), turned to 180 degrees
- moved R209 327.6 mm to (-39.8, 109.4), turned to 180 degrees
- moved R210 327.1 mm to (-39.8, 110.8), turned to 180 degrees
- moved R211 326.6 mm to (-39.8, 112.2), turned to 180 degrees
- moved C178 326.2 mm to (-35.4, 97.5), turned to 180 degrees
- moved R230 324.9 mm to (-39.5, 116.2), turned to 180 degrees
- moved R231 324.5 mm to (-39.5, 117.6), turned to 180 degrees
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Connections:
- C25 pad 1: +5V_HV -> /Balance Interface/VREG
- J4 pad 2: /Balance Interface/TAP12 -> /Balance Interface/TAP11
- J5 pad 3: +5V_HV -> /Balance Interface/VREG
- J6 pad 3: +5V_HV -> /Balance Interface/VREG
- Q1 pad 3: +5V_HV -> /Balance Interface/VREG
- R119 pad 1: +5V_HV -> /Balance Interface/VREG
- R121 pad 1: +5V_HV -> /Balance Interface/VREG
- R123 pad 1: +5V_HV -> /Balance Interface/VREG
- R125 pad 1: +5V_HV -> /Balance Interface/VREG
- R22 pad 1: +5V_HV -> /Balance Interface/VREG
- R252 pad 1: +5V_HV -> /Balance Interface/VREG
- TP25 pad 1: +5V_HV -> /Balance Interface/VREG
- U3 pad 37: +5V_HV -> /Balance Interface/VREG
Routing:
- net /Balance Interface/Upper Active Balance Group/BOOST: track 70.5 -> 166.7 mm
- net /Balance Interface/Lower Active Balance Group/BOOST: track 70.5 -> 166.7 mm
- net /Balance Interface/Upper Active Balance Group/ACTIVE_TAP3: track 55.1 -> 121.0 mm
- net /Balance Interface/Lower Active Balance Group/ACTIVE_TAP3: track 55.1 -> 120.9 mm
- net /Balance Interface/Upper Active Balance Group/ACTIVE_TAP2: track 55.1 -> 120.2 mm
- net /Balance Interface/Upper Active Balance Group/ACTIVE_TAP1: track 55.1 -> 100.6 mm
- net /Balance Interface/Lower Active Balance Group/ACTIVE_TAP4: track 55.1 -> 98.3 mm
- net /Balance Interface/Upper Active Balance Group/ACTIVE_TAP4: track 55.1 -> 98.3 mm
- net /UPPER_GND: track 109.3 -> 143.4 mm, vias 20 -> 24
- net /Balance Interface/Lower Active Balance Group/ACTIVE_TAP5: track 55.1 -> 79.4 mm
- net GND_HV: track 96.8 -> 120.6 mm, vias 22 -> 25
- net /Balance Interface/Upper Active Balance Group/ACTIVE_TAP5: track 55.1 -> 78.7 mm
- net /Balance Interface/VREG_UPPER: track 0.00 -> 20.3 mm, vias 0 -> 3
- net /Balance Interface/Lower Active Balance Group/ACTIVE_TAP1: track 80.5 -> 98.0 mm
- net /Balance Interface/Lower Active Balance Group/ACTIVE_TAP2: track 102.9 -> 119.3 mm
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Other:
- board outline added: 152 x 126.6 mm

Commit message: trying out a quick thing, recover
Parts:
- C17, C18, C19, C20, C21, C22, C23, C24, C7, R10, R11, R12, R13, R14, R15, R16, R17, R18, R19, R20, R21, R3, R4, R6, R7, R8, R9: moved to B.Cu
- moved C3 255.7 mm to (138.4, 77.7), turned to 0 degrees
- moved L1 246.5 mm to (138.7, 70.7), turned to 0 degrees
- moved C1 244.8 mm to (127.1, 73.2), turned to 180 degrees
- moved C2 237.1 mm to (138.4, 63.7), turned to 0 degrees
- moved D2 233.7 mm to (128.6, 64.5), turned to 180 degrees
- moved D1 229.4 mm to (134.3, 59.4), turned to 0 degrees
- moved J3 224.4 mm to (124.7, 149.7), turned to 0 degrees
- moved F1 223.0 mm to (125.9, 57.5), turned to -90 degrees
- moved J2 217.9 mm to (140.7, 48.1), turned to 180 degrees
- moved TP1 214.8 mm to (125.9, 51.4), turned to -90 degrees
- moved C17 214.2 mm to (125.5, 145.9), turned to 180 degrees
- moved C18 212.5 mm to (129.7, 145.9), turned to 180 degrees
- moved R6 212.2 mm to (125.6, 144.4), turned to 0 degrees
- moved C19 211.2 mm to (133.9, 145.9), turned to 180 degrees
- moved R7 211.1 mm to (125.6, 143.0), turned to 180 degrees
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Connections:
- net 0V_ISO renamed GND_ISO
- net 3.3V_ISO renamed +3V3_ISO
- C16 pad 1: 5V_HV -> +5V_HV
- C17 pad 1: 0V_HV -> GND_HV
- C18 pad 1: 0V_HV -> GND_HV
- C19 pad 1: 0V_HV -> GND_HV
- C20 pad 1: 0V_HV -> GND_HV
- C21 pad 1: 0V_HV -> GND_HV
- C22 pad 1: 0V_HV -> GND_HV
- C23 pad 1: 0V_HV -> GND_HV
- C24 pad 1: 0V_HV -> GND_HV
- C25 pad 2: 0V_HV -> GND_HV
- C26 pad 2: 0V_HV -> GND_HV
- C27 pad 2: 0V_HV -> GND_HV
- C28 pad 1: 0V_HV -> GND_HV
- C29 pad 2: 0V_HV -> GND_HV
- C78 pad 1: 5V_HV -> +5V_HV
- C78 pad 2: 0V_HV -> GND_HV
- D6 pad 1: 0V_HV -> GND_HV
- IC1 pad 10: 5V_HV -> +5V_HV
- J3 pad 10: 0V_HV -> GND_HV
- J3 pad 11: 0V_HV -> GND_HV
- J3 pad 12: 0V_HV -> GND_HV
- J3 pad 13: 0V_HV -> GND_HV
- J3 pad 14: 0V_HV -> GND_HV
- J3 pad 15: 0V_HV -> GND_HV
- J3 pad 16: 0V_HV -> GND_HV
- J3 pad 9: 0V_HV -> GND_HV
- J5 pad 1: 0V_HV -> GND_HV
- J6 pad 1: 0V_HV -> GND_HV
- PS2 pad 4: 0V_HV -> GND_HV
- PS2 pad 5: 5V_HV -> +5V_HV
- R10 pad 2: 5V_HV -> +5V_HV
- R12 pad 2: 5V_HV -> +5V_HV
- R14 pad 2: 5V_HV -> +5V_HV
- R16 pad 2: 5V_HV -> +5V_HV
- R18 pad 2: 5V_HV -> +5V_HV
- R20 pad 2: 5V_HV -> +5V_HV
- R24 pad 1: 0V_HV -> GND_HV
- R251 pad 1: 5V_HV -> +5V_HV
- R6 pad 2: 5V_HV -> +5V_HV
- R8 pad 2: 5V_HV -> +5V_HV
- TP30 pad 1: 5V_HV -> +5V_HV
- TP33 pad 1: 0V_HV -> GND_HV
- U3 pad 30: 0V_HV -> GND_HV
- U3 pad 31: 0V_HV -> GND_HV
Routing:
- net GND_HV: track 120.6 -> 146.3 mm, vias 25 -> 34
- net +5V_HV: track 0.00 -> 18.8 mm, vias 0 -> 8
- net /Balance Interface/Lower Active Balance Group/SI3: track 25.6 -> 8.85 mm
- net /Temperature Sensor/TmpOut7: track 0.00 -> 16.1 mm, vias 0 -> 1
- net /Temperature Sensor/TmpOut0: track 0.00 -> 14.6 mm, vias 0 -> 1
- net Net-(C28-Pad2): track 0.00 -> 13.2 mm
- net /Balance Interface/Lower Active Balance Group/PG3: track 17.3 -> 4.06 mm, vias 2 -> 1
- net /Balance Interface/Lower Active Balance Group/PG4: track 17.3 -> 5.26 mm
- net /Temperature Sensor/TmpOut6: track 0.00 -> 11.9 mm, vias 0 -> 1
- net /Balance Interface/VREG: track 0.00 -> 11.8 mm
- net /Balance Interface/Lower Active Balance Group/SI4: track 24.6 -> 12.8 mm
- net /Balance Interface/Lower Active Balance Group/SG4: track 17.6 -> 6.45 mm
- net /Balance Interface/Lower Active Balance Group/SG3: track 17.7 -> 7.42 mm
- net /Temperature Sensor/TmpOut1: track 0.00 -> 10.2 mm, vias 0 -> 1
- net /Balance Interface/Lower Active Balance Group/PI3: track 17.5 -> 7.23 mm, vias 2 -> 1
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Other:
- board size 152 x 126.6 mm -> 155.5 x 126.7 mm

Commit message: copying layout
Parts:
- moved C8 153.5 mm to (138.4, 107.8), turned to 0 degrees
- moved R3 151.6 mm to (137.6, 109.5), turned to 180 degrees
- moved C9 151.5 mm to (138.4, 113.0), turned to 0 degrees
- moved R4 150.9 mm to (137.6, 111.4), turned to 0 degrees
- moved L2 148.8 mm to (135.8, 110.4), turned to -90 degrees
- moved C7 146.4 mm to (134.0, 110.5), turned to 0 degrees
- moved C10 146.2 mm to (133.1, 107.8), turned to 180 degrees
- moved C11 144.1 mm to (133.1, 113.0), turned to 180 degrees
- moved D5 141.0 mm to (130.1, 110.4), turned to 180 degrees
- moved R5 138.3 mm to (129.1, 114.1), turned to 90 degrees
- moved R1 131.5 mm to (125.0, 117.4), turned to -90 degrees
- moved D3 129.1 mm to (123.2, 117.3), turned to -90 degrees
- moved U2 128.5 mm to (120.8, 110.4), turned to 0 degrees
- moved C5 128.3 mm to (123.5, 121.5), turned to 0 degrees
- moved C65 124.2 mm to (248.5, 165.2), turned to 0 degrees
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Connections:
- R127 pad 2: /Balance Interface/S6 -> /Balance Interface/C6
- R27 pad 2: /Balance Interface/S12 -> /Balance Interface/C12
- U4 pad 36: /Balance Interface/S11 -> /Balance Interface/C11
- U4 pad 39: /Balance Interface/S12 -> /Balance Interface/C12
- U5 pad 36: /Balance Interface/S5 -> /Balance Interface/C5
- U5 pad 39: /Balance Interface/S6 -> /Balance Interface/C6
Routing:
- net /Balance Interface/Upper Active Balance Group/SG1: track 14.1 -> 111.2 mm
- net /Balance Interface/Upper Active Balance Group/SI1: track 20.6 -> 102.8 mm
- net /Balance Interface/Upper Active Balance Group/PI6: track 13.7 -> 91.8 mm
- net /Balance Interface/Upper Active Balance Group/SG6: track 14.5 -> 89.6 mm
- net /Balance Interface/Upper Active Balance Group/SI6: track 24.2 -> 99.1 mm, vias 1 -> 2
- net /Balance Interface/Upper Active Balance Group/SG2: track 13.9 -> 87.5 mm, vias 1 -> 2
- net /Balance Interface/Upper Active Balance Group/PG6: track 15.2 -> 86.3 mm
- net /Balance Interface/Upper Active Balance Group/PG1: track 18.7 -> 83.9 mm
- net /Balance Interface/Upper Active Balance Group/PI1: track 18.8 -> 82.2 mm
- net /Balance Interface/S7: track 0.96 -> 61.2 mm
- net /Balance Interface/Upper Active Balance Group/SI5: track 22.4 -> 79.8 mm, vias 1 -> 2
- net /Balance Interface/Upper Active Balance Group/SI2: track 22.9 -> 79.9 mm, vias 1 -> 2
- net /Balance Interface/Upper Active Balance Group/SG5: track 14.5 -> 70.6 mm, vias 1 -> 2
- net /Balance Interface/S12: track 9.05 -> 58.5 mm, vias 3 -> 1
- net /Balance Interface/Upper Active Balance Group/PI5: track 17.8 -> 67.2 mm
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Other:
- board size 155.5 x 126.7 mm -> 199.4 x 126.7 mm

Commit message: Update 211006_lmu_r0.kicad_pcb
Parts:
- moved R202 72.5 mm to (240.5, 229.2), turned to 180 degrees
- moved C174 71.1 mm to (243.9, 229.2), turned to 180 degrees
- moved C150 69.1 mm to (225.9, 226.9)
- moved R178 69.1 mm to (222.5, 226.9)
- moved C114 69.0 mm to (264.6, 228.9)
- moved R142 69.0 mm to (268.0, 228.9)
- moved C126 68.6 mm to (256.8, 229.0)
- moved R154 68.6 mm to (260.1, 229.0)
- moved C138 68.3 mm to (248.3, 229.0)
- moved R166 68.3 mm to (251.7, 229.0)
- moved R190 65.8 mm to (230.8, 227.2), turned to 180 degrees
- moved C162 63.8 mm to (234.2, 227.2), turned to 180 degrees
- moved C29 46.4 mm to (116.0, 68.8)
- moved J5 46.4 mm to (101.4, 51.9)
- moved R121 46.4 mm to (115.6, 59.1)
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Routing:
- net /Balance Interface/Lower Active Balance Group/SG1: track 6.25 -> 109.7 mm
- net /Balance Interface/Lower Active Balance Group/SI1: track 3.77 -> 102.8 mm
- net /Balance Interface/Lower Active Balance Group/PI6: track 3.51 -> 91.8 mm, vias 1 -> 2
- net /Balance Interface/Lower Active Balance Group/PG6: track 2.04 -> 86.3 mm, vias 1 -> 2
- net /Balance Interface/Lower Active Balance Group/SI6: track 7.47 -> 90.4 mm
- net /Balance Interface/Lower Active Balance Group/PG1: track 5.54 -> 83.9 mm, vias 1 -> 2
- net /Balance Interface/Lower Active Balance Group/SG2: track 7.77 -> 85.8 mm, vias 2 -> 1
- net /Balance Interface/Lower Active Balance Group/SG6: track 4.20 -> 81.7 mm
- net /Balance Interface/Lower Active Balance Group/PI1: track 8.59 -> 82.2 mm, vias 1 -> 2
- net /Balance Interface/Lower Active Balance Group/SI2: track 7.66 -> 78.3 mm, vias 2 -> 1
- net /Balance Interface/Lower Active Balance Group/SI5: track 7.81 -> 69.4 mm
- net /Balance Interface/S1: track 0.96 -> 61.2 mm
- net /Balance Interface/Lower Active Balance Group/PI5: track 7.57 -> 67.2 mm, vias 1 -> 2
- net /Balance Interface/Lower Active Balance Group/PG2: track 6.33 -> 64.9 mm, vias 1 -> 2
- net /Balance Interface/S6: track 0.96 -> 58.5 mm
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- removed copper zone on B.Cu, net Net-(C108-Pad1)
- removed copper zone on F.Cu, net Net-(C108-Pad1)
- removed copper zone on B.Cu, net Net-(C109-Pad1)
- removed copper zone on F.Cu, net Net-(C109-Pad1)
- removed copper zone on B.Cu, net Net-(C120-Pad1)
- removed copper zone on F.Cu, net Net-(C120-Pad1)
- removed copper zone on B.Cu, net Net-(C121-Pad1)
- removed copper zone on F.Cu, net Net-(C121-Pad1)
- removed copper zone on B.Cu, net Net-(C132-Pad1)
- removed copper zone on F.Cu, net Net-(C132-Pad1)
- removed copper zone on B.Cu, net Net-(C133-Pad1)
- removed copper zone on F.Cu, net Net-(C133-Pad1)
- removed copper zone on B.Cu, net Net-(C144-Pad1)
- removed copper zone on F.Cu, net Net-(C144-Pad1)
- removed copper zone on B.Cu, net Net-(C145-Pad1)
- removed copper zone on F.Cu, net Net-(C145-Pad1)
- removed copper zone on B.Cu, net Net-(C156-Pad1)
- removed copper zone on F.Cu, net Net-(C156-Pad1)
- removed copper zone on B.Cu, net Net-(C157-Pad1)
- removed copper zone on F.Cu, net Net-(C157-Pad1)
- removed copper zone on B.Cu, net Net-(C168-Pad1)
- removed copper zone on F.Cu, net Net-(C168-Pad1)
- removed copper zone on B.Cu, net Net-(C169-Pad1)
- removed copper zone on F.Cu, net Net-(C169-Pad1)
Other:
- board outline removed
