File: 211006_lmu_r0/file6196A5FB.kicad_sch (KiCad schematic)
At the start: 7 parts, among them U5 LTC3300ILXE-2#PBF

Commit message: Updated lmu project with relative library paths and fixed broken symbols
Parts:
- U5: AVAILABILITY (none) -> Unavailable; MANUFACTURER (none) -> Linear Technology; MP (none) -> LTC3300ILXE-2#PBF; PACKAGE (none) -> LQFP-48 Linear Technology; STANDARD (none) -> IPC-7351B
Connections:
- net A0: now also U5.43 (A0)
- net A1: now also U5.44 (A1)
- net A2: now also U5.45 (A2)
- net A3: now also U5.46 (A3)
- net A4: now also U5.47 (A4)
- net ACTIVE_TAP0: now also U5.15 (CTRL), U5.21 (V-), U5.49 (V-)
- net C1: now also U5.24 (C1)
- net C2: now also U5.27 (C2)
- net C3: now also U5.30 (C3)
- net C4: now also U5.33 (C4)
- net C5: now also U5.36 (C5)
- net C6: now also U5.39 (C6)
- net PG1: now also U5.23 (G1P)
- net PG2: now also U5.26 (G2P)
- net PG3: now also U5.29 (G3P)
- net PG4: now also U5.32 (G4P)
- net PG5: now also U5.35 (G5P)
- net PG6: now also U5.38 (G6P)
- net PI1: now also U5.22 (I1P)
- net PI2: now also U5.25 (I2P)
- net PI3: now also U5.28 (I3P)
- net PI4: now also U5.31 (I4P)
- net PI5: now also U5.34 (I5P)
- net PI6: now also U5.37 (I6P)
- net SCKI: now also U5.17 (SCKI)
- net SDI: now also U5.18 (SDI)
- net SDO: now also U5.19 (SDO)
- net SG1: now also U5.11 (G1S)
- net SG2: now also U5.9 (G2S)
- net SG3: now also U5.7 (G3S)
- net SG4: now also U5.5 (G4S)
- net SG5: now also U5.3 (G5S)
- net SG6: now also U5.1 (G6S)
- net SI1: now also U5.12 (I1S)
- net SI2: now also U5.10 (I2S)
- net SI3: now also U5.8 (I3S)
- net SI4: now also U5.6 (I4S)
- net SI5: now also U5.4 (I5S)
- net SI6: now also U5.2 (I6S)
- net VREG: now also U5.42 (BOOST), U5.48 (VREG)
- net WDT: now also U5.20 (WDT)
- net nCSBI: now also U5.16 (~{CSBI})
- net at R129.1: now also U5.13 (RTONS)
- net at C103.2, D27.1 (K): now also U5.41 (BOOSTN)
- net at C103.1: now also U5.40 (BOOSTP)
- net at R130.1: now also U5.14 (RTONP)
Changed lines of the file:
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@@
       (effects (font (size 1.27 1.27)) (justify left bottom) hide)
     )
-    (property "PACKAGE" "" (id 4) (at 204.47 86.36 0)
+    (property "PACKAGE" "LQFP-48 Linear Technology" (id 4) (at 204.47 86.36 0)
       (effects (font (size 1.27 1.27)) (justify left bottom) hide)
     )
@@
       (effects (font (size 1.27 1.27)) (justify left bottom) hide)
     )
-    (property "STANDARD" "" (id 6) (at 204.47 86.36 0)
+    (property "STANDARD" "IPC-7351B" (id 6) (at 204.47 86.36 0)
       (effects (font (size 1.27 1.27)) (justify left bottom) hide)
     )
@@
       (effects (font (size 1.27 1.27)) (justify left bottom) hide)
     )
-    (property "MP" "" (id 8) (at 204.47 86.36 0)
+    (property "MP" "LTC3300ILXE-2#PBF" (id 8) (at 204.47 86.36 0)
       (effects (font (size 1.27 1.27)) (justify left bottom) hide)
     )
@@
       (effects (font (size 1.27 1.27)) (justify left bottom) hide)
     )
-    (property "MANUFACTURER" "" (id 10) (at 204.47 86.36 0)
+    (property "MANUFACTURER" "Linear Technology" (id 10) (at 204.47 86.36 0)
       (effects (font (size 1.27 1.27)) (justify left bottom) hide)
     )
-    (property "AVAILABILITY" "" (id 11) (at 204.47 86.36 0)
+    (property "AVAILABILITY" "Unavailable" (id 11) (at 204.47 86.36 0)
       (effects (font (size 1.27 1.27)) (justify left bottom) hide)
     )
@@
       (effects (font (size 1.27 1.27)) hide)
     )
+    (pin "1")
+    (pin "10")
+    (pin "11")
+    (pin "12")
+    (pin "13")
+    (pin "14")
+    (pin "15")
+    (pin "16")
+    (pin "17")
+    (pin "18")
+    (pin "19")
+    (pin "2")
+    (pin "20")
+    (pin "21")
+    (pin "22")
+    (pin "23")
+    (pin "24")
+    (pin "25")
+    (pin "26")
+    (pin "27")
+    (pin "28")
+    (pin "29")
+    (pin "3")
+    (pin "30")
+    (pin "31")
+    (pin "32")
+    (pin "33")
+    (pin "34")
+    (pin "35")
+    (pin "36")
+    (pin "37")
+    (pin "38")
+    (pin "39")
+    (pin "4")
+    (pin "40")
+    (pin "41")
+    (pin "42")
+    (pin "43")
+    (pin "44")
+    (pin "45")
+    (pin "46")
+    (pin "47")
+    (pin "48")
+    (pin "49")
+    (pin "5")
+    (pin "6")
+    (pin "7")
+    (pin "8")
+    (pin "9")
   )
   (symbol (lib_id "Device:R") (at 269.24 114.3 0)

Commit message: Updated some components to make sourcing easier
Parts:
- C103, R127, R128, R129, R130: Manufacturer (none) -> -; Part Number (none) -> -
Changed lines of the file:
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@@
+      (effects (font (size 1.27 1.27)) hide)
+    )
+    (property "Part Number" "-" (id 4) (at 260.35 114.3 0)
+      (effects (font (size 1.27 1.27)) hide)
+    )
+    (property "Manufacturer" "-" (id 5) (at 260.35 114.3 0)
       (effects (font (size 1.27 1.27)) hide)
     )
@@
       (effects (font (size 1.27 1.27)) hide)
     )
+    (property "Part Number" "-" (id 4) (at 240.03 132.08 0)
+      (effects (font (size 1.27 1.27)) hide)
+    )
+    (property "Manufacturer" "-" (id 5) (at 240.03 132.08 0)
+      (effects (font (size 1.27 1.27)) hide)
+    )
     (pin "1")
     (pin "2")
@@
     )
     (property "Datasheet" "~" (id 3) (at 248.92 115.57 0)
+      (effects (font (size 1.27 1.27)) hide)
+    )
+    (property "Part Number" "-" (id 4) (at 248.92 115.57 0)
+      (effects (font (size 1.27 1.27)) hide)
+    )
+    (property "Manufacturer" "-" (id 5) (at 248.92 115.57 0)
       (effects (font (size 1.27 1.27)) hide)
     )
@@
       (effects (font (size 1.27 1.27)) hide)
     )
+    (property "Part Number" "-" (id 4) (at 269.24 114.3 0)
+      (effects (font (size 1.27 1.27)) hide)
+    )
+    (property "Manufacturer" "-" (id 5) (at 269.24 114.3 0)
+      (effects (font (size 1.27 1.27)) hide)
+    )
     (pin "1")
     (pin "2")
@@
       (effects (font (size 1.27 1.27)) hide)
     )
+    (property "Part Number" "-" (id 4) (at 255.27 83.82 0)
+      (effects (font (size 1.27 1.27)) hide)
+    )
+    (property "Manufacturer" "-" (id 5) (at 255.27 83.82 0)
+      (effects (font (size 1.27 1.27)) hide)
+    )
