File: 211006_lmu_r0/file6196A5FB.kicad_sch (KiCad schematic)
At the start: 7 parts, among them U4 LTC3300ILXE-2#PBF

Commit message: fixed footprints for headers, started planning out zones
Connections:
- net RTONS: now reaches R29.1, U4.13 (RTONS)
- net RTONP: now reaches R30.1, U4.14 (RTONP)
Changed lines of the file:
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@@
+    (effects (font (size 1.27 1.27)) (justify left bottom))
+  )
+  (label "RTONS" (at 228.6 109.22 0)
     (effects (font (size 1.27 1.27)) (justify left bottom))
   )
@@
     (effects (font (size 1.27 1.27)) (justify left bottom))
   )
+  (label "RTONP" (at 228.6 106.68 0)
+    (effects (font (size 1.27 1.27)) (justify left bottom))
+  )

Commit message: Lots of routing and placing, according to planned layout
Parts:
- renumbered C30 to C103, D14 to D27, R27 to R127, R28 to R128, R29 to R129, R30 to R130, U4 to U5
Changed lines of the file:
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@@
   (symbol (lib_id "Device:R") (at 260.35 114.3 0)
     (in_bom yes) (on_board yes)
-    (property "Reference" "R29" (id 0) (at 262.128 113.1316 0)
+    (property "Reference" "R129" (id 0) (at 262.128 113.1316 0)
       (effects (font (size 1.27 1.27)) (justify left))
     )
@@
   (symbol (lib_id "Device:D_Schottky") (at 240.03 124.46 270)
     (in_bom yes) (on_board yes)
-    (property "Reference" "D14" (id 0) (at 242.062 123.2916 90)
+    (property "Reference" "D27" (id 0) (at 242.062 123.2916 90)
       (effects (font (size 1.27 1.27)) (justify left))
     )
@@
   (symbol (lib_id "Device:R") (at 240.03 132.08 0)
     (in_bom yes) (on_board yes)
-    (property "Reference" "R27" (id 0) (at 241.808 130.9116 0)
+    (property "Reference" "R127" (id 0) (at 241.808 130.9116 0)
       (effects (font (size 1.27 1.27)) (justify left))
     )
@@
   (symbol (lib_id "Device:C") (at 248.92 115.57 0)
     (in_bom yes) (on_board yes)
-    (property "Reference" "C30" (id 0) (at 251.841 114.4016 0)
+    (property "Reference" "C103" (id 0) (at 251.841 114.4016 0)
       (effects (font (size 1.27 1.27)) (justify left))
     )
@@
   (symbol (lib_id "LTC3300ILXE-2_PBF:LTC3300ILXE-2#PBF") (at 204.47 86.36 0)
     (in_bom yes) (on_board yes)
-    (property "Reference" "U4" (id 0) (at 204.47 46.482 0))
+    (property "Reference" "U5" (id 0) (at 204.47 46.482 0))
     (property "Value" "LTC3300ILXE-2#PBF" (id 1) (at 204.47 48.7934 0))
     (property "Footprint" "QFP50P900X900X160-49N" (id 2) (at 204.47 86.36 0)
@@
   (symbol (lib_id "Device:R") (at 269.24 114.3 0)
     (in_bom yes) (on_board yes)
-    (property "Reference" "R30" (id 0) (at 271.018 113.1316 0)
+    (property "Reference" "R130" (id 0) (at 271.018 113.1316 0)
       (effects (font (size 1.27 1.27)) (justify left))
     )
@@
   (symbol (lib_id "Device:R") (at 255.27 83.82 0)
     (in_bom yes) (on_board yes)
-    (property "Reference" "R28" (id 0) (at 257.048 82.6516 0)
-      (effects (font (size 1.27 1.27)) (justify left))
-    )
+    (property "Reference" "R128" (id 0) (at 257.048 82.6516 0)
+      (effects (font (size 1.27 1.27)) (justify left))
+    )

Commit message: final merge before branch
Parts:
- renumbered C103 to C30, D27 to D14, R127 to R27, R128 to R28, R129 to R29, R130 to R30, U5 to U4
Other:
- note added: "internally regulates 4.8V from c6, self powered device!"
Changed lines of the file:
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@@
     (stroke (width 0) (type default) (color 0 0 0 0))
   )
+  (text "internally regulates 4.8V from c6, self powered device!"
+    (at 220.98 41.91 0)
+    (effects (font (size 1.27 1.27)) (justify left bottom))
+  )
   (label "PI4" (at 119.38 95.25 0)
     (effects (font (size 1.27 1.27)) (justify left bottom))
@@
   (symbol (lib_id "Device:R") (at 260.35 114.3 0)
     (in_bom yes) (on_board yes)
-    (property "Reference" "R129" (id 0) (at 262.128 113.1316 0)
+    (property "Reference" "R29" (id 0) (at 262.128 113.1316 0)
       (effects (font (size 1.27 1.27)) (justify left))
     )
@@
   (symbol (lib_id "Device:D_Schottky") (at 240.03 124.46 270)
     (in_bom yes) (on_board yes)
-    (property "Reference" "D27" (id 0) (at 242.062 123.2916 90)
+    (property "Reference" "D14" (id 0) (at 242.062 123.2916 90)
       (effects (font (size 1.27 1.27)) (justify left))
     )
@@
   (symbol (lib_id "Device:R") (at 240.03 132.08 0)
     (in_bom yes) (on_board yes)
-    (property "Reference" "R127" (id 0) (at 241.808 130.9116 0)
+    (property "Reference" "R27" (id 0) (at 241.808 130.9116 0)
       (effects (font (size 1.27 1.27)) (justify left))
     )
@@
   (symbol (lib_id "Device:C") (at 248.92 115.57 0)
     (in_bom yes) (on_board yes)
-    (property "Reference" "C103" (id 0) (at 251.841 114.4016 0)
+    (property "Reference" "C30" (id 0) (at 251.841 114.4016 0)
       (effects (font (size 1.27 1.27)) (justify left))
     )
@@
   (symbol (lib_id "LTC3300ILXE-2_PBF:LTC3300ILXE-2#PBF") (at 204.47 86.36 0)
     (in_bom yes) (on_board yes)
-    (property "Reference" "U5" (id 0) (at 204.47 46.482 0))
+    (property "Reference" "U4" (id 0) (at 204.47 46.482 0))
     (property "Value" "LTC3300ILXE-2#PBF" (id 1) (at 204.47 48.7934 0))
     (property "Footprint" "QFP50P900X900X160-49N" (id 2) (at 204.47 86.36 0)
@@
   (symbol (lib_id "Device:R") (at 269.24 114.3 0)
     (in_bom yes) (on_board yes)
-    (property "Reference" "R130" (id 0) (at 271.018 113.1316 0)
+    (property "Reference" "R30" (id 0) (at 271.018 113.1316 0)
       (effects (font (size 1.27 1.27)) (justify left))
     )
@@
   (symbol (lib_id "Device:R") (at 255.27 83.82 0)
     (in_bom yes) (on_board yes)
-    (property "Reference" "R128" (id 0) (at 257.048 82.6516 0)
-      (effects (font (size 1.27 1.27)) (justify left))
-    )
+    (property "Reference" "R28" (id 0) (at 257.048 82.6516 0)
+      (effects (font (size 1.27 1.27)) (justify left))
+    )

Commit message: updated pcb still need to find j11
Parts:
- added C?: 1u, Capacitor_SMD:C_0805_2012Metric_Pad1.18x1.45mm_HandSolder, symbol Device:C
- renumbered C30 to C103, D14 to D27, R27 to R127, R28 to R128, R29 to R129, R30 to R130, U4 to U5
Connections:
- net ACTIVE_TAP0: now also C?.2
- net VREG: now also C?.1
Other:
- sheet Active_Passive_Balance_Filter renamed Balance Circuit 6
- sheet sheet6196DB49 renamed Balance Circuit 5
- sheet sheet6196F027 renamed Balance Circuit 4
- sheet sheet6196F028 renamed Balance Circuit 3
- sheet sheet6196F9A3 renamed Balance Circuit 2
- sheet sheet6196F9A4 renamed Balance Circuit 1
Changed lines of the file:
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@@
+    (stroke (width 0) (type default) (color 0 0 0 0))
+  )
+  (wire (pts (xy 245.11 62.23) (xy 243.84 60.96))
     (stroke (width 0) (type default) (color 0 0 0 0))
   )
@@
     (stroke (width 0) (type default) (color 0 0 0 0))
   )
-  (wire (pts (xy 227.33 53.34) (xy 232.41 53.34))
+  (wire (pts (xy 227.33 53.34) (xy 243.84 53.34))
     (stroke (width 0) (type default) (color 0 0 0 0))
   )
@@
     (effects (font (size 1.27 1.27)) (justify left bottom))
   )
-  (label "VREG" (at 232.41 53.34 0)
+  (label "VREG" (at 243.84 53.34 0)
     (effects (font (size 1.27 1.27)) (justify left bottom))
   )
@@
     (effects (font (size 1.27 1.27)) (justify left bottom))
   )
+  (label "BOOST" (at 55.88 17.78 0)
+    (effects (font (size 1.27 1.27)) (justify left bottom))
+  )
   (label "VREG" (at 255.27 76.2 0)
     (effects (font (size 1.27 1.27)) (justify left bottom))
@@
   )
   (label "SG3" (at 119.38 128.27 0)
+    (effects (font (size 1.27 1.27)) (justify left bottom))
+  )
+  (label "V-" (at 245.11 62.23 0)
     (effects (font (size 1.27 1.27)) (justify left bottom))
   )
@@
   (symbol (lib_id "Device:R") (at 260.35 114.3 0)
     (in_bom yes) (on_board yes)
-    (property "Reference" "R29" (id 0) (at 262.128 113.1316 0)
+    (property "Reference" "R129" (id 0) (at 262.128 113.1316 0)
       (effects (font (size 1.27 1.27)) (justify left))
     )
@@
   (symbol (lib_id "Device:D_Schottky") (at 240.03 124.46 270)
     (in_bom yes) (on_board yes)
-    (property "Reference" "D14" (id 0) (at 242.062 123.2916 90)
+    (property "Reference" "D27" (id 0) (at 242.062 123.2916 90)
       (effects (font (size 1.27 1.27)) (justify left))
     )
@@
   (symbol (lib_id "Device:R") (at 240.03 132.08 0)
     (in_bom yes) (on_board yes)
-    (property "Reference" "R27" (id 0) (at 241.808 130.9116 0)
+    (property "Reference" "R127" (id 0) (at 241.808 130.9116 0)
       (effects (font (size 1.27 1.27)) (justify left))
     )
@@
   (symbol (lib_id "Device:C") (at 248.92 115.57 0)
     (in_bom yes) (on_board yes)
-    (property "Reference" "C30" (id 0) (at 251.841 114.4016 0)
+    (property "Reference" "C103" (id 0) (at 251.841 114.4016 0)
       (effects (font (size 1.27 1.27)) (justify left))
     )
@@
   (symbol (lib_id "LTC3300ILXE-2_PBF:LTC3300ILXE-2#PBF") (at 204.47 86.36 0)
     (in_bom yes) (on_board yes)
-    (property "Reference" "U4" (id 0) (at 204.47 46.482 0))
+    (property "Reference" "U5" (id 0) (at 204.47 46.482 0))
     (property "Value" "LTC3300ILXE-2#PBF" (id 1) (at 204.47 48.7934 0))
     (property "Footprint" "QFP50P900X900X160-49N" (id 2) (at 204.47 86.36 0)
@@
   (symbol (lib_id "Device:R") (at 269.24 114.3 0)
     (in_bom yes) (on_board yes)
-    (property "Reference" "R30" (id 0) (at 271.018 113.1316 0)
+    (property "Reference" "R130" (id 0) (at 271.018 113.1316 0)
       (effects (font (size 1.27 1.27)) (justify left))
     )
@@
   (symbol (lib_id "Device:R") (at 255.27 83.82 0)
     (in_bom yes) (on_board yes)
-    (property "Reference" "R28" (id 0) (at 257.048 82.6516 0)
+    (property "Reference" "R128" (id 0) (at 257.048 82.6516 0)
       (effects (font (size 1.27 1.27)) (justify left))
     )
@@
     )
     (property "Manufacturer" "-" (id 5) (at 255.27 83.82 0)
+      (effects (font (size 1.27 1.27)) hide)
+    )
+    (pin "1")
+    (pin "2")
+  )
+  (symbol (lib_id "Device:C") (at 243.84 57.15 0)
+    (in_bom yes) (on_board yes) (fields_autoplaced)
+    (property "Reference" "C?" (id 0) (at 247.65 55.8799 0)
+      (effects (font (size 1.27 1.27)) (justify left))
+    )
+    (property "Value" "1u" (id 1) (at 247.65 58.4199 0)
+      (effects (font (size 1.27 1.27)) (justify left))
+    )
+    (property "Footprint" "Capacitor_SMD:C_0805_2012Metric_Pad1.18x1.45mm_HandSolder" (id 2) (at 244.8052 60.96 0)
+      (effects (font (size 1.27 1.27)) hide)
+    )
+    (property "Datasheet" "~" (id 3) (at 243.84 57.15 0)
       (effects (font (size 1.27 1.27)) hide)
     )
@@
     (stroke (width 0) (type solid) (color 0 0 0 0))
     (fill (color 0 0 0 0.0000))
-    (property "Sheet name" "sheet6196DB49" (id 0) (at 68.58 45.0084 0)
+    (property "Sheet name" "Balance Circuit 5" (id 0) (at 68.58 45.0084 0)
       (effects (font (size 1.27 1.27)) (justify left bottom))
     )
@@
     (stroke (width 0) (type solid) (color 0 0 0 0))
     (fill (color 0 0 0 0.0000))
-    (property "Sheet name" "sheet6196F027" (id 0) (at 68.58 76.7584 0)
+    (property "Sheet name" "Balance Circuit 4" (id 0) (at 68.58 76.7584 0)
       (effects (font (size 1.27 1.27)) (justify left bottom))
     )
@@
     (stroke (width 0) (type solid) (color 0 0 0 0))
     (fill (color 0 0 0 0.0000))
-    (property "Sheet name" "sheet6196F028" (id 0) (at 68.58 107.2384 0)
+    (property "Sheet name" "Balance Circuit 3" (id 0) (at 68.58 107.2384 0)
       (effects (font (size 1.27 1.27)) (justify left bottom))
     )
@@
     (stroke (width 0) (type solid) (color 0 0 0 0))
     (fill (color 0 0 0 0.0000))
-    (property "Sheet name" "sheet6196F9A3" (id 0) (at 68.58 138.9884 0)
+    (property "Sheet name" "Balance Circuit 2" (id 0) (at 68.58 138.9884 0)
       (effects (font (size 1.27 1.27)) (justify left bottom))
     )
@@
     (stroke (width 0) (type solid) (color 0 0 0 0))
     (fill (color 0 0 0 0.0000))
-    (property "Sheet name" "sheet6196F9A4" (id 0) (at 68.58 169.4684 0)
+    (property "Sheet name" "Balance Circuit 1" (id 0) (at 68.58 169.4684 0)
       (effects (font (size 1.27 1.27)) (justify left bottom))
     )
@@
     (stroke (width 0) (type solid) (color 0 0 0 0))
     (fill (color 0 0 0 0.0000))
-    (property "Sheet name" "Active_Passive_Balance_Filter" (id 0) (at 68.58 14.5284 0)
+    (property "Sheet name" "Balance Circuit 6" (id 0) (at 68.58 14.5284 0)
       (effects (font (size 1.27 1.27)) (justify left bottom))
     )

Commit message: fixed issues on higher cells, study into how to route
Parts:
- U4: renamed from U5; footprint QFP50P900X900X160-49N -> LTC3300ILXE-2_PBF:QFP50P900X900X160-49N
- gave numbers to parts that had none: 1
- renumbered C103 to C30, D27 to D14, R127 to R27, R128 to R28, R129 to R29, R130 to R30
Connections:
- net C1 is gone; now on net C_FILTERED1: U4.24 (C1)
- net C2 is gone; now on net C_FILTERED2: U4.27 (C2)
- net C3 is gone; now on net C_FILTERED3: U4.30 (C3)
- net C4 is gone; now on net C_FILTERED4: U4.33 (C4)
- net C5 is gone; now on net S5: U4.36 (C5)
- net C6 is gone; now on net S6: R27.2, U4.39 (C6)
Changed lines of the file:
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@@
   (junction (at 49.53 185.42) (diameter 0) (color 0 0 0 0)
   )
+  (junction (at 228.6 119.38) (diameter 0) (color 0 0 0 0)
+  )
   (junction (at 49.53 53.34) (diameter 0) (color 0 0 0 0)
   )
@@
     (stroke (width 0) (type default) (color 0 0 0 0))
   )
+  (wire (pts (xy 228.6 123.19) (xy 228.6 119.38))
+    (stroke (width 0) (type default) (color 0 0 0 0))
+  )
   (wire (pts (xy 104.14 160.02) (xy 119.38 160.02))
     (stroke (width 0) (type default) (color 0 0 0 0))
@@
     (stroke (width 0) (type default) (color 0 0 0 0))
   )
+  (wire (pts (xy 228.6 119.38) (xy 232.41 119.38))
+    (stroke (width 0) (type default) (color 0 0 0 0))
+  )
   (wire (pts (xy 227.33 101.6) (xy 232.41 101.6))
     (stroke (width 0) (type default) (color 0 0 0 0))
@@
     (stroke (width 0) (type default) (color 0 0 0 0))
   )
+  (wire (pts (xy 231.14 123.19) (xy 228.6 123.19))
+    (stroke (width 0) (type default) (color 0 0 0 0))
+  )
   (wire (pts (xy 240.03 135.89) (xy 240.03 139.7))
     (stroke (width 0) (type default) (color 0 0 0 0))
@@
     (stroke (width 0) (type default) (color 0 0 0 0))
   )
-  (wire (pts (xy 227.33 119.38) (xy 232.41 119.38))
+  (wire (pts (xy 227.33 119.38) (xy 228.6 119.38))
     (stroke (width 0) (type default) (color 0 0 0 0))
   )
@@
     (effects (font (size 1.27 1.27)) (justify left bottom))
   )
+  (label "C6" (at 113.03 17.78 0)
+    (effects (font (size 1.27 1.27)) (justify left bottom))
+  )
   (label "PG1" (at 232.41 58.42 0)
     (effects (font (size 1.27 1.27)) (justify left bottom))
@@
     (effects (font (size 1.27 1.27)) (justify left bottom))
   )
+  (label "C3" (at 113.03 115.57 0)
+    (effects (font (size 1.27 1.27)) (justify left bottom))
+  )
   (label "PG2" (at 119.38 154.94 0)
     (effects (font (size 1.27 1.27)) (justify left bottom))
@@
     (effects (font (size 1.27 1.27)) (justify left bottom))
   )
+  (label "C4" (at 113.03 85.09 0)
+    (effects (font (size 1.27 1.27)) (justify left bottom))
+  )
   (label "C5" (at 232.41 101.6 0)
     (effects (font (size 1.27 1.27)) (justify left bottom))
@@
     (effects (font (size 1.27 1.27)) (justify left bottom))
   )
+  (label "C1" (at 113.03 177.8 0)
+    (effects (font (size 1.27 1.27)) (justify left bottom))
+  )
   (label "PG3" (at 119.38 123.19 0)
     (effects (font (size 1.27 1.27)) (justify left bottom))
@@
     (effects (font (size 1.27 1.27)) (justify left bottom))
   )
+  (label "C2" (at 113.03 147.32 0)
+    (effects (font (size 1.27 1.27)) (justify left bottom))
+  )
   (label "PI2" (at 176.53 63.5 0)
     (effects (font (size 1.27 1.27)) (justify left bottom))
@@
     (effects (font (size 1.27 1.27)) (justify left bottom))
   )
+  (label "C5" (at 113.03 48.26 0)
+    (effects (font (size 1.27 1.27)) (justify left bottom))
+  )
   (label "C2" (at 232.41 93.98 0)
     (effects (font (size 1.27 1.27)) (justify left bottom))
@@
     (effects (font (size 1.27 1.27)) (justify left))
   )
-  (hierarchical_label "C_FILTERED4" (shape input) (at 119.38 80.01 0)
-    (effects (font (size 1.27 1.27)) (justify left))
-  )
   (hierarchical_label "SCKI" (shape input) (at 170.18 106.68 180)
     (effects (font (size 1.27 1.27)) (justify right))
@@
     (effects (font (size 1.27 1.27)) (justify left))
   )
+  (hierarchical_label "S4" (shape input) (at 119.38 80.01 0)
+    (effects (font (size 1.27 1.27)) (justify left))
+  )
   (hierarchical_label "ACTIVE_TAP5" (shape input) (at 41.91 53.34 180)
     (effects (font (size 1.27 1.27)) (justify right))
@@
     (effects (font (size 1.27 1.27)) (justify right))
   )
-  (hierarchical_label "S4" (shape input) (at 119.38 85.09 0)
-    (effects (font (size 1.27 1.27)) (justify left))
-  )
   (hierarchical_label "C_FILTERED3" (shape input) (at 119.38 115.57 0)
     (effects (font (size 1.27 1.27)) (justify left))
@@
     (effects (font (size 1.27 1.27)) (justify right))
   )
+  (hierarchical_label "C_FILTERED4" (shape input) (at 119.38 85.09 0)
+    (effects (font (size 1.27 1.27)) (justify left))
+  )
   (hierarchical_label "A0" (shape input) (at 176.53 88.9 180)
     (effects (font (size 1.27 1.27)) (justify right))
@@
   (hierarchical_label "ACTIVE_TAP0" (shape input) (at 41.91 185.42 180)
     (effects (font (size 1.27 1.27)) (justify right))
+  )
+  (hierarchical_label "V-" (shape input) (at 231.14 123.19 0)
+    (effects (font (size 1.27 1.27)) (justify left))
   )
   (hierarchical_label "ACTIVE_TAP3" (shape input) (at 41.91 115.57 180)
@@
   (symbol (lib_id "Device:R") (at 260.35 114.3 0)
     (in_bom yes) (on_board yes)
-    (property "Reference" "R129" (id 0) (at 262.128 113.1316 0)
+    (property "Reference" "R29" (id 0) (at 262.128 113.1316 0)
       (effects (font (size 1.27 1.27)) (justify left))
     )
@@
   (symbol (lib_id "Device:D_Schottky") (at 240.03 124.46 270)
     (in_bom yes) (on_board yes)
-    (property "Reference" "D27" (id 0) (at 242.062 123.2916 90)
+    (property "Reference" "D14" (id 0) (at 242.062 123.2916 90)
       (effects (font (size 1.27 1.27)) (justify left))
     )
@@
   (symbol (lib_id "Device:R") (at 240.03 132.08 0)
     (in_bom yes) (on_board yes)
-    (property "Reference" "R127" (id 0) (at 241.808 130.9116 0)
+    (property "Reference" "R27" (id 0) (at 241.808 130.9116 0)
       (effects (font (size 1.27 1.27)) (justify left))
     )
@@
   (symbol (lib_id "Device:C") (at 248.92 115.57 0)
     (in_bom yes) (on_board yes)
-    (property "Reference" "C103" (id 0) (at 251.841 114.4016 0)
+    (property "Reference" "C30" (id 0) (at 251.841 114.4016 0)
       (effects (font (size 1.27 1.27)) (justify left))
     )
@@
   (symbol (lib_id "LTC3300ILXE-2_PBF:LTC3300ILXE-2#PBF") (at 204.47 86.36 0)
     (in_bom yes) (on_board yes)
-    (property "Reference" "U5" (id 0) (at 204.47 46.482 0))
+    (property "Reference" "U4" (id 0) (at 204.47 46.482 0))
     (property "Value" "LTC3300ILXE-2#PBF" (id 1) (at 204.47 48.7934 0))
-    (property "Footprint" "QFP50P900X900X160-49N" (id 2) (at 204.47 86.36 0)
+    (property "Footprint" "LTC3300ILXE-2_PBF:QFP50P900X900X160-49N" (id 2) (at 204.47 86.36 0)
       (effects (font (size 1.27 1.27)) (justify left bottom) hide)
     )
@@
   (symbol (lib_id "Device:R") (at 269.24 114.3 0)
     (in_bom yes) (on_board yes)
-    (property "Reference" "R130" (id 0) (at 271.018 113.1316 0)
+    (property "Reference" "R30" (id 0) (at 271.018 113.1316 0)
       (effects (font (size 1.27 1.27)) (justify left))
     )
@@
   (symbol (lib_id "Device:R") (at 255.27 83.82 0)
     (in_bom yes) (on_board yes)
-    (property "Reference" "R128" (id 0) (at 257.048 82.6516 0)
+    (property "Reference" "R28" (id 0) (at 257.048 82.6516 0)
       (effects (font (size 1.27 1.27)) (justify left))
     )
@@
   (symbol (lib_id "Device:C") (at 243.84 57.15 0)
     (in_bom yes) (on_board yes) (fields_autoplaced)
-    (property "Reference" "C?" (id 0) (at 247.65 55.8799 0)
+    (property "Reference" "C42" (id 0) (at 247.65 55.8799 0)
       (effects (font (size 1.27 1.27)) (justify left))
     )
@@
       (effects (font (size 1.27 1.27)) (justify right))
     )
+    (pin "C_N" input (at 68.58 53.34 180)
+      (effects (font (size 1.27 1.27)) (justify left))
+    )
+    (pin "C_N-1" input (at 68.58 55.88 180)
+      (effects (font (size 1.27 1.27)) (justify left))
+    )
+    (pin "PG_N" input (at 104.14 60.96 0)
+      (effects (font (size 1.27 1.27)) (justify right))
+    )
+    (pin "PI_N" input (at 104.14 63.5 0)
+      (effects (font (size 1.27 1.27)) (justify right))
+    )
+    (pin "SG_N" input (at 104.14 66.04 0)
+      (effects (font (size 1.27 1.27)) (justify right))
+    )
+    (pin "SI_N" input (at 104.14 68.58 0)
+      (effects (font (size 1.27 1.27)) (justify right))
+    )
+    (pin "BOOST" input (at 68.58 48.26 180)
+      (effects (font (size 1.27 1.27)) (justify left))
+    )
+    (pin "V-" input (at 68.58 60.96 180)
+      (effects (font (size 1.27 1.27)) (justify left))
+    )
+    (pin "C_FILTERED_N-1" input (at 104.14 55.88 0)
+      (effects (font (size 1.27 1.27)) (justify right))
+    )
     (pin "SN" input (at 104.14 48.26 0)
       (effects (font (size 1.27 1.27)) (justify right))
     )
-    (pin "C_N" input (at 68.58 53.34 180)
-      (effects (font (size 1.27 1.27)) (justify left))
-    )
-    (pin "C_N-1" input (at 68.58 55.88 180)
-      (effects (font (size 1.27 1.27)) (justify left))
-    )
-    (pin "PG_N" input (at 104.14 60.96 0)
-      (effects (font (size 1.27 1.27)) (justify right))
-    )
-    (pin "PI_N" input (at 104.14 63.5 0)
-      (effects (font (size 1.27 1.27)) (justify right))
-    )
-    (pin "SG_N" input (at 104.14 66.04 0)
-      (effects (font (size 1.27 1.27)) (justify right))
-    )
-    (pin "SI_N" input (at 104.14 68.58 0)
-      (effects (font (size 1.27 1.27)) (justify right))
-    )
-    (pin "BOOST" input (at 68.58 48.26 180)
-      (effects (font (size 1.27 1.27)) (justify left))
-    )
-    (pin "V-" input (at 68.58 60.96 180)
-      (effects (font (size 1.27 1.27)) (justify left))
-    )
-    (pin "C_FILTERED_N-1" input (at 104.14 55.88 0)
-      (effects (font (size 1.27 1.27)) (justify right))
-    )
