File: 211006_lmu_r0/file6196A5FB.kicad_sch (KiCad schematic)
At the start: 8 parts, among them U4 LTC3300ILXE-2#PBF

Commit message: refined in-out routing mechanism
Parts:
- renumbered C30 to C103, C42 to C54, D14 to D27, R27 to R127, R28 to R128, R29 to R129, R30 to R130, U4 to U5
Changed lines of the file:
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@@
   (symbol (lib_id "Device:R") (at 260.35 114.3 0)
     (in_bom yes) (on_board yes)
-    (property "Reference" "R29" (id 0) (at 262.128 113.1316 0)
+    (property "Reference" "R129" (id 0) (at 262.128 113.1316 0)
       (effects (font (size 1.27 1.27)) (justify left))
     )
@@
   (symbol (lib_id "Device:D_Schottky") (at 240.03 124.46 270)
     (in_bom yes) (on_board yes)
-    (property "Reference" "D14" (id 0) (at 242.062 123.2916 90)
+    (property "Reference" "D27" (id 0) (at 242.062 123.2916 90)
       (effects (font (size 1.27 1.27)) (justify left))
     )
@@
   (symbol (lib_id "Device:R") (at 240.03 132.08 0)
     (in_bom yes) (on_board yes)
-    (property "Reference" "R27" (id 0) (at 241.808 130.9116 0)
+    (property "Reference" "R127" (id 0) (at 241.808 130.9116 0)
       (effects (font (size 1.27 1.27)) (justify left))
     )
@@
   (symbol (lib_id "Device:C") (at 248.92 115.57 0)
     (in_bom yes) (on_board yes)
-    (property "Reference" "C30" (id 0) (at 251.841 114.4016 0)
+    (property "Reference" "C103" (id 0) (at 251.841 114.4016 0)
       (effects (font (size 1.27 1.27)) (justify left))
     )
@@
   (symbol (lib_id "LTC3300ILXE-2_PBF:LTC3300ILXE-2#PBF") (at 204.47 86.36 0)
     (in_bom yes) (on_board yes)
-    (property "Reference" "U4" (id 0) (at 204.47 46.482 0))
+    (property "Reference" "U5" (id 0) (at 204.47 46.482 0))
     (property "Value" "LTC3300ILXE-2#PBF" (id 1) (at 204.47 48.7934 0))
     (property "Footprint" "LTC3300ILXE-2_PBF:QFP50P900X900X160-49N" (id 2) (at 204.47 86.36 0)
@@
   (symbol (lib_id "Device:R") (at 269.24 114.3 0)
     (in_bom yes) (on_board yes)
-    (property "Reference" "R30" (id 0) (at 271.018 113.1316 0)
+    (property "Reference" "R130" (id 0) (at 271.018 113.1316 0)
       (effects (font (size 1.27 1.27)) (justify left))
     )
@@
   (symbol (lib_id "Device:R") (at 255.27 83.82 0)
     (in_bom yes) (on_board yes)
-    (property "Reference" "R28" (id 0) (at 257.048 82.6516 0)
+    (property "Reference" "R128" (id 0) (at 257.048 82.6516 0)
       (effects (font (size 1.27 1.27)) (justify left))
     )
@@
   (symbol (lib_id "Device:C") (at 243.84 57.15 0)
     (in_bom yes) (on_board yes) (fields_autoplaced)
-    (property "Reference" "C42" (id 0) (at 247.65 55.8799 0)
-      (effects (font (size 1.27 1.27)) (justify left))
-    )
+    (property "Reference" "C54" (id 0) (at 247.65 55.8799 0)
+      (effects (font (size 1.27 1.27)) (justify left))
+    )

Commit message: trying out a quick thing, recover
Parts:
- renumbered C103 to C30, C54 to C42, D27 to D14, R127 to R27, R128 to R28, R129 to R29, R130 to R30, U5 to U4
Changed lines of the file:
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@@
   (symbol (lib_id "Device:R") (at 260.35 114.3 0)
     (in_bom yes) (on_board yes)
-    (property "Reference" "R129" (id 0) (at 262.128 113.1316 0)
+    (property "Reference" "R29" (id 0) (at 262.128 113.1316 0)
       (effects (font (size 1.27 1.27)) (justify left))
     )
@@
   (symbol (lib_id "Device:D_Schottky") (at 240.03 124.46 270)
     (in_bom yes) (on_board yes)
-    (property "Reference" "D27" (id 0) (at 242.062 123.2916 90)
+    (property "Reference" "D14" (id 0) (at 242.062 123.2916 90)
       (effects (font (size 1.27 1.27)) (justify left))
     )
@@
   (symbol (lib_id "Device:R") (at 240.03 132.08 0)
     (in_bom yes) (on_board yes)
-    (property "Reference" "R127" (id 0) (at 241.808 130.9116 0)
+    (property "Reference" "R27" (id 0) (at 241.808 130.9116 0)
       (effects (font (size 1.27 1.27)) (justify left))
     )
@@
   (symbol (lib_id "Device:C") (at 248.92 115.57 0)
     (in_bom yes) (on_board yes)
-    (property "Reference" "C103" (id 0) (at 251.841 114.4016 0)
+    (property "Reference" "C30" (id 0) (at 251.841 114.4016 0)
       (effects (font (size 1.27 1.27)) (justify left))
     )
@@
   (symbol (lib_id "LTC3300ILXE-2_PBF:LTC3300ILXE-2#PBF") (at 204.47 86.36 0)
     (in_bom yes) (on_board yes)
-    (property "Reference" "U5" (id 0) (at 204.47 46.482 0))
+    (property "Reference" "U4" (id 0) (at 204.47 46.482 0))
     (property "Value" "LTC3300ILXE-2#PBF" (id 1) (at 204.47 48.7934 0))
     (property "Footprint" "LTC3300ILXE-2_PBF:QFP50P900X900X160-49N" (id 2) (at 204.47 86.36 0)
@@
   (symbol (lib_id "Device:R") (at 269.24 114.3 0)
     (in_bom yes) (on_board yes)
-    (property "Reference" "R130" (id 0) (at 271.018 113.1316 0)
+    (property "Reference" "R30" (id 0) (at 271.018 113.1316 0)
       (effects (font (size 1.27 1.27)) (justify left))
     )
@@
   (symbol (lib_id "Device:R") (at 255.27 83.82 0)
     (in_bom yes) (on_board yes)
-    (property "Reference" "R128" (id 0) (at 257.048 82.6516 0)
+    (property "Reference" "R28" (id 0) (at 257.048 82.6516 0)
       (effects (font (size 1.27 1.27)) (justify left))
     )
@@
   (symbol (lib_id "Device:C") (at 243.84 57.15 0)
     (in_bom yes) (on_board yes) (fields_autoplaced)
-    (property "Reference" "C54" (id 0) (at 247.65 55.8799 0)
-      (effects (font (size 1.27 1.27)) (justify left))
-    )
+    (property "Reference" "C42" (id 0) (at 247.65 55.8799 0)
+      (effects (font (size 1.27 1.27)) (justify left))
+    )

Commit message: copying layout
Connections:
- net C_FILTERED5: now also U4.36 (C5)
- net C_FILTERED6: now also R27.2, U4.39 (C6)
- net S5: no longer U4.36 (C5)
- net S6: no longer R27.2, U4.39 (C6)
Changed lines of the file:
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@@
-    (effects (font (size 1.27 1.27)) (justify left bottom))
-  )
-  (label "C6" (at 113.03 17.78 0)
     (effects (font (size 1.27 1.27)) (justify left bottom))
   )
@@
     (effects (font (size 1.27 1.27)) (justify left bottom))
   )
+  (label "C5" (at 113.03 53.34 0)
+    (effects (font (size 1.27 1.27)) (justify left bottom))
+  )
   (label "PI2" (at 176.53 63.5 0)
     (effects (font (size 1.27 1.27)) (justify left bottom))
@@
   )
   (label "SG3" (at 232.41 71.12 0)
-    (effects (font (size 1.27 1.27)) (justify left bottom))
-  )
-  (label "C5" (at 113.03 48.26 0)
     (effects (font (size 1.27 1.27)) (justify left bottom))
   )
@@
     (effects (font (size 1.27 1.27)) (justify left bottom))
   )
+  (label "C6" (at 113.03 22.86 0)
+    (effects (font (size 1.27 1.27)) (justify left bottom))
+  )
