File: 211006_lmu_r0/file61619F33.kicad_sch (KiCad schematic)
At the start: 47 parts, among them J5 Conn_01x03, J6 Conn_01x03, J7 Conn_01x02, Q1 CZT5551, U3 LTC6811HG-2#PBF

Commit message: sorted header location
Parts:
- R252: footprint Resistor_SMD:R_0603_1608Metric_Pad0.98x0.95mm_HandSolder -> Resistor_SMD:R_1206_3216Metric_Pad1.30x1.75mm_HandSolder
Connections:
- net VREG: no longer R252.2
- new net VREG_PASSIVE: R252.2
Changed lines of the file:
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@@
     (effects (font (size 1.27 1.27)) (justify right))
   )
-  (hierarchical_label "VREG" (shape input) (at 39.37 154.94 180)
+  (hierarchical_label "VREG_PASSIVE" (shape input) (at 39.37 154.94 180)
     (effects (font (size 1.27 1.27)) (justify right))
   )
@@
     (property "Reference" "R252" (id 0) (at 48.26 149.6822 90))
     (property "Value" "0R DNP" (id 1) (at 48.26 151.9936 90))
-    (property "Footprint" "Resistor_SMD:R_0603_1608Metric_Pad0.98x0.95mm_HandSolder" (id 2) (at 48.26 153.162 90)
-      (effects (font (size 1.27 1.27)) hide)
-    )
+    (property "Footprint" "Resistor_SMD:R_1206_3216Metric_Pad1.30x1.75mm_HandSolder" (id 2) (at 48.26 153.162 90)
+      (effects (font (size 1.27 1.27)) hide)
+    )

Commit message: trying out a quick thing, recover
Changed lines of the file:
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@@
     (stroke (width 0) (type default) (color 0 0 0 0))
   )
-  (wire (pts (xy 226.06 81.28) (xy 229.87 81.28))
+  (wire (pts (xy 226.06 81.28) (xy 228.6 81.28))
     (stroke (width 0) (type default) (color 0 0 0 0))
   )
@@
     (pin "2")
   )
-  (symbol (lib_name "GND_HV_11") (lib_id "gnd_hv:GND_HV") (at 54.61 120.65 0) (unit 1)
-    (in_bom yes) (on_board yes)
-    (property "Reference" "#PWR040" (id 0) (at 54.61 127 0)
-      (effects (font (size 1.27 1.27)) hide)
-    )
-    (property "Value" "GND_HV" (id 1) (at 54.737 125.0442 0))
-    (property "Footprint" "" (id 2) (at 54.61 120.65 0)
-      (effects (font (size 1.27 1.27)) hide)
-    )
-    (property "Datasheet" "" (id 3) (at 54.61 120.65 0)
-      (effects (font (size 1.27 1.27)) hide)
-    )
-    (pin "1")
-  )
   (symbol (lib_id "czt5551:CZT5551") (at 257.81 142.24 0) (unit 1)
     (in_bom yes) (on_board yes)
@@
     (pin "1")
   )
-  (symbol (lib_name "GND_HV_5") (lib_id "gnd_hv:GND_HV") (at 229.87 81.28 0) (unit 1)
-    (in_bom yes) (on_board yes)
-    (property "Reference" "#PWR047" (id 0) (at 229.87 87.63 0)
-      (effects (font (size 1.27 1.27)) hide)
-    )
-    (property "Value" "GND_HV" (id 1) (at 233.68 81.28 0))
-    (property "Footprint" "" (id 2) (at 229.87 81.28 0)
-      (effects (font (size 1.27 1.27)) hide)
-    )
-    (property "Datasheet" "" (id 3) (at 229.87 81.28 0)
-      (effects (font (size 1.27 1.27)) hide)
-    )
+  (symbol (lib_name "GND_HV_5") (lib_id "gnd_hv:GND_HV") (at 228.6 81.28 0) (unit 1)
+    (in_bom yes) (on_board yes)
+    (property "Reference" "#PWR047" (id 0) (at 228.6 87.63 0)
+      (effects (font (size 1.27 1.27)) hide)
+    )
+    (property "Value" "GND_HV" (id 1) (at 232.41 81.28 0))
+    (property "Footprint" "" (id 2) (at 228.6 81.28 0)
+      (effects (font (size 1.27 1.27)) hide)
+    )
+    (property "Datasheet" "" (id 3) (at 228.6 81.28 0)
+      (effects (font (size 1.27 1.27)) hide)
+    )

Commit message: silkscreen changes, shifting bun leds
Parts:
- TP10, TP11, TP12, TP13, TP14, TP15, TP16, TP17, TP18, TP19, TP20, TP21, TP22, TP23, TP24, TP25, TP8, TP9: footprint TestPoint:TestPoint_Pad_D1.0mm -> custom:TestPoint_Pad_D1.0mm
Changed lines of the file:
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@@
     (property "Reference" "TP21" (id 0) (at 226.7712 20.447 90))
     (property "Value" "TestPoint" (id 1) (at 226.7712 22.7584 90))
-    (property "Footprint" "TestPoint:TestPoint_Pad_D1.0mm" (id 2) (at 228.6 20.32 0)
+    (property "Footprint" "custom:TestPoint_Pad_D1.0mm" (id 2) (at 228.6 20.32 0)
       (effects (font (size 1.27 1.27)) hide)
     )
@@
     (property "Reference" "TP22" (id 0) (at 226.7712 28.067 90))
     (property "Value" "TestPoint" (id 1) (at 226.7712 30.3784 90))
-    (property "Footprint" "TestPoint:TestPoint_Pad_D1.0mm" (id 2) (at 228.6 27.94 0)
+    (property "Footprint" "custom:TestPoint_Pad_D1.0mm" (id 2) (at 228.6 27.94 0)
       (effects (font (size 1.27 1.27)) hide)
     )
@@
       (effects (font (size 1.27 1.27)) (justify left))
     )
-    (property "Footprint" "TestPoint:TestPoint_Pad_D1.0mm" (id 2) (at 247.65 142.24 0)
+    (property "Footprint" "custom:TestPoint_Pad_D1.0mm" (id 2) (at 247.65 142.24 0)
       (effects (font (size 1.27 1.27)) hide)
     )
@@
       (effects (font (size 1.27 1.27)) (justify right))
     )
-    (property "Footprint" "TestPoint:TestPoint_Pad_D1.0mm" (id 2) (at 255.27 153.67 0)
+    (property "Footprint" "custom:TestPoint_Pad_D1.0mm" (id 2) (at 255.27 153.67 0)
       (effects (font (size 1.27 1.27)) hide)
     )
@@
       (effects (font (size 1.27 1.27)) (justify left))
     )
-    (property "Footprint" "TestPoint:TestPoint_Pad_D1.0mm" (id 2) (at 245.11 76.2 0)
+    (property "Footprint" "custom:TestPoint_Pad_D1.0mm" (id 2) (at 245.11 76.2 0)
       (effects (font (size 1.27 1.27)) hide)
     )
@@
       (effects (font (size 1.27 1.27)) (justify left) hide)
     )
-    (property "Footprint" "TestPoint:TestPoint_Pad_D1.0mm" (id 2) (at 38.1 24.13 0)
+    (property "Footprint" "custom:TestPoint_Pad_D1.0mm" (id 2) (at 38.1 24.13 0)
       (effects (font (size 1.27 1.27)) hide)
     )
@@
       (effects (font (size 1.27 1.27)) (justify left) hide)
     )
-    (property "Footprint" "TestPoint:TestPoint_Pad_D1.0mm" (id 2) (at 38.1 29.21 0)
+    (property "Footprint" "custom:TestPoint_Pad_D1.0mm" (id 2) (at 38.1 29.21 0)
       (effects (font (size 1.27 1.27)) hide)
     )
@@
       (effects (font (size 1.27 1.27)) (justify left) hide)
     )
-    (property "Footprint" "TestPoint:TestPoint_Pad_D1.0mm" (id 2) (at 38.1 34.29 0)
+    (property "Footprint" "custom:TestPoint_Pad_D1.0mm" (id 2) (at 38.1 34.29 0)
       (effects (font (size 1.27 1.27)) hide)
     )
@@
       (effects (font (size 1.27 1.27)) (justify left) hide)
     )
-    (property "Footprint" "TestPoint:TestPoint_Pad_D1.0mm" (id 2) (at 38.1 39.37 0)
+    (property "Footprint" "custom:TestPoint_Pad_D1.0mm" (id 2) (at 38.1 39.37 0)
       (effects (font (size 1.27 1.27)) hide)
     )
@@
       (effects (font (size 1.27 1.27)) (justify left) hide)
     )
-    (property "Footprint" "TestPoint:TestPoint_Pad_D1.0mm" (id 2) (at 38.1 44.45 0)
+    (property "Footprint" "custom:TestPoint_Pad_D1.0mm" (id 2) (at 38.1 44.45 0)
       (effects (font (size 1.27 1.27)) hide)
     )
@@
       (effects (font (size 1.27 1.27)) (justify left) hide)
     )
-    (property "Footprint" "TestPoint:TestPoint_Pad_D1.0mm" (id 2) (at 38.1 49.53 0)
+    (property "Footprint" "custom:TestPoint_Pad_D1.0mm" (id 2) (at 38.1 49.53 0)
       (effects (font (size 1.27 1.27)) hide)
     )
@@
       (effects (font (size 1.27 1.27)) (justify left) hide)
     )
-    (property "Footprint" "TestPoint:TestPoint_Pad_D1.0mm" (id 2) (at 38.1 90.17 0)
+    (property "Footprint" "custom:TestPoint_Pad_D1.0mm" (id 2) (at 38.1 90.17 0)
       (effects (font (size 1.27 1.27)) hide)
     )
@@
       (effects (font (size 1.27 1.27)) (justify left) hide)
     )
-    (property "Footprint" "TestPoint:TestPoint_Pad_D1.0mm" (id 2) (at 38.1 95.25 0)
+    (property "Footprint" "custom:TestPoint_Pad_D1.0mm" (id 2) (at 38.1 95.25 0)
       (effects (font (size 1.27 1.27)) hide)
     )
@@
       (effects (font (size 1.27 1.27)) (justify left) hide)
     )
-    (property "Footprint" "TestPoint:TestPoint_Pad_D1.0mm" (id 2) (at 38.1 100.33 0)
+    (property "Footprint" "custom:TestPoint_Pad_D1.0mm" (id 2) (at 38.1 100.33 0)
       (effects (font (size 1.27 1.27)) hide)
     )
@@
       (effects (font (size 1.27 1.27)) (justify left) hide)
     )
-    (property "Footprint" "TestPoint:TestPoint_Pad_D1.0mm" (id 2) (at 38.1 105.41 0)
+    (property "Footprint" "custom:TestPoint_Pad_D1.0mm" (id 2) (at 38.1 105.41 0)
       (effects (font (size 1.27 1.27)) hide)
     )
@@
       (effects (font (size 1.27 1.27)) (justify left) hide)
     )
-    (property "Footprint" "TestPoint:TestPoint_Pad_D1.0mm" (id 2) (at 38.1 110.49 0)
+    (property "Footprint" "custom:TestPoint_Pad_D1.0mm" (id 2) (at 38.1 110.49 0)
       (effects (font (size 1.27 1.27)) hide)
     )
@@
       (effects (font (size 1.27 1.27)) (justify left) hide)
     )
-    (property "Footprint" "TestPoint:TestPoint_Pad_D1.0mm" (id 2) (at 38.1 115.57 0)
+    (property "Footprint" "custom:TestPoint_Pad_D1.0mm" (id 2) (at 38.1 115.57 0)
       (effects (font (size 1.27 1.27)) hide)
     )
@@
       (effects (font (size 1.27 1.27)) (justify left) hide)
     )
-    (property "Footprint" "TestPoint:TestPoint_Pad_D1.0mm" (id 2) (at 38.1 120.65 0)
-      (effects (font (size 1.27 1.27)) hide)
-    )
+    (property "Footprint" "custom:TestPoint_Pad_D1.0mm" (id 2) (at 38.1 120.65 0)
+      (effects (font (size 1.27 1.27)) hide)
+    )

Commit message: started to export and fix things
Parts:
- U3: MANUFACTURER Linear Technology -> (none)
Changed lines of the file:
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@@
-      (effects (font (size 1.27 1.27)) (justify left bottom) hide)
-    )
-    (property "MANUFACTURER" "Linear Technology" (id 4) (at 200.66 119.38 0)
       (effects (font (size 1.27 1.27)) (justify left bottom) hide)
     )
