File: 211006_lmu_r0/active_passive_balance.kicad_sch (KiCad schematic)
At the start: 41 parts, among them Q35 BSS308PE, Q36 SiR882DP, Q37 SiR882DP, T12 750312504

Commit message: Updated lmu project with relative library paths and fixed broken symbols
Parts:
- D38: MANUFACTURER (none) -> Diodes Inc
Connections:
- net BOOST: now also T12.5
- net C_N: now also D38.1, Q35.2 (S), T12.1, T12.2
- net C_N-1: now also D38.2, D38.3
- net at R191.2, R192.2, TP148.1: now also Q35.3 (D)
- net at R201.2: now also Q37.4 (G)
- net at C169.1, TP153.1: now also Q37.5 (D), T12.7
- net at R195.1, R197.1, TP151.1: now also Q36.1 (S), Q36.2 (S), Q36.3 (S)
- net at R199.1, R200.2, TP154.1: now also Q37.1 (S), Q37.2 (S), Q37.3 (S)
- net at C168.1, TP152.1: now also Q36.5 (D), T12.10, T12.9
- net at R193.1: now also Q35.1 (G)
- net at R194.1: now also Q36.4 (G)
- new net: T12.4, T12.6
Changed lines of the file:
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@@
       (effects (font (size 1.27 1.27)) hide)
     )
+    (pin "1")
+    (pin "2")
+    (pin "3")
   )
   (symbol (lib_id "Device:R") (at 228.6 71.12 270)
@@
       (effects (font (size 1.27 1.27)) (justify left bottom) hide)
     )
-    (property "MANUFACTURER" "" (id 4) (at 22.86 99.06 0)
+    (property "MANUFACTURER" "Diodes Inc" (id 4) (at 22.86 99.06 0)
       (effects (font (size 1.27 1.27)) (justify left bottom) hide)
     )
@@
       (effects (font (size 1.27 1.27)) hide)
     )
+    (pin "1")
+    (pin "2")
+    (pin "3")
   )
   (symbol (lib_id "Device:C") (at 74.93 82.55 180)
@@
       (effects (font (size 1.27 1.27)) hide)
     )
+    (pin "1")
+    (pin "10")
+    (pin "2")
+    (pin "4")
+    (pin "5")
+    (pin "6")
+    (pin "7")
+    (pin "9")
   )
   (symbol (lib_id "Device:C") (at 252.73 78.74 180)
@@
       (effects (font (size 1.27 1.27)) hide)
     )
+    (pin "1")
+    (pin "2")
+    (pin "3")
+    (pin "4")
+    (pin "5")
   )
   (symbol (lib_id "Device:R") (at 111.76 115.57 0)
@@
       (effects (font (size 1.27 1.27)) hide)
     )
+    (pin "1")
+    (pin "2")
+    (pin "3")
+    (pin "4")
+    (pin "5")
   )
   (symbol (lib_id "Device:R") (at 162.56 109.22 270) (mirror x)

Commit message: Updated some components to make sourcing easier
Parts:
- C164, C165, C167, C170, C172, C173: Manufacturer (none) -> Walsin; Part Number (none) -> 1210F107Z6R3CT
- C166, C168, C169, C171, C174, C175, R191, R192, R193, R194, R195, R196, R198, R200, R201, R202: Manufacturer (none) -> -; Part Number (none) -> -
- R197, R199: Manufacturer (none) -> -
Changed lines of the file:
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@@
+      (effects (font (size 1.27 1.27)) hide)
+    )
+    (property "Part Number" "-" (id 4) (at 228.6 71.12 0)
+      (effects (font (size 1.27 1.27)) hide)
+    )
+    (property "Manufacturer" "-" (id 5) (at 228.6 71.12 0)
       (effects (font (size 1.27 1.27)) hide)
     )
@@
       (effects (font (size 1.27 1.27)) hide)
     )
+    (property "Part Number" "-" (id 4) (at 241.3 78.74 0)
+      (effects (font (size 1.27 1.27)) hide)
+    )
+    (property "Manufacturer" "-" (id 5) (at 241.3 78.74 0)
+      (effects (font (size 1.27 1.27)) hide)
+    )
     (pin "1")
     (pin "2")
@@
     )
     (property "Datasheet" "~" (id 3) (at 43.18 99.06 0)
+      (effects (font (size 1.27 1.27)) hide)
+    )
+    (property "Part Number" "-" (id 4) (at 43.18 99.06 0)
+      (effects (font (size 1.27 1.27)) hide)
+    )
+    (property "Manufacturer" "-" (id 5) (at 43.18 99.06 0)
       (effects (font (size 1.27 1.27)) hide)
     )
@@
       (effects (font (size 1.27 1.27)) hide)
     )
+    (property "Part Number" "-" (id 4) (at 170.18 115.57 0)
+      (effects (font (size 1.27 1.27)) hide)
+    )
+    (property "Manufacturer" "-" (id 5) (at 170.18 115.57 0)
+      (effects (font (size 1.27 1.27)) hide)
+    )
     (pin "1")
     (pin "2")
@@
     )
     (property "Voltage" "100V" (id 4) (at 77.47 87.63 0))
+    (property "Manufacturer" "Walsin" (id 5) (at 74.93 82.55 0)
+      (effects (font (size 1.27 1.27)) hide)
+    )
+    (property "Part Number" "1210F107Z6R3CT" (id 6) (at 74.93 82.55 0)
+      (effects (font (size 1.27 1.27)) hide)
+    )
     (pin "1")
     (pin "2")
@@
       (effects (font (size 1.27 1.27)) hide)
     )
+    (property "Part Number" "-" (id 4) (at 165.1 101.6 0)
+      (effects (font (size 1.27 1.27)) hide)
+    )
+    (property "Manufacturer" "-" (id 5) (at 165.1 101.6 0)
+      (effects (font (size 1.27 1.27)) hide)
+    )
     (pin "1")
     (pin "2")
@@
       (effects (font (size 1.27 1.27)) hide)
     )
+    (property "Part Number" "-" (id 5) (at 153.67 92.71 0)
+      (effects (font (size 1.27 1.27)) hide)
+    )
+    (property "Manufacturer" "-" (id 6) (at 153.67 92.71 0)
+      (effects (font (size 1.27 1.27)) hide)
+    )
     (pin "1")
     (pin "2")
@@
       (effects (font (size 1.27 1.27)) hide)
     )
+    (property "Part Number" "-" (id 4) (at 102.87 109.22 0)
+      (effects (font (size 1.27 1.27)) hide)
+    )
+    (property "Manufacturer" "-" (id 5) (at 102.87 109.22 0)
+      (effects (font (size 1.27 1.27)) hide)
+    )
     (pin "1")
     (pin "2")
@@
       (effects (font (size 1.27 1.27)) hide)
     )
+    (property "Manufacturer" "-" (id 4) (at 153.67 115.57 0)
+      (effects (font (size 1.27 1.27)) hide)
+    )
     (pin "1")
     (pin "2")
@@
       (effects (font (size 1.27 1.27)) hide)
     )
+    (property "Manufacturer" "Walsin" (id 4) (at 86.36 82.55 0)
+      (effects (font (size 1.27 1.27)) hide)
+    )
+    (property "Part Number" "1210F107Z6R3CT" (id 5) (at 86.36 82.55 0)
+      (effects (font (size 1.27 1.27)) hide)
+    )
     (pin "1")
     (pin "2")
@@
       (effects (font (size 1.27 1.27)) hide)
     )
+    (property "Manufacturer" "Walsin" (id 4) (at 97.79 82.55 0)
+      (effects (font (size 1.27 1.27)) hide)
+    )
+    (property "Part Number" "1210F107Z6R3CT" (id 5) (at 97.79 82.55 0)
+      (effects (font (size 1.27 1.27)) hide)
+    )
     (pin "1")
     (pin "2")
@@
     )
     (property "Voltage" "100V" (id 4) (at 166.37 90.17 0))
+    (property "Manufacturer" "Walsin" (id 5) (at 163.83 85.09 0)
+      (effects (font (size 1.27 1.27)) hide)
+    )
+    (property "Part Number" "1210F107Z6R3CT" (id 6) (at 163.83 85.09 0)
+      (effects (font (size 1.27 1.27)) hide)
+    )
     (pin "1")
     (pin "2")
@@
       (effects (font (size 1.27 1.27)) hide)
     )
+    (property "Manufacturer" "Walsin" (id 4) (at 175.26 85.09 0)
+      (effects (font (size 1.27 1.27)) hide)
+    )
+    (property "Part Number" "1210F107Z6R3CT" (id 5) (at 175.26 85.09 0)
+      (effects (font (size 1.27 1.27)) hide)
+    )
     (pin "1")
     (pin "2")
@@
     )
     (property "Datasheet" "~" (id 3) (at 186.69 85.09 0)
+      (effects (font (size 1.27 1.27)) hide)
+    )
+    (property "Manufacturer" "Walsin" (id 4) (at 186.69 85.09 0)
+      (effects (font (size 1.27 1.27)) hide)
+    )
+    (property "Part Number" "1210F107Z6R3CT" (id 5) (at 186.69 85.09 0)
       (effects (font (size 1.27 1.27)) hide)
     )
@@
       (effects (font (size 1.27 1.27)) hide)
     )
+    (property "Part Number" "-" (id 4) (at 60.96 86.36 0)
+      (effects (font (size 1.27 1.27)) hide)
+    )
+    (property "Manufacturer" "-" (id 5) (at 60.96 86.36 0)
+      (effects (font (size 1.27 1.27)) hide)
+    )
     (pin "1")
     (pin "2")
@@
     )
     (property "Datasheet" "~" (id 3) (at 53.34 95.25 0)
+      (effects (font (size 1.27 1.27)) hide)
+    )
+    (property "Part Number" "-" (id 4) (at 53.34 95.25 0)
+      (effects (font (size 1.27 1.27)) hide)
+    )
+    (property "Manufacturer" "-" (id 5) (at 53.34 95.25 0)
       (effects (font (size 1.27 1.27)) hide)
     )
@@
     )
     (property "Voltage" "100V" (id 4) (at 257.81 82.55 0))
+    (property "Manufacturer" "-" (id 5) (at 252.73 78.74 0)
+      (effects (font (size 1.27 1.27)) hide)
+    )
+    (property "Part Number" "-" (id 6) (at 252.73 78.74 0)
+      (effects (font (size 1.27 1.27)) hide)
+    )
     (pin "1")
     (pin "2")
@@
       (effects (font (size 1.27 1.27)) hide)
     )
+    (property "Part Number" "-" (id 4) (at 111.76 83.82 0)
+      (effects (font (size 1.27 1.27)) hide)
+    )
+    (property "Manufacturer" "-" (id 5) (at 111.76 83.82 0)
+      (effects (font (size 1.27 1.27)) hide)
+    )
     (pin "1")
     (pin "2")
@@
       (effects (font (size 1.27 1.27)) hide)
     )
+    (property "Part Number" "-" (id 5) (at 111.76 91.44 0)
+      (effects (font (size 1.27 1.27)) hide)
+    )
+    (property "Manufacturer" "-" (id 6) (at 111.76 91.44 0)
+      (effects (font (size 1.27 1.27)) hide)
+    )
     (pin "1")
     (pin "2")
@@
     )
     (property "Datasheet" "~" (id 3) (at 153.67 85.09 0)
+      (effects (font (size 1.27 1.27)) hide)
+    )
+    (property "Part Number" "-" (id 4) (at 153.67 85.09 0)
+      (effects (font (size 1.27 1.27)) hide)
+    )
+    (property "Manufacturer" "-" (id 5) (at 153.67 85.09 0)
       (effects (font (size 1.27 1.27)) hide)
     )
@@
       (effects (font (size 1.27 1.27)) hide)
     )
+    (property "Manufacturer" "-" (id 4) (at 111.76 115.57 0)
+      (effects (font (size 1.27 1.27)) hide)
+    )
     (pin "1")
     (pin "2")
@@
       (effects (font (size 1.27 1.27)) hide)
     )
+    (property "Part Number" "-" (id 4) (at 95.25 115.57 0)
+      (effects (font (size 1.27 1.27)) hide)
+    )
+    (property "Manufacturer" "-" (id 5) (at 95.25 115.57 0)
+      (effects (font (size 1.27 1.27)) hide)
+    )
     (pin "1")
     (pin "2")
@@
     )
     (property "Datasheet" "~" (id 3) (at 100.33 101.6 0)
+      (effects (font (size 1.27 1.27)) hide)
+    )
+    (property "Part Number" "-" (id 4) (at 100.33 101.6 0)
+      (effects (font (size 1.27 1.27)) hide)
+    )
+    (property "Manufacturer" "-" (id 5) (at 100.33 101.6 0)
       (effects (font (size 1.27 1.27)) hide)
     )
@@
       (effects (font (size 1.27 1.27)) hide)
     )
+    (property "Part Number" "-" (id 4) (at 162.56 109.22 0)
+      (effects (font (size 1.27 1.27)) hide)
+    )
+    (property "Manufacturer" "-" (id 5) (at 162.56 109.22 0)
+      (effects (font (size 1.27 1.27)) hide)
+    )

Commit message: fixed footprints for headers, started planning out zones
Connections:
- net GND renamed GND_HV
Changed lines of the file:
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@@
     (pin "2")
-  )
-  (symbol (lib_id "power:GND") (at 252.73 82.55 0)
-    (in_bom yes) (on_board yes)
-    (property "Reference" "#PWR065" (id 0) (at 252.73 88.9 0)
-      (effects (font (size 1.27 1.27)) hide)
-    )
-    (property "Value" "GND" (id 1) (at 252.857 86.9442 0))
-    (property "Footprint" "" (id 2) (at 252.73 82.55 0)
-      (effects (font (size 1.27 1.27)) hide)
-    )
-    (property "Datasheet" "" (id 3) (at 252.73 82.55 0)
-      (effects (font (size 1.27 1.27)) hide)
-    )
-    (pin "1")
   )
   (symbol (lib_id "Device:C") (at 170.18 115.57 0) (mirror x)
@@
     (pin "2")
   )
+  (symbol (lib_id "gnd_hv:GND_HV") (at 252.73 82.55 0)
+    (in_bom yes) (on_board yes) (fields_autoplaced)
+    (property "Reference" "#PWR0118" (id 0) (at 252.73 88.9 0)
+      (effects (font (size 1.27 1.27)) hide)
+    )
+    (property "Value" "GND_HV" (id 1) (at 252.73 87.63 0))
+    (property "Footprint" "" (id 2) (at 252.73 82.55 0)
+      (effects (font (size 1.27 1.27)) hide)
+    )
+    (property "Datasheet" "" (id 3) (at 252.73 82.55 0)
+      (effects (font (size 1.27 1.27)) hide)
+    )
+    (pin "1")
+  )
 )

Commit message: final merge before branch
Parts:
- D15: renamed from D38; value SBR10U200P5-13 -> SDT15H100P5-7; Mouser Part Number NOT AVAILABLE! -> 621-SDT15H100P5-7; Mouser URL NOT AVAILABLE! -> https://au.mouser.com/ProductDetail/Diodes-Incorporated/SDT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
- renumbered C164 to C31, C165 to C32, C166 to C33, C167 to C34, C168 to C35, C169 to C36, C170 to C37, C171 to C38, C172 to C39, C173 to C40, C174 to C41, C175 to C42, D39 to D16, Q35 to Q2, Q36 to Q3, Q37 to Q4, R191 to R31, R192 to R32, R193 to R33, R194 to R34, R195 to R35, R196 to R36, R197 to R37, R198 to R38, R199 to R39, R200 to R40, R201 to R41, R202 to R42, T12 to T1, TP147 to TP26, TP148 to TP27, TP149 to TP28, TP150 to TP29, TP151 to TP30, TP152 to TP31, TP153 to TP32, TP154 to TP33, TP155 to TP34, TP156 to TP35, TP157 to TP36
Other:
- note added: "can maybe substitute for BUK9K13-60EX"
- note added: "or AOD66920"
- note added: "order inductor from digikey"

Commit message: updated pcb still need to find j11
Parts:
- removed C42: DNP 10nF, Capacitor_SMD:C_0805_2012Metric_Pad1.18x1.45mm_HandSolder, symbol Device:C
- removed Q3, Q4: SiR882DP, Package_SO:PowerPAK_SO-8_Single, symbol sir882dp:SiR882DP
- removed TP30, TP33: TestPoint, TestPoint:TestPoint_Pad_D1.0mm, symbol Connector:TestPoint
- added T24 (x2): BUK9K13-60EX, BUK9K17-60E:SOT1205, symbol BUK9K17-60E:BUK9K17-60E
- renumbered C31 to C164, C32 to C165, C33 to C166, C34 to C167, C35 to C168, C36 to C169, C37 to C170, C38 to C171, C39 to C172, C40 to C173, C41 to C174, D15 to D38, D16 to D39, Q2 to Q35, R31 to R191, R32 to R192, R33 to R193, R34 to R194, R35 to R195, R36 to R196, R37 to R197, R38 to R198, R39 to R199, R40 to R200, R41 to R201, R42 to R202, T1 to T12, TP26 to TP147, TP27 to TP148, TP28 to TP149, TP29 to TP150, TP31 to TP152, TP32 to TP153, TP34 to TP155, TP35 to TP156, TP36 to TP157
Connections:
- net at R201.2: now also T24.2
- net at C169.1, T12.7, TP153.1: now also T24.7, T24.8, T24.S1
- net at R195.1, R197.1: now also T24.1
- net at R199.1, R200.2: now also T24.1
- net at C168.1, T12.10, T12.9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: now also T24.7, T24.8, T24.S1
- net at R194.1: now also T24.2
Other:
- note added: "^ forms RC network for filtering"
- note added: "r_sense = 50mV/i_peak"
- note added: "snubber"
- moved on the sheet: R194, R201, TP149, TP155

Commit message: fixed issues on higher cells, study into how to route
Parts:
- D38: footprint DIO_SBR10U200P5-13 -> SBR10U200P5-13:DIO_SBR10U200P5-13
- T12: footprint EP13_SMT_H_8PIN_(750312504) -> 750312504:EP13_SMT_H_8PIN_(750312504)
Changed lines of the file:
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@@
       (effects (font (size 1.27 1.27)) (justify right))
     )
-    (property "Footprint" "DIO_SBR10U200P5-13" (id 2) (at 22.86 99.06 0)
+    (property "Footprint" "SBR10U200P5-13:DIO_SBR10U200P5-13" (id 2) (at 22.86 99.06 0)
       (effects (font (size 1.27 1.27)) (justify left bottom) hide)
     )
@@
     (property "Reference" "T12" (id 0) (at 132.8166 73.2282 0))
     (property "Value" "750312504" (id 1) (at 132.8166 75.5396 0))
-    (property "Footprint" "EP13_SMT_H_8PIN_(750312504)" (id 2) (at 133.35 86.36 0)
+    (property "Footprint" "750312504:EP13_SMT_H_8PIN_(750312504)" (id 2) (at 133.35 86.36 0)
       (effects (font (size 1.27 1.27)) (justify left bottom) hide)
     )
@@
       (effects (font (size 1.27 1.27)) (justify left bottom) hide)
     )
-    (pin "3")
-    (pin "4")
-    (pin "5")
-    (pin "6")
-    (pin "S2")
+    (pin "1")
+    (pin "2")
+    (pin "7")
+    (pin "8")
+    (pin "S1")
   )
 )

Commit message: refined in-out routing mechanism
Parts:
- renumbered C164 to C140, C165 to C141, C166 to C142, C167 to C143, C168 to C144, C169 to C145, C170 to C146, C171 to C147, C172 to C148, C173 to C149, C174 to C150, D38 to D34, D39 to D35, Q35 to Q29, R191 to R167, R192 to R168, R193 to R169, R194 to R170, R195 to R171, R196 to R172, R197 to R173, R198 to R174, R199 to R175, R200 to R176, R201 to R177, R202 to R178, T12 to T10, T24 to T22, TP147 to TP125, TP148 to TP126, TP149 to TP127, TP150 to TP128, TP152 to TP130, TP153 to TP131, TP155 to TP133, TP156 to TP134, TP157 to TP135

Commit message: first proposal routing
Parts:
- renumbered C140 to C164, C141 to C165, C142 to C166, C143 to C167, C144 to C168, C145 to C169, C146 to C170, C147 to C171, C148 to C172, C149 to C173, C150 to C174, D34 to D38, D35 to D39, Q29 to Q35, R167 to R191, R168 to R192, R169 to R193, R170 to R194, R171 to R195, R172 to R196, R173 to R197, R174 to R198, R175 to R199, R176 to R200, R177 to R201, R178 to R202, T10 to T12, T22 to T24, TP125 to TP147, TP126 to TP148, TP127 to TP149, TP128 to TP150, TP130 to TP152, TP131 to TP153, TP133 to TP155, TP134 to TP156, TP135 to TP157
