File: 211006_lmu_r0/active_passive_balance.kicad_sch (KiCad schematic)
At the start: 38 parts, among them Q2 BSS308PE, T1 750312504, T13 BUK9K13-60EX

Commit message: started to export and fix things
Parts:
- C32, C34, C39, C40: Voltage (none) -> 100V
- C35, C36: Voltage 100V -> (none)
- D15: MANUFACTURER Diodes Inc -> (none)
- T13: Manufacturer (none) -> -; Part Number (none) -> -
Changed lines of the file:
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@@
-      (effects (font (size 1.27 1.27)) (justify left bottom) hide)
-    )
-    (property "MANUFACTURER" "Diodes Inc" (id 4) (at 22.86 99.06 0)
       (effects (font (size 1.27 1.27)) (justify left bottom) hide)
     )
@@
       (effects (font (size 1.27 1.27)) hide)
     )
-    (property "Voltage" "100V" (id 4) (at 153.67 92.71 0)
+    (property "Voltage" "" (id 4) (at 153.67 92.71 0)
       (effects (font (size 1.27 1.27)) hide)
     )
@@
       (effects (font (size 1.27 1.27)) hide)
     )
+    (property "Voltage" "100V" (id 6) (at 86.36 82.55 0)
+      (effects (font (size 1.27 1.27)) hide)
+    )
     (pin "1")
     (pin "2")
@@
     )
     (property "Part Number" "1210F107Z6R3CT" (id 5) (at 97.79 82.55 0)
+      (effects (font (size 1.27 1.27)) hide)
+    )
+    (property "Voltage" "100V" (id 6) (at 97.79 82.55 0)
       (effects (font (size 1.27 1.27)) hide)
     )
@@
       (effects (font (size 1.27 1.27)) hide)
     )
+    (property "Voltage" "100V" (id 6) (at 175.26 85.09 0)
+      (effects (font (size 1.27 1.27)) hide)
+    )
     (pin "1")
     (pin "2")
@@
     )
     (property "Part Number" "1210F107Z6R3CT" (id 5) (at 186.69 85.09 0)
+      (effects (font (size 1.27 1.27)) hide)
+    )
+    (property "Voltage" "100V" (id 6) (at 186.69 85.09 0)
       (effects (font (size 1.27 1.27)) hide)
     )
@@
       (effects (font (size 1.27 1.27)) hide)
     )
-    (property "Voltage" "100V" (id 4) (at 111.76 91.44 0)
+    (property "Voltage" "" (id 4) (at 111.76 91.44 0)
       (effects (font (size 1.27 1.27)) hide)
     )
@@
       (effects (font (size 1.27 1.27)) (justify left bottom) hide)
     )
+    (property "Manufacturer" "-" (id 4) (at 109.22 101.6 0)
+      (effects (font (size 1.27 1.27)) hide)
+    )
+    (property "Part Number" "-" (id 5) (at 109.22 101.6 0)
+      (effects (font (size 1.27 1.27)) hide)
+    )
     (pin "1")
     (pin "2")
@@
       (effects (font (size 1.27 1.27)) (justify left bottom) hide)
     )
+    (property "Manufacturer" "-" (id 4) (at 156.21 101.6 0)
+      (effects (font (size 1.27 1.27)) hide)
+    )
+    (property "Part Number" "-" (id 5) (at 156.21 101.6 0)
+      (effects (font (size 1.27 1.27)) hide)
+    )
     (pin "3")

Commit message: more changes
Parts:
- renumbered C90 to C102, C31 to C43, C32 to C44, C33 to C45, C34 to C46, C35 to C47, C36 to C48, C37 to C49, C38 to C50, C39 to C51, C40 to C52, C41 to C53, D15 to D17, D16 to D18, Q2 to Q5, R31 to R43, R32 to R44, R33 to R45, R34 to R46, R35 to R47, R36 to R48, R37 to R49, R38 to R50, R39 to R51, R40 to R52, R41 to R53, R42 to R54, T13 to T14, T1 to T2, TP26 to TP37, TP28 to TP39, TP29 to TP40, TP31 to TP42, TP32 to TP43, TP34 to TP45, TP35 to TP46, TP36 to TP47
