File: 211006_lmu_r0/file615D6D62.kicad_sch (KiCad schematic)
At the start: 30 parts, among them U1 R-78C5.0-1.0

Commit message: started layout
Connections:
- net +3V3_ISO: no longer R251.1
- net +5V_HV: now also R251.1
- net GND_HV: now also D6.1 (K)
- net GND_ISO: no longer D6.1 (K)
Changed lines of the file:
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@@
     (pin "2")
+  )
+  (symbol (lib_id "+5v_hv:+5V_HV") (at 269.24 57.15 0) (unit 1)
+    (in_bom yes) (on_board yes) (fields_autoplaced)
+    (property "Reference" "#PWR?" (id 0) (at 269.24 60.96 0)
+      (effects (font (size 1.27 1.27)) hide)
+    )
+    (property "Value" "+5V_HV" (id 1) (at 269.24 52.07 0))
+    (property "Footprint" "" (id 2) (at 269.24 57.15 0)
+      (effects (font (size 1.27 1.27)) hide)
+    )
+    (property "Datasheet" "" (id 3) (at 269.24 57.15 0)
+      (effects (font (size 1.27 1.27)) hide)
+    )
+    (pin "1")
   )
   (symbol (lib_id "power:GND") (at 191.77 71.12 0) (unit 1)
@@
     )
     (property "Datasheet" "" (id 3) (at 191.77 71.12 0)
-      (effects (font (size 1.27 1.27)) hide)
-    )
-    (pin "1")
-  )
-  (symbol (lib_name "+3V3_ISO_1") (lib_id "+3v3_iso:+3V3_ISO") (at 269.24 57.15 0) (unit 1)
-    (in_bom yes) (on_board yes)
-    (property "Reference" "#PWR023" (id 0) (at 269.24 60.96 0)
-      (effects (font (size 1.27 1.27)) hide)
-    )
-    (property "Value" "+3V3_ISO" (id 1) (at 269.621 52.7558 0))
-    (property "Footprint" "" (id 2) (at 269.24 57.15 0)
-      (effects (font (size 1.27 1.27)) hide)
-    )
-    (property "Datasheet" "" (id 3) (at 269.24 57.15 0)
       (effects (font (size 1.27 1.27)) hide)
     )
@@
     (pin "2")
   )
-  (symbol (lib_id "gnd_iso:GND_ISO") (at 269.24 73.66 0) (unit 1)
-    (in_bom yes) (on_board yes)
-    (property "Reference" "#PWR024" (id 0) (at 269.24 80.01 0)
+  (symbol (lib_id "gnd_hv:GND_HV") (at 269.24 73.66 0) (unit 1)
+    (in_bom yes) (on_board yes) (fields_autoplaced)
+    (property "Reference" "#PWR?" (id 0) (at 269.24 80.01 0)
       (effects (font (size 1.27 1.27)) hide)
     )
-    (property "Value" "GND_ISO" (id 1) (at 269.367 78.0542 0))
+    (property "Value" "GND_HV" (id 1) (at 269.24 78.74 0))
     (property "Footprint" "" (id 2) (at 269.24 73.66 0)
       (effects (font (size 1.27 1.27)) hide)

Commit message: trying out a quick thing, recover
Changed lines of the file:
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@@
   (junction (at 92.71 97.79) (diameter 0) (color 0 0 0 0)
   )
-  (junction (at 245.11 60.96) (diameter 0) (color 0 0 0 0)
-  )
   (junction (at 236.22 71.12) (diameter 0) (color 0 0 0 0)
   )
@@
   (junction (at 142.24 107.95) (diameter 0) (color 0 0 0 0)
   )
-  (junction (at 245.11 71.12) (diameter 0) (color 0 0 0 0)
-  )
   (junction (at 48.26 105.41) (diameter 0) (color 0 0 0 0)
   )
   (junction (at 177.8 107.95) (diameter 0) (color 0 0 0 0)
   )
-  (junction (at 245.11 97.79) (diameter 0) (color 0 0 0 0)
-  )
   (junction (at 165.1 107.95) (diameter 0) (color 0 0 0 0)
   )
-  (junction (at 245.11 107.95) (diameter 0) (color 0 0 0 0)
-  )
   (junction (at 106.68 105.41) (diameter 0) (color 0 0 0 0)
   )
@@
     (stroke (width 0) (type default) (color 0 0 0 0))
   )
-  (wire (pts (xy 255.27 60.96) (xy 245.11 60.96))
-    (stroke (width 0) (type default) (color 0 0 0 0))
-  )
   (wire (pts (xy 196.85 71.12) (xy 191.77 71.12))
-    (stroke (width 0) (type default) (color 0 0 0 0))
-  )
-  (wire (pts (xy 255.27 97.79) (xy 245.11 97.79))
     (stroke (width 0) (type default) (color 0 0 0 0))
   )
@@
     (stroke (width 0) (type default) (color 0 0 0 0))
   )
-  (wire (pts (xy 255.27 107.95) (xy 245.11 107.95))
-    (stroke (width 0) (type default) (color 0 0 0 0))
-  )
   (wire (pts (xy 190.5 107.95) (xy 196.85 107.95))
     (stroke (width 0) (type default) (color 0 0 0 0))
@@
   )
   (wire (pts (xy 190.5 107.95) (xy 177.8 107.95))
-    (stroke (width 0) (type default) (color 0 0 0 0))
-  )
-  (wire (pts (xy 255.27 71.12) (xy 245.11 71.12))
     (stroke (width 0) (type default) (color 0 0 0 0))
   )
@@
     (effects (font (size 1.27 1.27)) (justify left bottom))
   )
-  (global_label "0V_HV" (shape input) (at 255.27 71.12 0) (fields_autoplaced)
-    (effects (font (size 1.27 1.27)) (justify left))
-    (property "Intersheet References" "${INTERSHEET_REFS}" (id 0) (at 263.279 71.0406 0)
-      (effects (font (size 1.27 1.27)) (justify left) hide)
-    )
-  )
-  (global_label "5V_HV" (shape input) (at 255.27 60.96 0) (fields_autoplaced)
-    (effects (font (size 1.27 1.27)) (justify left))
-    (property "Intersheet References" "${INTERSHEET_REFS}" (id 0) (at 263.279 60.8806 0)
-      (effects (font (size 1.27 1.27)) (justify left) hide)
-    )
-  )
-  (global_label "3.3V_ISO" (shape input) (at 255.27 97.79 0) (fields_autoplaced)
-    (effects (font (size 1.27 1.27)) (justify left))
-    (property "Intersheet References" "${INTERSHEET_REFS}" (id 0) (at -1.27 38.1 0)
-      (effects (font (size 1.27 1.27)) hide)
-    )
-  )
-  (global_label "0V_ISO" (shape input) (at 255.27 107.95 0) (fields_autoplaced)
-    (effects (font (size 1.27 1.27)) (justify left))
-    (property "Intersheet References" "${INTERSHEET_REFS}" (id 0) (at -1.27 38.1 0)
-      (effects (font (size 1.27 1.27)) hide)
-    )
-  )
   (hierarchical_label "VBAT+" (shape input) (at 46.99 97.79 180)

Commit message: silkscreen changes, shifting bun leds
Parts:
- PS2: footprint CONV_R2S-0505 -> R2S-0505:CONV_R2S-0505
- TP1, TP2, TP3, TP30, TP33, TP4, TP5, TP6, TP7: footprint TestPoint:TestPoint_Pad_D1.0mm -> custom:TestPoint_Pad_D1.0mm
Connections:
- net VBAT_FUSED: now reaches D1.1 (A1), D2.2 (A), F1.2
Changed lines of the file:
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@@
+    (effects (font (size 1.27 1.27)) (justify left bottom))
+  )
+  (label "VBAT_FUSED" (at 62.23 97.79 0)
     (effects (font (size 1.27 1.27)) (justify left bottom))
   )
@@
       (effects (font (size 1.27 1.27)) (justify left))
     )
-    (property "Footprint" "TestPoint:TestPoint_Pad_D1.0mm" (id 2) (at 147.32 97.79 0)
+    (property "Footprint" "custom:TestPoint_Pad_D1.0mm" (id 2) (at 147.32 97.79 0)
       (effects (font (size 1.27 1.27)) hide)
     )
@@
       (effects (font (size 1.27 1.27)) (justify left))
     )
-    (property "Footprint" "TestPoint:TestPoint_Pad_D1.0mm" (id 2) (at 97.79 97.79 0)
+    (property "Footprint" "custom:TestPoint_Pad_D1.0mm" (id 2) (at 97.79 97.79 0)
       (effects (font (size 1.27 1.27)) hide)
     )
@@
       (effects (font (size 1.27 1.27)) (justify left))
     )
-    (property "Footprint" "TestPoint:TestPoint_Pad_D1.0mm" (id 2) (at 53.34 97.79 0)
+    (property "Footprint" "custom:TestPoint_Pad_D1.0mm" (id 2) (at 53.34 97.79 0)
       (effects (font (size 1.27 1.27)) hide)
     )
@@
       (effects (font (size 1.27 1.27)) (justify right))
     )
-    (property "Footprint" "TestPoint:TestPoint_Pad_D1.0mm" (id 2) (at 43.18 105.41 0)
+    (property "Footprint" "custom:TestPoint_Pad_D1.0mm" (id 2) (at 43.18 105.41 0)
       (effects (font (size 1.27 1.27)) hide)
     )
@@
       (effects (font (size 1.27 1.27)) (justify right))
     )
-    (property "Footprint" "TestPoint:TestPoint_Pad_D1.0mm" (id 2) (at 137.16 107.95 0)
+    (property "Footprint" "custom:TestPoint_Pad_D1.0mm" (id 2) (at 137.16 107.95 0)
       (effects (font (size 1.27 1.27)) hide)
     )
@@
       (effects (font (size 1.27 1.27)) (justify left))
     )
-    (property "Footprint" "TestPoint:TestPoint_Pad_D1.0mm" (id 2) (at 250.19 97.79 0)
+    (property "Footprint" "custom:TestPoint_Pad_D1.0mm" (id 2) (at 250.19 97.79 0)
       (effects (font (size 1.27 1.27)) hide)
     )
@@
       (effects (font (size 1.27 1.27)) (justify right))
     )
-    (property "Footprint" "TestPoint:TestPoint_Pad_D1.0mm" (id 2) (at 240.03 107.95 0)
+    (property "Footprint" "custom:TestPoint_Pad_D1.0mm" (id 2) (at 240.03 107.95 0)
       (effects (font (size 1.27 1.27)) hide)
     )
@@
     (property "Reference" "PS2" (id 0) (at 212.09 53.34 0))
     (property "Value" "R2S-0505" (id 1) (at 212.09 55.88 0))
-    (property "Footprint" "CONV_R2S-0505" (id 2) (at 212.09 66.04 0)
+    (property "Footprint" "R2S-0505:CONV_R2S-0505" (id 2) (at 212.09 66.04 0)
       (effects (font (size 1.27 1.27)) (justify left bottom) hide)
     )
@@
       (effects (font (size 1.27 1.27)) (justify left))
     )
-    (property "Footprint" "TestPoint:TestPoint_Pad_D1.0mm" (id 2) (at 250.19 60.96 0)
+    (property "Footprint" "custom:TestPoint_Pad_D1.0mm" (id 2) (at 250.19 60.96 0)
       (effects (font (size 1.27 1.27)) hide)
     )
@@
       (effects (font (size 1.27 1.27)) (justify right))
     )
-    (property "Footprint" "TestPoint:TestPoint_Pad_D1.0mm" (id 2) (at 240.03 71.12 0)
-      (effects (font (size 1.27 1.27)) hide)
-    )
+    (property "Footprint" "custom:TestPoint_Pad_D1.0mm" (id 2) (at 240.03 71.12 0)
+      (effects (font (size 1.27 1.27)) hide)
+    )

Commit message: started to export and fix things
Parts:
- PS1: MANUFACTURER RECOM -> (none); MAXIMUM_PACKAGE_HEIGHT 9.0mm -> (none); PARTREV 0 -> (none); STANDARD Manufacturer Recommendations -> (none)
- PS2: MANUFACTURER RECOM -> (none); MAXIMUM_PACKAGE_HEIGHT 9.0mm -> (none); Manufacturer (none) -> -; PARTREV 0 -> (none); STANDARD Manufacturer Recommendations -> (none)
Changed lines of the file:
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@@
-      (effects (font (size 1.27 1.27)) (justify left bottom) hide)
-    )
-    (property "MANUFACTURER" "RECOM" (id 4) (at 212.09 102.87 0)
-      (effects (font (size 1.27 1.27)) (justify left bottom) hide)
-    )
-    (property "MAXIMUM_PACKAGE_HEIGHT" "9.0mm" (id 5) (at 212.09 102.87 0)
-      (effects (font (size 1.27 1.27)) (justify left bottom) hide)
-    )
-    (property "STANDARD" "Manufacturer Recommendations" (id 6) (at 212.09 102.87 0)
-      (effects (font (size 1.27 1.27)) (justify left bottom) hide)
-    )
-    (property "PARTREV" "0" (id 7) (at 212.09 102.87 0)
       (effects (font (size 1.27 1.27)) (justify left bottom) hide)
     )
@@
       (effects (font (size 1.27 1.27)) (justify left bottom) hide)
     )
-    (property "MANUFACTURER" "RECOM" (id 4) (at 212.09 66.04 0)
-      (effects (font (size 1.27 1.27)) (justify left bottom) hide)
-    )
-    (property "MAXIMUM_PACKAGE_HEIGHT" "9.0mm" (id 5) (at 212.09 66.04 0)
-      (effects (font (size 1.27 1.27)) (justify left bottom) hide)
-    )
-    (property "STANDARD" "Manufacturer Recommendations" (id 6) (at 212.09 66.04 0)
-      (effects (font (size 1.27 1.27)) (justify left bottom) hide)
-    )
-    (property "PARTREV" "0" (id 7) (at 212.09 66.04 0)
-      (effects (font (size 1.27 1.27)) (justify left bottom) hide)
-    )
-    (pin "1")
+    (property "Manufacturer" "-" (id 4) (at 212.09 66.04 0)
+      (effects (font (size 1.27 1.27)) hide)
+    )
+    (pin "1")
