File: 211006_lmu_r0/file61711469.kicad_sch (KiCad schematic)
At the start: 4 parts, among them IC1 ADS7028QRTERQ1

Commit message: started to export and fix things
Parts:
- IC1: Height 0.8 -> (none); Mouser Price/Stock https://au.mouser.com/ProductDetail/Texas-Instruments/ADS70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 -> (none)
Changed lines of the file:
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@@
-      (effects (font (size 1.27 1.27)) (justify left) hide)
-    )
-    (property "Height" "0.8" (id 5) (at 189.23 80.01 0)
       (effects (font (size 1.27 1.27)) (justify left) hide)
     )
@@
       (effects (font (size 1.27 1.27)) (justify left) hide)
     )
-    (property "Mouser Price/Stock" "https://au.mouser.com/ProductDetail/Texas-Instruments/ADS7028IRTER?qs=%252B6g0mu59x7L0mzHBJBWvJw%3D%3D" (id 7) (at 189.23 85.09 0)
-      (effects (font (size 1.27 1.27)) (justify left) hide)
-    )
-    (property "Manufacturer_Name" "" (id 8) (at 189.23 87.63 0)
-      (effects (font (size 1.27 1.27)) (justify left) hide)
-    )
-    (property "Manufacturer_Part_Number" "" (id 9) (at 189.23 90.17 0)
-      (effects (font (size 1.27 1.27)) (justify left) hide)
-    )
