File: 220203_terminal_board_r0/220203_terminal_board_r0/220203_terminal_board_r0.kicad_sch (KiCad schematic)
At the start: 38 parts, among them J1 Conn_01x13

Commit message: changed to M4 terminal boards
Parts:
- H1, H10, H11, H12, H13, H14, H15, H16, H17, H18, H19, H2, H20, H21, H22, H23, H24, H3, H4, H5, H6, H7, H8, H9: footprint MountingHole:MountingHole_5.5mm_Pad_Via -> MountingHole:MountingHole_4.3mm_M4_Pad_Via
